Commit message: vhacd objects

File: myGym/envs/objects/assembly/urdf/car_roof.urdf (robot description, URDF)
Before this commit: robot car_roof, 1 links, 0 joints
Links:
- link baseLink: geometry collision mesh filename=../obj/car_roof_vhacd.obj scale=.001 .001 .001; visual mesh filename=../obj/car_roof_vhacd.obj scale=.001 .001 .001

File: myGym/envs/objects/assembly/urdf/cube_holes.urdf (robot description, URDF)
Before this commit: robot cube_holes, 1 links, 0 joints
Links:
- link baseLink: geometry collision mesh filename=../obj/cube_holes_vhacd.obj scale=.001 .001 .001; visual mesh filename=../obj/cube_holes_vhacd.obj scale=.001 .001 .001

File: myGym/envs/objects/assembly/urdf/ex_bucket.urdf (robot description, URDF)
Before this commit: robot ex_bucket, 1 links, 0 joints
Links:
- link baseLink: geometry collision mesh filename=../obj/ex_bucket_vhacd.obj scale=.001 .001 .001; visual mesh filename=../obj/ex_bucket_vhacd.obj scale=.001 .001 .001

File: myGym/envs/objects/assembly/urdf/hammer.urdf (robot description, URDF)
Before this commit: robot hammer, 1 links, 0 joints
Links:
- link baseLink: geometry collision mesh filename=../obj/hammer_vhacd.obj scale=.008 .008 .008; visual mesh filename=../obj/hammer_vhacd.obj scale=.008 .008 .008

File: myGym/envs/objects/assembly/urdf/nut.urdf (robot description, URDF)
Before this commit: robot nut, 1 links, 0 joints
Links:
- link baseLink: geometry collision mesh filename=../obj/nut_vhacd.obj scale=.001 .001 .001; visual mesh filename=../obj/nut_vhacd.obj scale=.001 .001 .001

File: myGym/envs/objects/assembly/urdf/peg_screw.urdf (robot description, URDF)
Before this commit: robot peg_screw, 1 links, 0 joints
Links:
- link baseLink: geometry collision mesh filename=../obj/peg_screw_vhacd.obj scale=.001 .001 .001; visual mesh filename=../obj/peg_screw_vhacd.obj scale=.001 .001 .001

File: myGym/envs/objects/assembly/urdf/pliers.urdf (robot description, URDF)
Before this commit: robot pliers, 1 links, 0 joints
Links:
- link baseLink: geometry collision mesh filename=../obj/pliers_vhacd.obj scale=.02 .02 .02; visual mesh filename=../obj/pliers_vhacd.obj scale=.02 .02 .02

File: myGym/envs/objects/assembly/urdf/screw_round.urdf (robot description, URDF)
Before this commit: robot screw_round, 1 links, 0 joints
Links:
- link baseLink: geometry collision mesh filename=../obj/screw_round_vhacd.obj scale=.001 .001 .001; visual mesh filename=../obj/screw_round_vhacd.obj scale=.001 .001 .001

File: myGym/envs/objects/assembly/urdf/screwdriver.urdf (robot description, URDF)
Before this commit: robot screwdriver, 1 links, 0 joints
Links:
- link baseLink: geometry collision mesh filename=../obj/screwdriver_vhacd.obj scale=.001 .001 .001; visual mesh filename=../obj/screwdriver_vhacd.obj scale=.001 .001 .001

File: myGym/envs/objects/assembly/urdf/sphere_holes.urdf (robot description, URDF)
Before this commit: robot sphere_holes, 1 links, 0 joints
Links:
- link baseLink: geometry collision mesh filename=../obj/sphere_holes_vhacd.obj scale=.001 .001 .001; visual mesh filename=../obj/sphere_holes_vhacd.obj scale=.001 .001 .001

File: myGym/envs/objects/assembly/urdf/wafer.urdf (robot description, URDF)
Before this commit: robot wafer, 1 links, 0 joints
Links:
- link baseLink: geometry collision mesh filename=../obj/wafer_vhacd.obj scale=.001 .001 .001; visual mesh filename=../obj/wafer_vhacd.obj scale=.001 .001 .001

File: myGym/envs/objects/assembly/urdf/wheel.urdf (robot description, URDF)
Before this commit: robot wheel, 1 links, 0 joints
Links:
- link baseLink: geometry collision mesh filename=../obj/wheel_vhacd.obj scale=.001 .001 .001; visual mesh filename=../obj/wheel_vhacd.obj scale=.001 .001 .001

File: myGym/envs/objects/assembly/urdf/wrench.urdf (robot description, URDF)
Before this commit: robot wrench, 1 links, 0 joints
Links:
- link baseLink: geometry collision mesh filename=../obj/wrench_vhacd.obj scale=.001 .001 .001; visual mesh filename=../obj/wrench_vhacd.obj scale=.001 .001 .001

File: myGym/envs/objects/furniture/urdf/armchair.urdf (robot description, URDF)
Before this commit: robot armchair, 1 links, 0 joints
Links:
- link baseLink: geometry collision mesh filename=../obj/armchair_vhacd.obj scale=0.02 0.02 0.02; visual mesh filename=../obj/armchair_vhacd.obj scale=0.02 0.02 0.02

File: myGym/envs/objects/furniture/urdf/bookcase.urdf (robot description, URDF)
Before this commit: robot bookcase, 1 links, 0 joints
Links:
- link baseLink: geometry collision mesh filename=../obj/bookcase_vhacd.obj scale=0.02 0.02 0.02; visual mesh filename=../obj/bookcase_vhacd.obj scale=0.02 0.02 0.02

File: myGym/envs/objects/furniture/urdf/chair.urdf (robot description, URDF)
Before this commit: robot chair, 1 links, 0 joints
Links:
- link baseLink: geometry collision mesh filename=../obj/chair_vhacd.obj scale=0.02 0.02 0.02; visual mesh filename=../obj/chair_vhacd.obj scale=0.02 0.02 0.02

File: myGym/envs/objects/furniture/urdf/cupboard.urdf (robot description, URDF)
Before this commit: robot cupboard, 1 links, 0 joints
Links:
- link baseLink: geometry collision mesh filename=../obj/cupboard_vhacd.obj scale=0.02 0.02 0.02; visual mesh filename=../obj/cupboard_vhacd.obj scale=0.02 0.02 0.02

File: myGym/envs/objects/furniture/urdf/sofa.urdf (robot description, URDF)
Before this commit: robot sofa, 1 links, 0 joints
Links:
- link baseLink: geometry collision mesh filename=../obj/sofa_vhacd.obj scale=0.02 0.02 0.02; visual mesh filename=../obj/sofa_vhacd.obj scale=0.02 0.02 0.02

File: myGym/envs/objects/furniture/urdf/table.urdf (robot description, URDF)
Before this commit: robot table, 1 links, 0 joints
Links:
- link baseLink: geometry collision mesh filename=../obj/table_vhacd.obj scale=0.02 0.02 0.02; visual mesh filename=../obj/table_vhacd.obj scale=0.02 0.02 0.02

File: myGym/envs/objects/geometric/urdf/cube.urdf (robot description, URDF)
Before this commit: robot cube.urdf, 1 links, 0 joints
Links:
- link baseLink: geometry collision mesh filename=./obj/cube_vhacd.obj scale=.001 .001 .001; visual mesh filename=./obj/cube_vhacd.obj scale=.001 .001 .001
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