Commit message: gripping ability update

File: myGym/envs/objects/assembly/urdf/kostka1.urdf (robot description, URDF)
Before this commit: robot cube_holes, 1 links, 0 joints
Links:
- link baseLink: mass 1 -> 10; geometry collision box size=.2 .05 .1; visual box size=.2 .05 .1

File: myGym/envs/robots/franka_emika/panda/urdf/panda1.urdf (robot description, URDF)
Before this commit: robot panda, 14 links, 13 joints
Joints:
- joint panda_finger_gjoint1: limit lower=0.0 upper=0.04 effort=30 velocity=1 -> lower=0.0 upper=0.06 effort=100 velocity=10
- joint panda_finger_gjoint2: limit lower=0.0 upper=0.04 effort=30 velocity=1 -> lower=0.0 upper=0.06 effort=100 velocity=10
