Commit message: verbose debug and multi network eval callback debug

File: myGym/envs/objects/assembly/urdf/towertarget.urdf (robot description, URDF)
Before this commit: robot towertarget, 1 links, 0 joints
Links:
- link baseLink: mass None -> 1

File: myGym/envs/robots/kuka_magnetic_gripper_sdf/kuka_magnetic.urdf (robot description, URDF)
Before this commit: robot lbr_iiwa, 13 links, 12 joints
Links:
- link endeffector: mass None -> 0
