Commit message: object color dict, bug fixes

File: myGym/envs/objects/storage/urdf/crate.urdf (robot description, URDF)
Before this commit: robot crate, 1 links, 0 joints
Links:
- link baseLink: geometry collision mesh filename=../obj/crate.obj scale=0.0007 0.001 0.001; visual mesh filename=../obj/crate.obj scale=0.0007 0.001 0.001
