Commit message: test scrpit update + robot urdf with similar velocity and force

File: myGym/envs/robots/franka_emika/panda/urdf/panda.urdf (robot description, URDF)
Before this commit: robot panda, 13 links, 12 joints
Joints:
- joint panda_finger_joint1: limit lower=0.0 upper=0.04 effort=20 velocity=0.2 -> lower=0.0 upper=0.04 effort=30 velocity=1
- joint panda_finger_joint2: limit lower=0.0 upper=0.04 effort=20 velocity=0.2 -> lower=0.0 upper=0.04 effort=30 velocity=1
- joint panda_joint1: limit lower=-2.9671 upper=2.9671 effort=87 velocity=2.1750 -> lower=-2.9671 upper=2.9671 effort=30 velocity=1
- joint panda_joint2: limit lower=-1.8326 upper=1.8326 effort=87 velocity=2.1750 -> lower=-1.8326 upper=1.8326 effort=87 velocity=1
- joint panda_joint3: limit lower=-2.9671 upper=2.9671 effort=87 velocity=2.1750 -> lower=-2.9671 upper=2.9671 effort=30 velocity=1
- joint panda_joint4: limit lower=-3.1416 upper=0.0 effort=87 velocity=2.1750 -> lower=-3.1416 upper=0.0 effort=30 velocity=1
- joint panda_joint5: limit lower=-2.9671 upper=2.9671 effort=12 velocity=2.6100 -> lower=-2.9671 upper=2.9671 effort=30 velocity=1
- joint panda_joint6: limit lower=-0.0873 upper=3.8223 effort=12 velocity=2.6100 -> lower=-0.0873 upper=3.8223 effort=30 velocity=1
- joint panda_joint7: limit lower=-2.9671 upper=2.9671 effort=12 velocity=2.6100 -> lower=-2.9671 upper=2.9671 effort=30 velocity=1

File: myGym/envs/robots/jaco_arm/jaco/urdf/jaco_robotiq.urdf (robot description, URDF)
Before this commit: robot j2s7s300, 19 links, 18 joints
Joints:
- joint j2s7s300_joint_1: limit lower=-6.28318530718 upper=6.28318530718 effort=2000 velocity=10.0 -> lower=-6.28318530718 upper=6.28318530718 effort=40 velocity=1.0
- joint j2s7s300_joint_2: limit lower=0.523598775598 upper=5.75958653158 effort=2000 velocity=1 -> lower=0.523598775598 upper=5.75958653158 effort=40 velocity=1
- joint j2s7s300_joint_3: limit lower=-6.28318530718 upper=6.28318530718 effort=2000 velocity=1 -> lower=-6.28318530718 upper=6.28318530718 effort=40 velocity=1
- joint j2s7s300_joint_4: limit lower=0.523598775598 upper=5.75958653158 effort=2000 velocity=1 -> lower=0.523598775598 upper=5.75958653158 effort=40 velocity=1
- joint j2s7s300_joint_5: limit lower=-6.28318530718 upper=6.28318530718 effort=2000 velocity=1 -> lower=-6.28318530718 upper=6.28318530718 effort=40 velocity=1
- joint j2s7s300_joint_6: limit lower=0.523598775598 upper=5.75958653158 effort=2000 velocity=1 -> lower=0.523598775598 upper=5.75958653158 effort=40 velocity=1
- joint j2s7s300_joint_7: limit lower=-3.14159265359 upper=3.14159265359 effort=600.8 velocity=0.785 -> lower=-3.14159265359 upper=3.14159265359 effort=40 velocity=0.785
- joint robotiq_85_left_finger_joint: limit lower=-3.14 upper=3.14 velocity=100.0 -> lower=-3.14 upper=3.14 velocity=1.0
- joint robotiq_85_left_finger_tip_joint: limit lower=-0.8757 upper=0.0 velocity=100.0 -> lower=-0.8757 upper=0.0 velocity=1.0
- joint robotiq_85_left_inner_knuckle_joint: limit lower=0.0 upper=0.8757 velocity=100.0 -> lower=0.0 upper=0.8757 velocity=1.0
- joint robotiq_85_left_knuckle_joint: limit lower=0.0 upper=0.81 velocity=100.0 -> lower=0.0 upper=0.81 velocity=1.0
- joint robotiq_85_right_finger_joint: limit lower=-3.14 upper=3.14 velocity=100.0 -> lower=-3.14 upper=3.14 velocity=1.0
- joint robotiq_85_right_finger_tip_joint: limit lower=-0.8757 upper=0.0 velocity=100.0 -> lower=-0.8757 upper=0.0 velocity=1.0
- joint robotiq_85_right_inner_knuckle_joint: limit lower=0.0 upper=0.8757 velocity=100.0 -> lower=0.0 upper=0.8757 velocity=1.0
- joint robotiq_85_right_knuckle_joint: limit lower=0.0 upper=0.81 velocity=100.0 -> lower=0.0 upper=0.81 velocity=1.0

File: myGym/envs/robots/jaco_arm/jaco/urdf/jaco_robotiq_fixed.urdf (robot description, URDF)
Before this commit: robot j2s7s300, 19 links, 18 joints
Joints:
- joint j2s7s300_joint_1: limit lower=-6.28318530718 upper=6.28318530718 effort=2000 velocity=10.0 -> lower=-6.28318530718 upper=6.28318530718 effort=40 velocity=1.0
- joint j2s7s300_joint_2: limit lower=0.523598775598 upper=5.75958653158 effort=2000 velocity=1 -> lower=0.523598775598 upper=5.75958653158 effort=40 velocity=1
- joint j2s7s300_joint_3: limit lower=-6.28318530718 upper=6.28318530718 effort=2000 velocity=1 -> lower=-6.28318530718 upper=6.28318530718 effort=40 velocity=1
- joint j2s7s300_joint_4: limit lower=0.523598775598 upper=5.75958653158 effort=2000 velocity=1 -> lower=0.523598775598 upper=5.75958653158 effort=40 velocity=1
- joint j2s7s300_joint_5: limit lower=-6.28318530718 upper=6.28318530718 effort=2000 velocity=1 -> lower=-6.28318530718 upper=6.28318530718 effort=40 velocity=1
- joint j2s7s300_joint_6: limit lower=0.523598775598 upper=5.75958653158 effort=2000 velocity=1 -> lower=0.523598775598 upper=5.75958653158 effort=40 velocity=1
- joint j2s7s300_joint_7: limit lower=-3.14159265359 upper=3.14159265359 effort=600.8 velocity=0.785 -> lower=-3.14159265359 upper=3.14159265359 effort=40 velocity=1
- joint robotiq_85_left_finger_joint: limit lower=-3.14 upper=3.14 velocity=100.0 -> lower=-3.14 upper=3.14 velocity=1.0
- joint robotiq_85_left_finger_tip_joint: limit lower=-0.8757 upper=0.0 velocity=100.0 -> lower=-0.8757 upper=0.0 velocity=1.0
- joint robotiq_85_left_inner_knuckle_joint: limit lower=0.0 upper=0.8757 velocity=100.0 -> lower=0.0 upper=0.8757 velocity=1.0
- joint robotiq_85_left_knuckle_joint: limit lower=0.0 upper=0.81 velocity=100.0 -> lower=0.0 upper=0.81 velocity=1.0
- joint robotiq_85_right_finger_joint: limit lower=-3.14 upper=3.14 velocity=100.0 -> lower=-3.14 upper=3.14 velocity=1.0
- joint robotiq_85_right_finger_tip_joint: limit lower=-0.8757 upper=0.0 velocity=100.0 -> lower=-0.8757 upper=0.0 velocity=1.0
- joint robotiq_85_right_inner_knuckle_joint: limit lower=0.0 upper=0.8757 velocity=100.0 -> lower=0.0 upper=0.8757 velocity=1.0
- joint robotiq_85_right_knuckle_joint: limit lower=0.0 upper=0.81 velocity=100.0 -> lower=0.0 upper=0.81 velocity=1.0

File: myGym/envs/robots/kuka_gripper/kuka_gripper.urdf (robot description, URDF)
Before this commit: robot kuka_gripper, 17 links, 16 joints
Joints:
- joint base_to_finger00_joint: limit lower=0 upper=1.5707963267948966 effort=300 velocity=10 -> lower=0 upper=1.5707963267948966 effort=30 velocity=1
- joint base_to_finger10_joint: limit lower=0 upper=1.5707963267948966 effort=300 velocity=10 -> lower=0 upper=1.5707963267948966 effort=30 velocity=1
- joint finger00_to_finger01_joint: limit lower=0 upper=-1.5707963267948966 effort=300 velocity=10 -> lower=0 upper=-1.5707963267948966 effort=30 velocity=1
- joint finger10_to_finger11_joint: limit lower=0 upper=-1.5707963267948966 effort=300 velocity=10 -> lower=0 upper=-1.5707963267948966 effort=30 velocity=1
- joint lbr_iiwa_joint_1: limit lower=-2.96705972839 upper=2.96705972839 effort=300 velocity=10 -> lower=-2.96705972839 upper=2.96705972839 effort=30 velocity=1
- joint lbr_iiwa_joint_2: limit lower=-2.09439510239 upper=2.09439510239 effort=300 velocity=10 -> lower=-2.09439510239 upper=2.09439510239 effort=30 velocity=1
- joint lbr_iiwa_joint_3: limit lower=-2.96705972839 upper=2.96705972839 effort=300 velocity=10 -> lower=-2.96705972839 upper=2.96705972839 effort=30 velocity=1
- joint lbr_iiwa_joint_4: limit lower=-2.09439510239 upper=2.09439510239 effort=300 velocity=10 -> lower=-2.09439510239 upper=2.09439510239 effort=30 velocity=1
- joint lbr_iiwa_joint_5: limit lower=-2.96705972839 upper=2.96705972839 effort=300 velocity=10 -> lower=-2.96705972839 upper=2.96705972839 effort=30 velocity=1
- joint lbr_iiwa_joint_6: limit lower=-2.09439510239 upper=2.09439510239 effort=300 velocity=10 -> lower=-2.09439510239 upper=2.09439510239 effort=30 velocity=1
- joint lbr_iiwa_joint_7: limit lower=-3.05432619099 upper=3.05432619099 effort=300 velocity=10 -> lower=-3.05432619099 upper=3.05432619099 effort=30 velocity=1

File: myGym/envs/robots/pollen/reachy/urdf/leachy.urdf (robot description, URDF)
Before this commit: robot Leachy_w_hand, 10 links, 9 joints
Joints:
- joint head_pitch: limit lower=-3.14159 upper=0.174533 -> lower=-3.14159 upper=0.174533 effort=30 velocity=1
- joint head_yaw: limit lower=-1.5708 upper=3.14159 -> lower=-1.5708 upper=3.14159 effort=30 velocity=1
- joint l_arm_yaw: limit lower=-1.5708 upper=1.5708 -> lower=-1.5708 upper=1.5708 effort=30 velocity=1
- joint l_elbow_pitch: limit lower=-2.18166 upper=0 -> lower=-2.18166 upper=0 effort=30 velocity=1
- joint l_forearm_yaw: limit lower=-2.61799 upper=2.61799 -> lower=-2.61799 upper=2.61799 effort=30 velocity=1
- joint l_shoulder_pitch: limit lower=-1.5708 upper=3.14159 -> lower=-1.5708 upper=3.14159 effort=30 velocity=1
- joint l_shoulder_roll: limit lower=-0.174533 upper=3.14159 -> lower=-0.174533 upper=3.14159 effort=30 velocity=1
- joint l_wrist_pitch: limit lower=-1.22173 upper=1.22173 -> lower=-1.22173 upper=1.22173 effort=30 velocity=1

File: myGym/envs/robots/pollen/reachy/urdf/reachy.urdf (robot description, URDF)
Before this commit: robot Reachy, 11 links, 10 joints
Joints:
- joint arm_yaw: limit lower=-1.5708 upper=1.5708 -> lower=-1.5708 upper=1.5708 effort=30 velocity=1
- joint elbow_pitch: limit lower=-2.18166 upper=0 -> lower=-2.18166 upper=0 effort=30 velocity=1
- joint forearm_yaw: limit lower=-2.61799 upper=2.61799 -> lower=-2.61799 upper=2.61799 effort=30 velocity=1
- joint head_pitch: limit lower=-3.14159 upper=0.174533 -> lower=-3.14159 upper=0.174533 effort=30 velocity=1
- joint head_yaw: limit lower=-1.5708 upper=3.14159 -> lower=-1.5708 upper=3.14159 effort=30 velocity=1
- joint shoulder_pitch: limit lower=-1.5708 upper=3.14159 -> lower=-1.5708 upper=3.14159 effort=30 velocity=1
- joint shoulder_roll: limit lower=-3.14159 upper=0.174533 -> lower=-3.14159 upper=0.174533 effort=30 velocity=1
- joint wrist_pitch: limit lower=-1.22173 upper=1.22173 -> lower=-1.22173 upper=1.22173 effort=30 velocity=1
- joint wrist_roll: limit lower=-1.0472 upper=1.0472 -> lower=-1.0472 upper=1.0472 effort=30 velocity=1
