Commit message: robot control UPDATE - gripper and end effector universalization, robot.py rewritten, urdf changed (rjoint and gjoints), gripper idependetly controlled, gripper=last IK joint, end effector=graspable point

File: myGym/envs/robots/franka_emika/panda/urdf/panda1.urdf (robot description, URDF)
Before this commit: robot panda, 13 links, 12 joints
Links:
- removed link end_effector
- added link endeffector; visual sphere radius=0.01
- added link panda_rightfinger; collision mesh filename=meshes/collision/finger.obj; visual mesh filename=meshes/collision/finger.obj
Joints:
- removed joint panda_finger_joint1
- removed joint panda_finger_joint2
- removed joint panda_joint1
- removed joint panda_joint2
- removed joint panda_joint3
- removed joint panda_joint4
- removed joint panda_joint5
- removed joint panda_joint6
- removed joint panda_joint7
- removed joint panda_joint8
- added joint endeffector_joint: type fixed, parent gripper, child endeffector, origin xyz=0 0.0 0.1 rpy=0 0 0
- added joint panda_finger_gjoint1: type prismatic, parent gripper, child panda_leftfinger, origin xyz=0 0 0.0584 rpy=0 0 0, axis 0 1 0, limit lower=0.0 upper=0.04 effort=30 velocity=1
- added joint panda_finger_gjoint2: type prismatic, parent gripper, child panda_rightfinger, origin xyz=0 0 0.0584 rpy=0 0 0, axis 0 -1 0, limit lower=0.0 upper=0.04 effort=30 velocity=1, mimic joint=panda_finger_gjoint1
- added joint panda_rjoint1: type revolute, parent panda_link0, child panda_link1, origin xyz=0 0 0.333 rpy=0 0 0, axis 0 0 1, limit lower=-2.9671 upper=2.9671 effort=30 velocity=1
- added joint panda_rjoint2: type revolute, parent panda_link1, child panda_link2, origin xyz=0 0 0 rpy=-1.57079632679 0 0, axis 0 0 1, limit lower=-1.8326 upper=1.8326 effort=87 velocity=1
- added joint panda_rjoint3: type revolute, parent panda_link2, child panda_link3, origin xyz=0 -0.316 0 rpy=1.57079632679 0 0, axis 0 0 1, limit lower=-2.9671 upper=2.9671 effort=30 velocity=1
- added joint panda_rjoint4: type revolute, parent panda_link3, child panda_link4, origin xyz=0.0825 0 0 rpy=1.57079632679 0 0, axis 0 0 1, limit lower=-3.1416 upper=0.0 effort=30 velocity=1
- added joint panda_rjoint5: type revolute, parent panda_link4, child panda_link5, origin xyz=-0.0825 0.384 0 rpy=-1.57079632679 0 0, axis 0 0 1, limit lower=-2.9671 upper=2.9671 effort=30 velocity=1
- added joint panda_rjoint6: type revolute, parent panda_link5, child panda_link6, origin xyz=0 0 0 rpy=1.57079632679 0 0, axis 0 0 1, limit lower=-0.0873 upper=3.8223 effort=30 velocity=1
- added joint panda_rjoint7: type revolute, parent panda_link6, child panda_link7, origin xyz=0.088 0 0 rpy=0 0 0, axis 0 0 1, limit lower=-2.9671 upper=2.9671 effort=30 velocity=1
- added joint panda_rjoint8: type fixed, parent panda_link7, child panda_link8, origin xyz=0 0 0.107 rpy=0 0 0, axis 0 0 0

File: myGym/envs/robots/franka_emika/panda_bullet/panda.urdf (robot description, URDF)
Before this commit: robot panda, 13 links, 12 joints
Links:
- removed link panda_grasptarget
- removed link panda_hand
- added link endeffector; visual sphere radius=0.01
- added link gripper; collision mesh filename=package://meshes/collision/hand.obj; visual mesh filename=package://meshes/visual/hand.obj
Joints:
- removed joint panda_finger_joint1
- removed joint panda_finger_joint2
- removed joint panda_grasptarget_hand
- removed joint panda_hand_joint
- removed joint panda_joint1
- removed joint panda_joint2
- removed joint panda_joint3
- removed joint panda_joint4
- removed joint panda_joint5
- removed joint panda_joint6
- removed joint panda_joint7
- removed joint panda_joint8
- added joint endeffector_joint: type fixed, parent gripper, child endeffector, origin xyz=0 0.0 0.1 rpy=0 0 0
- added joint gripper_joint: type fixed, parent panda_link8, child gripper, origin xyz=0 0 0.0 rpy=0 0 0
- added joint panda_finger_gjoint1: type prismatic, parent gripper, child panda_leftfinger, origin xyz=0 0 0.0584 rpy=0 0 0, axis 0 1 0, limit lower=0.0 upper=.07 effort=20 velocity=1
- added joint panda_finger_gjoint2: type prismatic, parent gripper, child panda_rightfinger, origin xyz=0 0 0.0584 rpy=0 0 0, axis 0 -1 0, limit lower=0.0 upper=.07 effort=20 velocity=1, mimic joint=panda_finger_gjoint1
- added joint panda_rjoint1: type revolute, parent panda_link0, child panda_link1, origin xyz=0 0 0.333 rpy=0 0 0, axis 0 0 1, limit lower=-2.9671 upper=2.9671 effort=87 velocity=2.1750
- added joint panda_rjoint2: type revolute, parent panda_link1, child panda_link2, origin xyz=0 0 0 rpy=-1.57079632679 0 0, axis 0 0 1, limit lower=-1.8326 upper=1.8326 effort=87 velocity=2.1750
- added joint panda_rjoint3: type revolute, parent panda_link2, child panda_link3, origin xyz=0 -0.316 0 rpy=1.57079632679 0 0, axis 0 0 1, limit lower=-2.9671 upper=2.9671 effort=87 velocity=2.1750
- added joint panda_rjoint4: type revolute, parent panda_link3, child panda_link4, origin xyz=0.0825 0 0 rpy=1.57079632679 0 0, axis 0 0 1, limit lower=-3.1416 upper=0.0 effort=87 velocity=2.1750
- added joint panda_rjoint5: type revolute, parent panda_link4, child panda_link5, origin xyz=-0.0825 0.384 0 rpy=-1.57079632679 0 0, axis 0 0 1, limit lower=-2.9671 upper=2.9671 effort=12 velocity=2.6100
- added joint panda_rjoint6: type revolute, parent panda_link5, child panda_link6, origin xyz=0 0 0 rpy=1.57079632679 0 0, axis 0 0 1, limit lower=-0.0873 upper=3.8223 effort=12 velocity=2.6100
- added joint panda_rjoint7: type revolute, parent panda_link6, child panda_link7, origin xyz=0.088 0 0 rpy=1.57079632679 0 0, axis 0 0 1, limit lower=-2.9671 upper=2.9671 effort=12 velocity=2.6100
- added joint panda_rjoint8: type fixed, parent panda_link7, child panda_link8, origin xyz=0 0 0.107 rpy=0 0 0, axis 0 0 0

File: myGym/envs/robots/franka_emika/panda_moveit/urdf/panda2.urdf (robot description, URDF)
Before this commit: robot panda, 12 links, 11 joints
Links:
- removed link end_effector
- added link endeffector; visual sphere radius=0.01
- added link panda_rightfinger; collision mesh filename=meshes/collision/finger.stl; visual mesh filename=meshes/visual/finger.dae
Joints:
- removed joint panda_finger_joint1
- removed joint panda_finger_joint2
- removed joint panda_hand_joint
- removed joint panda_joint1
- removed joint panda_joint2
- removed joint panda_joint3
- removed joint panda_joint4
- removed joint panda_joint5
- removed joint panda_joint6
- removed joint panda_joint7
- added joint endeffector_joint: type fixed, parent gripper, child endeffector, origin xyz=0 0.0 0.1 rpy=0 0 0
- added joint gripper_joint: type fixed, parent panda_link8, child gripper, origin xyz=0 0 0 rpy=0 0 -0.785398163397
- added joint panda_finger_gjoint1: type prismatic, parent gripper, child panda_leftfinger, origin xyz=0 0 0.0584 rpy=0 0 0, axis 0 1 0, limit lower=0.0 upper=0.04 effort=20 velocity=0.2
- added joint panda_finger_gjoint2: type prismatic, parent gripper, child panda_rightfinger, origin xyz=0 0 0.0584 rpy=0 0 0, axis 0 -1 0, limit lower=0.0 upper=0.04 effort=20 velocity=0.2, mimic joint=panda_finger_joint1
- added joint panda_rjoint1: type revolute, parent panda_link0, child panda_link1, origin xyz=0 0 0.333 rpy=0 0 0, axis 0 0 1, limit lower=-2.9671 upper=2.9671 effort=87 velocity=2.3925
- added joint panda_rjoint2: type revolute, parent panda_link1, child panda_link2, origin xyz=0 0 0 rpy=-1.57079632679 0 0, axis 0 0 1, limit lower=-1.8326 upper=1.8326 effort=87 velocity=2.3925
- added joint panda_rjoint3: type revolute, parent panda_link2, child panda_link3, origin xyz=0 -0.316 0 rpy=1.57079632679 0 0, axis 0 0 1, limit lower=-2.9671 upper=2.9671 effort=87 velocity=2.3925
- added joint panda_rjoint4: type revolute, parent panda_link3, child panda_link4, origin xyz=0.0825 0 0 rpy=1.57079632679 0 0, axis 0 0 1, limit lower=-3.1416 upper=0.0873 effort=87 velocity=2.3925
- added joint panda_rjoint5: type revolute, parent panda_link4, child panda_link5, origin xyz=-0.0825 0.384 0 rpy=-1.57079632679 0 0, axis 0 0 1, limit lower=-2.9671 upper=2.9671 effort=12 velocity=2.8710
- added joint panda_rjoint6: type revolute, parent panda_link5, child panda_link6, origin xyz=0 0 0 rpy=1.57079632679 0 0, axis 0 0 1, limit lower=-0.0873 upper=3.8223 effort=12 velocity=2.8710
- added joint panda_rjoint7: type revolute, parent panda_link6, child panda_link7, origin xyz=0.088 0 0 rpy=1.57079632679 0 0, axis 0 0 1, limit lower=-2.9671 upper=2.9671 effort=12 velocity=2.8710

File: myGym/envs/robots/jaco_arm/jaco/urdf/jaco_robotiq.urdf (robot description, URDF)
Before this commit: robot j2s7s300, 19 links, 18 joints
Links:
- removed link end_effector
- added link endeffector; visual sphere radius=0.01
- added link robotiq_85_left_finger_tip_link, mass 0.019555; collision mesh filename=robotiq/collision/robotiq_85_finger_tip_link.stl; visual mesh filename=robotiq/collision/robotiq_85_finger_tip_link.stl
Joints:
- removed joint j2s7s300_joint_1
- removed joint j2s7s300_joint_2
- removed joint j2s7s300_joint_3
- removed joint j2s7s300_joint_4
- removed joint j2s7s300_joint_5
- removed joint j2s7s300_joint_6
- removed joint j2s7s300_joint_7
- removed joint robotiq_85_left_finger_joint
- removed joint robotiq_85_left_finger_tip_joint
- removed joint robotiq_85_left_inner_knuckle_joint
- removed joint robotiq_85_left_knuckle_joint
- removed joint robotiq_85_right_finger_joint
- removed joint robotiq_85_right_finger_tip_joint
- removed joint robotiq_85_right_inner_knuckle_joint
- removed joint robotiq_85_right_knuckle_joint
- added joint endeffector_joint: type fixed, parent gripper, child endeffector, origin xyz=0 0.0 -0.23 rpy=0 0 0
- added joint j2s7s300_rjoint_1: type continuous, parent j2s7s300_link_base, child j2s7s300_link_1, origin xyz=0 0 0.15675 rpy=0 3.14159265359 0, axis 0 0 1, limit lower=-6.28318530718 upper=6.28318530718 effort=40 velocity=1.0
- added joint j2s7s300_rjoint_2: type revolute, parent j2s7s300_link_1, child j2s7s300_link_2, origin xyz=0 0.0016 -0.11875 rpy=-1.57079632679 0 3.14159265359, axis 0 0 1, limit lower=0.523598775598 upper=5.75958653158 effort=40 velocity=1
- added joint j2s7s300_rjoint_3: type continuous, parent j2s7s300_link_2, child j2s7s300_link_3, origin xyz=0 -0.205 0 rpy=-1.57079632679 0 0, axis 0 0 1, limit lower=-6.28318530718 upper=6.28318530718 effort=40 velocity=1
- added joint j2s7s300_rjoint_4: type revolute, parent j2s7s300_link_3, child j2s7s300_link_4, origin xyz=0 0 -0.205 rpy=1.57079632679 0 3.14159265359, axis 0 0 1, limit lower=0.523598775598 upper=5.75958653158 effort=40 velocity=1
- added joint j2s7s300_rjoint_5: type continuous, parent j2s7s300_link_4, child j2s7s300_link_5, origin xyz=0 0.2073 -0.0114 rpy=-1.57079632679 0 3.14159265359, axis 0 0 1, limit lower=-6.28318530718 upper=6.28318530718 effort=40 velocity=1
- added joint j2s7s300_rjoint_6: type revolute, parent j2s7s300_link_5, child j2s7s300_link_6, origin xyz=0 0 -0.10375 rpy=1.57079632679 0 3.14159265359, axis 0 0 1, limit lower=0.523598775598 upper=5.75958653158 effort=40 velocity=1
- added joint j2s7s300_rjoint_7: type continuous, parent j2s7s300_link_6, child gripper, origin xyz=0 0.06075 0 rpy=1.5707 0 0, axis 0 0 1, limit lower=-3.14159265359 upper=3.14159265359 effort=40 velocity=0.785
- added joint robotiq_85_left_finger_gjoint: type fixed, parent robotiq_85_left_knuckle_link, child robotiq_85_left_finger_link, origin xyz=-0.00408552455 -0.03148604435 0.0 rpy=0 0 0, limit lower=-3.14 upper=3.14 velocity=1.0
- added joint robotiq_85_left_finger_tip_gjoint: type revolute, parent robotiq_85_left_inner_knuckle_link, child robotiq_85_left_finger_tip_link, origin xyz=0.04303959807 -0.03759940821 0.0 rpy=0.0 0.0 0.0, axis 0 0 1, limit lower=-0.8757 upper=0.0 velocity=1.0
- added joint robotiq_85_left_inner_knuckle_gjoint: type revolute, parent robotiq_85_base_link, child robotiq_85_left_inner_knuckle_link, origin xyz=0.06142 0.0127 0 rpy=3.14159 0.0 0.0, axis 0 0 1, limit lower=0.0 upper=0.8757 velocity=1.0
- added joint robotiq_85_left_knuckle_gjoint: type revolute, parent robotiq_85_base_link, child robotiq_85_left_knuckle_link, origin xyz=0.05490451627 0.03060114443 0.0 rpy=3.14159 0.0 0.0, axis 0 0 1, limit lower=0.0 upper=0.81 velocity=1.0
- added joint robotiq_85_right_finger_gjoint: type fixed, parent robotiq_85_right_knuckle_link, child robotiq_85_right_finger_link, origin xyz=-0.00408552455 -0.03148604435 0.0 rpy=0 0 0, limit lower=-3.14 upper=3.14 velocity=1.0
- added joint robotiq_85_right_finger_tip_gjoint: type revolute, parent robotiq_85_right_inner_knuckle_link, child robotiq_85_right_finger_tip_link, origin xyz=0.04303959807 -0.03759940821  0.0 rpy=0.0 0.0 0.0, axis 0 0 1, limit lower=-0.8757 upper=0.0 velocity=1.0
- added joint robotiq_85_right_inner_knuckle_gjoint: type revolute, parent robotiq_85_base_link, child robotiq_85_right_inner_knuckle_link, origin xyz=0.06142 -0.0127 0 rpy=0 0 0, axis 0 0 1, limit lower=0.0 upper=0.8757 velocity=1.0
- added joint robotiq_85_right_knuckle_gjoint: type revolute, parent robotiq_85_base_link, child robotiq_85_right_knuckle_link, origin xyz=0.05490451627 -0.03060114443 0.0 rpy=0.0 0.0 0.0, axis 0 0 1, limit lower=0.0 upper=0.81 velocity=1.0

File: myGym/envs/robots/jaco_arm/jaco/urdf/jaco_robotiq_fixed.urdf (robot description, URDF)
Before this commit: robot j2s7s300, 19 links, 18 joints
Links:
- removed link end_effector
- added link endeffector; visual sphere radius=0.01
- added link robotiq_85_left_finger_tip_link, mass 0.019555; collision mesh filename=robotiq/collision/robotiq_85_finger_tip_link.stl; visual mesh filename=robotiq/collision/robotiq_85_finger_tip_link.stl
Joints:
- removed joint j2s7s300_joint_1
- removed joint j2s7s300_joint_2
- removed joint j2s7s300_joint_3
- removed joint j2s7s300_joint_4
- removed joint j2s7s300_joint_5
- removed joint j2s7s300_joint_6
- removed joint j2s7s300_joint_7
- removed joint robotiq_85_left_finger_joint
- removed joint robotiq_85_left_knuckle_joint
- removed joint robotiq_85_right_finger_joint
- removed joint robotiq_85_right_knuckle_joint
- added joint endeffector_joint: type fixed, parent gripper, child endeffector, origin xyz=0 0.0 -0.23 rpy=0 0 0
- added joint j2s7s300_rjoint_1: type continuous, parent j2s7s300_link_base, child j2s7s300_link_1, origin xyz=0 0 0.15675 rpy=0 3.14159265359 0, axis 0 0 1, limit lower=-6.28318530718 upper=6.28318530718 effort=40 velocity=1.0
- added joint j2s7s300_rjoint_2: type revolute, parent j2s7s300_link_1, child j2s7s300_link_2, origin xyz=0 0.0016 -0.11875 rpy=-1.57079632679 0 3.14159265359, axis 0 0 1, limit lower=0.523598775598 upper=5.75958653158 effort=40 velocity=1
- added joint j2s7s300_rjoint_3: type continuous, parent j2s7s300_link_2, child j2s7s300_link_3, origin xyz=0 -0.205 0 rpy=-1.57079632679 0 0, axis 0 0 1, limit lower=-6.28318530718 upper=6.28318530718 effort=40 velocity=1
- added joint j2s7s300_rjoint_4: type revolute, parent j2s7s300_link_3, child j2s7s300_link_4, origin xyz=0 0 -0.205 rpy=1.57079632679 0 3.14159265359, axis 0 0 1, limit lower=0.523598775598 upper=5.75958653158 effort=40 velocity=1
- added joint j2s7s300_rjoint_5: type continuous, parent j2s7s300_link_4, child j2s7s300_link_5, origin xyz=0 0.2073 -0.0114 rpy=-1.57079632679 0 3.14159265359, axis 0 0 1, limit lower=-6.28318530718 upper=6.28318530718 effort=40 velocity=1
- added joint j2s7s300_rjoint_6: type revolute, parent j2s7s300_link_5, child j2s7s300_link_6, origin xyz=0 0 -0.10375 rpy=1.57079632679 0 3.14159265359, axis 0 0 1, limit lower=0.523598775598 upper=5.75958653158 effort=40 velocity=1
- added joint j2s7s300_rjoint_7: type continuous, parent j2s7s300_link_6, child gripper, origin xyz=0 0.06075 0 rpy=1.5707 0 0, axis 0 0 1, limit lower=-3.14159265359 upper=3.14159265359 effort=40 velocity=1
- added joint robotiq_85_left_finger_gjoint: type fixed, parent robotiq_85_left_knuckle_link, child robotiq_85_left_finger_link, origin xyz=-0.00408552455 -0.03148604435 0.0 rpy=0 0 0, limit lower=-3.14 upper=3.14 velocity=1.0
- added joint robotiq_85_left_knuckle_gjoint: type revolute, parent robotiq_85_base_link, child robotiq_85_left_knuckle_link, origin xyz=0.05490451627 0.03060114443 0.0 rpy=3.14159 0.0 0.0, axis 0 0 1, limit lower=0.0 upper=0.81 velocity=1.0
- added joint robotiq_85_right_finger_gjoint: type fixed, parent robotiq_85_right_knuckle_link, child robotiq_85_right_finger_link, origin xyz=-0.00408552455 -0.03148604435 0.0 rpy=0 0 0, limit lower=-3.14 upper=3.14 velocity=1.0
- added joint robotiq_85_right_knuckle_gjoint: type revolute, parent robotiq_85_base_link, child robotiq_85_right_knuckle_link, origin xyz=0.05490451627 -0.03060114443 0.0 rpy=0.0 0.0 0.0, axis 0 0 1, limit lower=0.0 upper=0.81 velocity=1.0
- joint robotiq_85_left_finger_tip_joint: child end_effector -> robotiq_85_left_finger_tip_link

File: myGym/envs/robots/kuka_gripper/kuka_gripper.urdf (robot description, URDF)
Before this commit: robot kuka_gripper, 17 links, 16 joints
Links:
- removed link base
- added link endeffector; visual sphere radius=0.01
- added link gripper, mass 2.0; collision mesh filename=/meshes/base.obj; visual mesh filename=/meshes/base.obj
Joints:
- removed joint base_to_finger00_joint
- removed joint base_to_finger10_joint
- removed joint finger00_to_finger01_joint
- removed joint finger10_to_finger11_joint
- removed joint kuka_to_gripper_joint
- removed joint lbr_iiwa_joint_1
- removed joint lbr_iiwa_joint_2
- removed joint lbr_iiwa_joint_3
- removed joint lbr_iiwa_joint_4
- removed joint lbr_iiwa_joint_5
- removed joint lbr_iiwa_joint_6
- removed joint lbr_iiwa_joint_7
- added joint base_to_finger00_gjoint: type revolute, parent gripper, child finger_00, origin xyz=0.023510971786833857 0 0 rpy=0 0 0, axis 0 1 0, limit lower=0 upper=1.5707963267948966 effort=30 velocity=1
- added joint base_to_finger10_gjoint: type revolute, parent gripper, child finger_10, origin xyz=-0.023510971786833857 0 0 rpy=0 0 3.141592653589793, axis 0 1 0, limit lower=0 upper=1.5707963267948966 effort=30 velocity=1
- added joint endeffector_joint: type fixed, parent gripper, child endeffector, origin xyz=0 0.0 0.1 rpy=0 0 0
- added joint finger00_to_finger01_gjoint: type revolute, parent finger_00, child finger_01, origin xyz=0 0  0.0768025078369906 rpy=0 0 0, axis 0 1 0, limit lower=0 upper=-1.5707963267948966 effort=30 velocity=1
- added joint finger10_to_finger11_gjoint: type revolute, parent finger_10, child finger_11, origin xyz=0 0 0.0768025078369906 rpy=0 0 0, axis 0 1 0, limit lower=0 upper=-1.5707963267948966 effort=30 velocity=1
- added joint gripper_joint: type fixed, parent lbr_iiwa_link_7, child gripper, origin xyz=0 0 0.05 rpy=0 0 0
- added joint lbr_iiwa_rjoint_1: type revolute, parent lbr_iiwa_link_0, child lbr_iiwa_link_1, origin xyz=0 0 0.1575 rpy=0 0 0, axis 0 0 1, limit lower=-2.96705972839 upper=2.96705972839 effort=30 velocity=1
- added joint lbr_iiwa_rjoint_2: type revolute, parent lbr_iiwa_link_1, child lbr_iiwa_link_2, origin xyz=0 0 0.2025 rpy=1.57079632679   0 3.14159265359, axis 0 0 1, limit lower=-2.09439510239 upper=2.09439510239 effort=30 velocity=1
- added joint lbr_iiwa_rjoint_3: type revolute, parent lbr_iiwa_link_2, child lbr_iiwa_link_3, origin xyz=0 0.2045 0 rpy=1.57079632679 0 3.14159265359, axis 0 0 1, limit lower=-2.96705972839 upper=2.96705972839 effort=30 velocity=1
- added joint lbr_iiwa_rjoint_4: type revolute, parent lbr_iiwa_link_3, child lbr_iiwa_link_4, origin xyz=0 0 0.2155 rpy=1.57079632679 0 0, axis 0 0 1, limit lower=-2.09439510239 upper=2.09439510239 effort=30 velocity=1
- added joint lbr_iiwa_rjoint_5: type revolute, parent lbr_iiwa_link_4, child lbr_iiwa_link_5, origin xyz=0 0.1845 0 rpy=-1.57079632679 3.14159265359 0, axis 0 0 1, limit lower=-2.96705972839 upper=2.96705972839 effort=30 velocity=1
- added joint lbr_iiwa_rjoint_6: type revolute, parent lbr_iiwa_link_5, child lbr_iiwa_link_6, origin xyz=0 0 0.2155 rpy=1.57079632679 0 0, axis 0 0 1, limit lower=-2.09439510239 upper=2.09439510239 effort=30 velocity=1
- added joint lbr_iiwa_rjoint_7: type revolute, parent lbr_iiwa_link_6, child lbr_iiwa_link_7, origin xyz=0 0.081 0 rpy=-1.57079632679 3.14159265359 0, axis 0 0 1, limit lower=-3.05432619099 upper=3.05432619099 effort=30 velocity=1

File: myGym/envs/robots/kuka_magnetic_gripper_sdf/kuka_magnetic.urdf (robot description, URDF)
Before this commit: robot lbr_iiwa, 12 links, 11 joints
Links:
- removed link end_effector
- added link endeffector; visual sphere radius=0.01
- added link sensor, mass 0.2; collision mesh filename=meshes/sensor_old.stl scale=0.001 0.001 0.001; visual mesh filename=meshes/sensor_old.stl scale=0.001 0.001 0.001
Joints:
- removed joint gripper_to_arm
- removed joint lbr_iiwa_joint_1
- removed joint lbr_iiwa_joint_2
- removed joint lbr_iiwa_joint_3
- removed joint lbr_iiwa_joint_4
- removed joint lbr_iiwa_joint_5
- removed joint lbr_iiwa_joint_6
- removed joint lbr_iiwa_joint_7
- added joint endeffector_joint: type fixed, parent gripper, child endeffector, origin xyz=0 0.0 0.15 rpy=0 0 0
- added joint gripper_joint: type fixed, parent lbr_iiwa_link_7, child gripper
- added joint lbr_iiwa_rjoint_1: type revolute, parent lbr_iiwa_link_0, child lbr_iiwa_link_1, origin xyz=0 0 0.1575 rpy=0 0 0, axis 0 0 1, limit lower=-2.96705972839 upper=2.96705972839 effort=30 velocity=1
- added joint lbr_iiwa_rjoint_2: type revolute, parent lbr_iiwa_link_1, child lbr_iiwa_link_2, origin xyz=0 0 0.2025 rpy=1.57079632679   0 3.14159265359, axis 0 0 1, limit lower=-2.09439510239 upper=2.09439510239 effort=30 velocity=1
- added joint lbr_iiwa_rjoint_3: type revolute, parent lbr_iiwa_link_2, child lbr_iiwa_link_3, origin xyz=0 0.2045 0 rpy=1.57079632679 0 3.14159265359, axis 0 0 1, limit lower=-2.96705972839 upper=2.96705972839 effort=30 velocity=1
- added joint lbr_iiwa_rjoint_4: type revolute, parent lbr_iiwa_link_3, child lbr_iiwa_link_4, origin xyz=0 0 0.2155 rpy=1.57079632679 0 0, axis 0 0 1, limit lower=-2.09439510239 upper=2.09439510239 effort=30 velocity=1
- added joint lbr_iiwa_rjoint_5: type revolute, parent lbr_iiwa_link_4, child lbr_iiwa_link_5, origin xyz=0 0.1845 0 rpy=-1.57079632679 3.14159265359 0, axis 0 0 1, limit lower=-2.96705972839 upper=2.96705972839 effort=30 velocity=1
- added joint lbr_iiwa_rjoint_6: type revolute, parent lbr_iiwa_link_5, child lbr_iiwa_link_6, origin xyz=0 0 0.2155 rpy=1.57079632679 0 0, axis 0 0 1, limit lower=-2.09439510239 upper=2.09439510239 effort=30 velocity=1
- added joint lbr_iiwa_rjoint_7: type revolute, parent lbr_iiwa_link_6, child lbr_iiwa_link_7, origin xyz=0 0.081 0 rpy=-1.57079632679 3.14159265359 0, axis 0 0 1, limit lower=-3.05432619099 upper=3.05432619099 effort=30 velocity=1
- joint sensor_joint: child end_effector -> sensor
