Commit message: robot control UPDATE - gripper and end effector universalization, robot.py rewritten, urdf changed (rjoint and gjoints), gripper idependetly controlled, gripper=last IK joint, end effector=graspable point

File: myGym/envs/robots/pollen/reachy/urdf/reachy.urdf (robot description, URDF)
Before this commit: robot Reachy, 11 links, 10 joints
Links:
- removed link end_effector
- added link ball, mass 0.090; collision mesh filename=package://reachy/meshes/ball-tip-respondable.stl; visual mesh filename=package://reachy/meshes/ball-tip-visual.stl
- added link endeffector; visual sphere radius=0.01
Joints:
- removed joint arm_yaw
- removed joint elbow_pitch
- removed joint forearm_yaw
- removed joint shoulder_pitch
- removed joint shoulder_roll
- removed joint wrist_pitch
- removed joint wrist_roll
- added joint arm_yaw_rjoint: type revolute, parent shoulder_to_arm, child upper_arm, origin xyz=0 0 0 rpy=0 0 0, axis 0 0 1, limit lower=-1.5708 upper=1.5708 effort=30 velocity=1
- added joint elbow_pitch_rjoint: type revolute, parent upper_arm, child forearm, origin xyz=0 0 -0.30745 rpy=0 0 0, axis 0 1 0, limit lower=-2.18166 upper=0 effort=30 velocity=1
- added joint endeffector_joint: type fixed, parent gripper, child endeffector, origin xyz=0 0.0 -0.13 rpy=0 0 0
- added joint forearm_yaw_rjoint: type revolute, parent forearm, child wrist, origin xyz=0 0 0 rpy=0 0 0, axis 0 0 1, limit lower=-2.61799 upper=2.61799 effort=30 velocity=1
- added joint shoulder_pitch_rjoint: type revolute, parent base, child shoulder, origin xyz=0 -0.14 0 rpy=0 -1.5 0, axis 0 1 0, limit lower=-1.5708 upper=3.14159 effort=30 velocity=1
- added joint shoulder_roll_rjoint: type revolute, parent shoulder, child shoulder_to_arm, origin xyz=0 0 0 rpy=0 0 0, axis 1 0 0, limit lower=-3.14159 upper=0.174533 effort=30 velocity=1
- added joint wrist_pitch_rjoint: type revolute, parent wrist, child gripper, origin xyz=0 0 -0.22425 rpy=0 0 0, axis 0 1 0, limit lower=-1.22173 upper=1.22173 effort=30 velocity=1
- added joint wrist_roll_rjoint: type revolute, parent gripper, child ball, origin xyz=0 0 -0.03243 rpy=0 0 0, axis 1 0 0, limit lower=-1.0472 upper=1.0472 effort=30 velocity=1

Commit message: robot and config update

File: myGym/envs/robots/franka_emika/panda/urdf/panda1.urdf (robot description, URDF)
Before this commit: robot panda, 14 links, 13 joints
Links:
- link panda_leftfinger: geometry collision mesh filename=meshes/collision/finger1.obj; visual mesh filename=meshes/collision/finger1.obj
- link panda_rightfinger: geometry collision mesh filename=meshes/collision/finger1.obj; visual mesh filename=meshes/collision/finger1.obj

Commit message: ROBOT REPOSITIONING - WIP

File: myGym/envs/robots/franka_emika/panda/urdf/panda1.urdf (robot description, URDF)
Before this commit: robot panda, 14 links, 13 joints
Joints:
- joint endeffector_joint: origin xyz=0.0 0.0 0.12 rpy=3.14 0 0 -> xyz=0.0 0.0 0.12 rpy=3.14 0 1.57

File: myGym/envs/robots/franka_emika/panda_bullet/panda.urdf (robot description, URDF)
Before this commit: robot panda, 13 links, 12 joints
Joints:
- joint endeffector_joint: origin xyz=0.0 0.0 0.12 rpy=3.14 0 0 -> xyz=0.0 0.0 0.12 rpy=3.14 0 1.57

File: myGym/envs/robots/franka_emika/panda_moveit/urdf/panda2.urdf (robot description, URDF)
Before this commit: robot panda, 13 links, 12 joints
Joints:
- joint endeffector_joint: origin xyz=0.0 0.0 0.12 rpy=3.14 0 0 -> xyz=0.0 0.0 0.12 rpy=3.14 0 1.57

File: myGym/envs/robots/jaco_arm/jaco/urdf/jaco_robotiq_fixed.urdf (robot description, URDF)
Before this commit: robot j2s7s300, 20 links, 19 joints
Links:
- link endeffector: mass None -> 0.0000332; geometry visual cylinder length=0.05 radius=0.002
Joints:
- joint endeffector_joint: origin xyz=0 0.0 -0.23 rpy=0 0 0 -> xyz=0.0 0.0 -0.23 rpy=0 0 1.57

File: myGym/envs/robots/kuka_gripper/kuka_gripper.urdf (robot description, URDF)
Before this commit: robot kuka_gripper, 18 links, 17 joints
Joints:
- joint endeffector_joint: origin xyz=0.0 0.0 0.12 rpy=3.14 0 0 -> xyz=0.0 0.0 0.12 rpy=3.14 0 -1.57

File: myGym/envs/robots/kuka_magnetic_gripper_sdf/kuka_magnetic.urdf (robot description, URDF)
Before this commit: robot lbr_iiwa, 13 links, 12 joints
Links:
- link endeffector: mass 0 -> 0.0000332; geometry visual cylinder length=0.05 radius=0.002
Joints:
- joint endeffector_joint: origin xyz=0 0.0 0.15 rpy=0 0 0 -> xyz=0.0 0.0 0.12 rpy=3.14 0 0

File: myGym/envs/robots/kuka_magnetic_gripper_sdf/kuka_push.urdf (robot description, URDF)
Before this commit: robot lbr_iiwa, 13 links, 12 joints
Links:
- link endeffector: mass None -> 0.0000332; geometry visual cylinder length=0.05 radius=0.002
Joints:
- joint endeffector_joint: origin xyz=0 0.0 0.10 rpy=0 0 0 -> xyz=0.0 0.0 0.12 rpy=3.14 0 0

File: myGym/envs/robots/nico/nico_grasper.urdf (robot description, URDF)
Before this commit: robot nico_upper_rh6d, 29 links, 28 joints
Joints:
- joint endeffector_joint: origin xyz=0.03 0.0 -0.05 rpy=3.14 1.57 0 -> xyz=0.03 0.0 -0.05 rpy=1.57 0 1.57 

Commit message: robot end effector visualization update

File: myGym/envs/robots/franka_emika/panda/urdf/panda1.urdf (robot description, URDF)
Before this commit: robot panda, 14 links, 13 joints
Links:
- added link ee_x_axis; visual cylinder length=0.06 radius=0.002
- added link ee_y_axis; visual cylinder length=0.06 radius=0.002
- added link ee_z_axis; visual cylinder length=0.06 radius=0.002
- link endeffector: mass 0.0000332 -> None; geometry visual sphere radius=0.005
Joints:
- added joint ee_x_axis_joint: type fixed, parent gripper, child ee_x_axis, origin xyz=0.0 0.0 0.1 rpy=0 0 0
- added joint ee_y_axis_joint: type fixed, parent gripper, child ee_y_axis, origin xyz=0.0 0.0 0.1 rpy=0 0 0
- added joint ee_z_axis_joint: type fixed, parent gripper, child ee_z_axis, origin xyz=0.0 0.0 0.1 rpy=0 0 0
- joint endeffector_joint: origin xyz=0.0 0.0 0.12 rpy=3.14 0 1.57 -> xyz=0.0 0.0 0.1 rpy=0 3.14 0

File: myGym/envs/robots/franka_emika/panda/urdf/panda_cgripper.urdf (robot description, URDF)
Before this commit: robot panda, 22 links, 21 joints
Links:
- added link ee_x_axis; visual cylinder length=0.06 radius=0.002
- added link ee_y_axis; visual cylinder length=0.06 radius=0.002
- added link ee_z_axis; visual cylinder length=0.06 radius=0.002
- link endeffector: mass 0.0000332 -> None; geometry visual sphere radius=0.005
Joints:
- added joint ee_x_axis_joint: type fixed, parent gripper, child ee_x_axis, origin xyz=0.0 0.0 0.15 rpy=0 0 0
- added joint ee_y_axis_joint: type fixed, parent gripper, child ee_y_axis, origin xyz=0.0 0.0 0.15 rpy=0 0 0
- added joint ee_z_axis_joint: type fixed, parent gripper, child ee_z_axis, origin xyz=0.0 0.0 0.15 rpy=0 0 0
- joint endeffector_joint: origin xyz=0.0 0.0 0.12 rpy=3.14 0 0 -> xyz=0.0 0.0 0.15 rpy=0 3.14 0

File: myGym/envs/robots/franka_emika/panda_bullet/panda.urdf (robot description, URDF)
Before this commit: robot panda, 13 links, 12 joints
Links:
- added link ee_x_axis; visual cylinder length=0.06 radius=0.002
- added link ee_y_axis; visual cylinder length=0.06 radius=0.002
- added link ee_z_axis; visual cylinder length=0.06 radius=0.002
- link endeffector: mass 0.0000332 -> None; geometry visual sphere radius=0.005
Joints:
- added joint ee_x_axis_joint: type fixed, parent gripper, child ee_x_axis, origin xyz=0.0 0.0 0.1 rpy=0 0 0
- added joint ee_y_axis_joint: type fixed, parent gripper, child ee_y_axis, origin xyz=0.0 0.0 0.1 rpy=0 0 0
- added joint ee_z_axis_joint: type fixed, parent gripper, child ee_z_axis, origin xyz=0.0 0.0 0.1 rpy=0 0 0
- joint endeffector_joint: origin xyz=0.0 0.0 0.12 rpy=3.14 0 1.57 -> xyz=0.0 0.0 0.1 rpy=0 3.14 0

File: myGym/envs/robots/franka_emika/panda_moveit/urdf/panda2.urdf (robot description, URDF)
Before this commit: robot panda, 13 links, 12 joints
Links:
- added link ee_x_axis; visual cylinder length=0.06 radius=0.002
- added link ee_y_axis; visual cylinder length=0.06 radius=0.002
- added link ee_z_axis; visual cylinder length=0.06 radius=0.002
- link endeffector: mass 0.0000332 -> None; geometry visual sphere radius=0.005
Joints:
- added joint ee_x_axis_joint: type fixed, parent gripper, child ee_x_axis, origin xyz=0.0 0.0 0.1 rpy=0 0 0
- added joint ee_y_axis_joint: type fixed, parent gripper, child ee_y_axis, origin xyz=0.0 0.0 0.1 rpy=0 0 0
- added joint ee_z_axis_joint: type fixed, parent gripper, child ee_z_axis, origin xyz=0.0 0.0 0.1 rpy=0 0 0
- joint endeffector_joint: origin xyz=0.0 0.0 0.12 rpy=3.14 0 1.57 -> xyz=0.0 0.0 0.1 rpy=0 3.14 0

File: myGym/envs/robots/kuka_gripper/kuka_gripper.urdf (robot description, URDF)
Before this commit: robot kuka_gripper, 18 links, 17 joints
Links:
- added link ee_x_axis; visual cylinder length=0.06 radius=0.002
- added link ee_y_axis; visual cylinder length=0.06 radius=0.002
- added link ee_z_axis; visual cylinder length=0.06 radius=0.002
- link endeffector: mass 0.0000332 -> None; geometry visual sphere radius=0.005
Joints:
- added joint ee_x_axis_joint: type fixed, parent gripper, child ee_x_axis, origin xyz=0.0 0.0 0.1 rpy=0 0 0
- added joint ee_y_axis_joint: type fixed, parent gripper, child ee_y_axis, origin xyz=0.0 0.0 0.1 rpy=0 0 0
- added joint ee_z_axis_joint: type fixed, parent gripper, child ee_z_axis, origin xyz=0.0 0.0 0.1 rpy=0 0 0
- joint endeffector_joint: origin xyz=0.0 0.0 0.12 rpy=3.14 0 -1.57 -> xyz=0.0 0.0 0.1 rpy=0 3.14 0

File: myGym/envs/robots/kuka_magnetic_gripper_sdf/kuka_magnetic.urdf (robot description, URDF)
Before this commit: robot lbr_iiwa, 13 links, 12 joints
Links:
- added link ee_x_axis; visual cylinder length=0.06 radius=0.002
- added link ee_y_axis; visual cylinder length=0.06 radius=0.002
- added link ee_z_axis; visual cylinder length=0.06 radius=0.002
- link endeffector: mass 0.0000332 -> None; geometry visual sphere radius=0.005
Joints:
- added joint ee_x_axis_joint: type fixed, parent gripper, child ee_x_axis, origin xyz=0.0 0.0 0.15 rpy=0 0 0
- added joint ee_y_axis_joint: type fixed, parent gripper, child ee_y_axis, origin xyz=0.0 0.0 0.15 rpy=0 0 0
- added joint ee_z_axis_joint: type fixed, parent gripper, child ee_z_axis, origin xyz=0.0 0.0 0.15 rpy=0 0 0
- joint endeffector_joint: origin xyz=0.0 0.0 0.12 rpy=3.14 0 0 -> xyz=0.0 0.0 0.15 rpy=0 3.14 0

File: myGym/envs/robots/kuka_magnetic_gripper_sdf/kuka_push.urdf (robot description, URDF)
Before this commit: robot lbr_iiwa, 13 links, 12 joints
Links:
- added link ee_x_axis; visual cylinder length=0.06 radius=0.002
- added link ee_y_axis; visual cylinder length=0.06 radius=0.002
- added link ee_z_axis; visual cylinder length=0.06 radius=0.002
- link endeffector: mass 0.0000332 -> None; geometry visual sphere radius=0.005
Joints:
- added joint ee_x_axis_joint: type fixed, parent gripper, child ee_x_axis, origin xyz=0.0 0.0 0.1 rpy=0 0 0
- added joint ee_y_axis_joint: type fixed, parent gripper, child ee_y_axis, origin xyz=0.0 0.0 0.1 rpy=0 0 0
- added joint ee_z_axis_joint: type fixed, parent gripper, child ee_z_axis, origin xyz=0.0 0.0 0.1 rpy=0 0 0
- joint endeffector_joint: origin xyz=0.0 0.0 0.12 rpy=3.14 0 0 -> xyz=0.0 0.0 0.1 rpy=0 3.14 0

File: myGym/envs/robots/nico/nico_grasper.urdf (robot description, URDF)
Before this commit: robot nico_upper_rh6d, 29 links, 28 joints
Links:
- added link ee_x_axis; visual cylinder length=0.06 radius=0.002
- added link ee_y_axis; visual cylinder length=0.06 radius=0.002
- added link ee_z_axis; visual cylinder length=0.06 radius=0.002
- link endeffector: mass 0.0000332 -> None; geometry visual sphere radius=0.005
Joints:
- added joint ee_x_axis_joint: type fixed, parent gripper, child ee_x_axis, origin xyz=0.03 0.0 -0.05 rpy=0 1.57 0
- added joint ee_y_axis_joint: type fixed, parent gripper, child ee_y_axis, origin xyz=0.03 0.0 -0.05 rpy=0 1.57 0
- added joint ee_z_axis_joint: type fixed, parent gripper, child ee_z_axis, origin xyz=0.03 0.0 -0.05 rpy=0 1.57 0

File: myGym/envs/robots/pollen/reachy/urdf/leachy.urdf (robot description, URDF)
Before this commit: robot Leachy_w_hand, 11 links, 10 joints
Links:
- added link ee_x_axis; visual cylinder length=0.06 radius=0.002
- added link ee_y_axis; visual cylinder length=0.06 radius=0.002
- added link ee_z_axis; visual cylinder length=0.06 radius=0.002
- link endeffector: mass 0.0000332 -> None; geometry visual sphere radius=0.005
Joints:
- added joint ee_x_axis_joint: type fixed, parent gripper, child ee_x_axis, origin xyz=0.0 -0.05 -0.12 rpy=-1.57 0 3.14
- added joint ee_y_axis_joint: type fixed, parent gripper, child ee_y_axis, origin xyz=0.0 -0.05 -0.12 rpy=-1.57 0 3.14
- added joint ee_z_axis_joint: type fixed, parent gripper, child ee_z_axis, origin xyz=0.0 -0.05 -0.12 rpy=-1.57 0 3.14
- joint endeffector_joint: origin xyz=0.0 -0.05 -0.12 rpy=-1.57 0 0 -> xyz=0.0 -0.05 -0.12 rpy=0 1.57 0
