Commit message: robot parameters update + visualization of sampling space

File: myGym/envs/robots/pollen/reachy/urdf/reachy_and_leachy.urdf (robot description, URDF)
Before this commit: robot Leachy_w_hand, 17 links, 16 joints
Joints:
- joint arm_yaw: limit lower=-1.5708 upper=1.5708 -> lower=-1.5708 upper=1.5708 effort=30 velocity=1
- joint elbow_pitch: limit lower=-2.18166 upper=0 -> lower=-2.18166 upper=0 effort=30 velocity=1
- joint forearm_yaw: limit lower=-2.61799 upper=2.61799 -> lower=-2.61799 upper=2.61799 effort=30 velocity=1
- joint head_pitch: limit lower=-3.14159 upper=0.174533 -> lower=-3.14159 upper=0.174533 effort=30 velocity=1
- joint head_yaw: limit lower=-1.5708 upper=3.14159 -> lower=-1.5708 upper=3.14159 effort=30 velocity=1
- joint l_arm_yaw: limit lower=-1.5708 upper=1.5708 -> lower=-1.5708 upper=1.5708 effort=30 velocity=1
- joint l_elbow_pitch: limit lower=-2.18166 upper=0 -> lower=-2.18166 upper=0 effort=30 velocity=1
- joint l_forearm_yaw: limit lower=-2.61799 upper=2.61799 -> lower=-2.61799 upper=2.61799 effort=30 velocity=1
- joint l_shoulder_pitch: limit lower=-1.5708 upper=3.14159 -> lower=-1.5708 upper=3.14159 effort=30 velocity=1
- joint l_shoulder_roll: limit lower=-0.174533 upper=3.14159 -> lower=-0.174533 upper=3.14159 effort=30 velocity=1
- joint l_wrist_pitch: limit lower=-1.22173 upper=1.22173 -> lower=-1.22173 upper=1.22173 effort=30 velocity=1
- joint shoulder_pitch: limit lower=-1.5708 upper=3.14159 -> lower=-1.5708 upper=3.14159 effort=30 velocity=1
- joint shoulder_roll: limit lower=-3.14159 upper=0.174533 -> lower=-3.14159 upper=0.174533 effort=30 velocity=1
- joint wrist_pitch: limit lower=-1.22173 upper=1.22173 -> lower=-1.22173 upper=1.22173 effort=30 velocity=1
- joint wrist_roll: limit lower=-1.0472 upper=1.0472 -> lower=-1.0472 upper=1.0472 effort=30 velocity=1

File: myGym/envs/robots/universal_robots/urdf/ur10.urdf (robot description, URDF)
Before this commit: robot ur10, 12 links, 11 joints
Joints:
- joint elbow_joint: limit lower=-3.14159265359 upper=3.14159265359 effort=150.0 velocity=3.15 -> lower=-3.14159265359 upper=3.14159265359 effort=30.0 velocity=1
- joint shoulder_lift_joint: limit lower=-6.28318530718 upper=6.28318530718 effort=330.0 velocity=2.16 -> lower=-6.28318530718 upper=6.28318530718 effort=30.0 velocity=1
- joint shoulder_pan_joint: limit lower=-6.28318530718 upper=6.28318530718 effort=330.0 velocity=2.16 -> lower=-6.28318530718 upper=6.28318530718 effort=30.0 velocity=1
- joint wrist_1_joint: limit lower=-6.28318530718 upper=6.28318530718 effort=54.0 velocity=3.2 -> lower=-6.28318530718 upper=6.28318530718 effort=30.0 velocity=1
- joint wrist_2_joint: limit lower=-6.28318530718 upper=6.28318530718 effort=54.0 velocity=3.2 -> lower=-6.28318530718 upper=6.28318530718 effort=30.0 velocity=1
- joint wrist_3_joint: limit lower=-6.28318530718 upper=6.28318530718 effort=54.0 velocity=3.2 -> lower=-6.28318530718 upper=6.28318530718 effort=30.0 velocity=1

File: myGym/envs/robots/universal_robots/urdf/ur3.urdf (robot description, URDF)
Before this commit: robot ur3, 12 links, 11 joints
Joints:
- joint elbow_joint: limit lower=-3.14159265359 upper=3.14159265359 effort=150.0 velocity=3.15 -> lower=-3.14159265359 upper=3.14159265359 effort=30.0 velocity=1
- joint shoulder_lift_joint: limit lower=-6.28318530718 upper=6.28318530718 effort=330.0 velocity=2.16 -> lower=-6.28318530718 upper=6.28318530718 effort=30.0 velocity=1
- joint shoulder_pan_joint: limit lower=-6.28318530718 upper=6.28318530718 effort=330.0 velocity=2.16 -> lower=-6.28318530718 upper=6.28318530718 effort=30.0 velocity=1
- joint wrist_1_joint: limit lower=-6.28318530718 upper=6.28318530718 effort=54.0 velocity=3.2 -> lower=-6.28318530718 upper=6.28318530718 effort=30 velocity=1
- joint wrist_2_joint: limit lower=-6.28318530718 upper=6.28318530718 effort=54.0 velocity=3.2 -> lower=-6.28318530718 upper=6.28318530718 effort=30.0 velocity=1
- joint wrist_3_joint: limit lower=-6.28318530718 upper=6.28318530718 effort=54.0 velocity=3.2 -> lower=-6.28318530718 upper=6.28318530718 effort=30 velocity=1

File: myGym/envs/robots/universal_robots/urdf/ur5.urdf (robot description, URDF)
Before this commit: robot ur5, 12 links, 11 joints
Joints:
- joint elbow_joint: limit lower=-3.14159265359 upper=3.14159265359 effort=150.0 velocity=3.15 -> lower=-3.14159265359 upper=3.14159265359 effort=30 velocity=1
- joint shoulder_lift_joint: limit lower=-6.28318530718 upper=6.28318530718 effort=150.0 velocity=3.15 -> lower=-6.28318530718 upper=6.28318530718 effort=30.0 velocity=1
- joint shoulder_pan_joint: limit lower=-6.28318530718 upper=6.28318530718 effort=150.0 velocity=3.15 -> lower=-6.28318530718 upper=6.28318530718 effort=30.0 velocity=1
- joint wrist_1_joint: limit lower=-6.28318530718 upper=6.28318530718 effort=28.0 velocity=3.2 -> lower=-6.28318530718 upper=6.28318530718 effort=30 velocity=1
- joint wrist_2_joint: limit lower=-6.28318530718 upper=6.28318530718 effort=28.0 velocity=3.2 -> lower=-6.28318530718 upper=6.28318530718 effort=30.0 velocity=1
- joint wrist_3_joint: limit lower=-6.28318530718 upper=6.28318530718 effort=28.0 velocity=3.2 -> lower=-6.28318530718 upper=6.28318530718 effort=30.0 velocity=1
