Commit message: ur robots gripper update, pnp multitask bugfix, 4network pnp

File: myGym/envs/robots/universal_robots/urdf/ur10.urdf (robot description, URDF)
Before this commit: robot ur10, 12 links, 11 joints
Links:
- added link endeffector; visual sphere radius=0.01
- link gripper: geometry visual box size=0.01 0.01 0.01
Joints:
- added joint endeffector_joint: type fixed, parent gripper, child endeffector, origin xyz=0.05 0.0 0.0 rpy=0 0 0

File: myGym/envs/robots/universal_robots/urdf/ur3.urdf (robot description, URDF)
Before this commit: robot ur3, 12 links, 11 joints
Links:
- added link endeffector; visual sphere radius=0.01
- link gripper: geometry visual box size=0.01 0.01 0.01
Joints:
- added joint endeffector_joint: type fixed, parent gripper, child endeffector, origin xyz=0.05 0.0 0.0 rpy=0 0 0

File: myGym/envs/robots/universal_robots/urdf/ur5.urdf (robot description, URDF)
Before this commit: robot ur5, 12 links, 11 joints
Links:
- added link endeffector; visual sphere radius=0.01
- link gripper: geometry visual box size=0.01 0.01 0.01
Joints:
- added joint endeffector_joint: type fixed, parent gripper, child endeffector, origin xyz=0.05 0.0 0.0 rpy=0 0 0
