Commit message: pepper right_hand working

File: myGym/envs/robots/pepper/pepper.urdf (robot description, URDF)
Before this commit: robot JulietteY20MP, 99 links, 98 joints
Links:
- removed link RFinger23_link
- added link LFinger23_link, mass 2e-03; collision mesh filename=meshes/pepper/PhalaxEnd.obj scale=1 1 1; visual mesh filename=meshes/pepper/PhalaxEnd.obj scale=1 1 1
Joints:
- removed joint LElbowRoll_rjoint
- removed joint LElbowYaw_rjoint
- removed joint LHand_rjoint
- removed joint LShoulderPitch_rjoint
- removed joint LShoulderRoll_rjoint
- removed joint LThumb2_rjoint
- removed joint LWristYaw_rjoint
- removed joint RElbowRoll
- removed joint RElbowYaw
- removed joint RFinger21
- removed joint RFinger22
- removed joint RFinger23
- removed joint RShoulderPitch
- removed joint RShoulderRoll
- removed joint RWristYaw
- added joint LElbowRoll: type fixed, parent LElbow, child LForeArm, origin xyz=0 0 0 rpy=0 0 0, axis 0 0 1.0, limit lower=-1.56207 upper=-0.00872665 effort=2.666 velocity=9.22756
- added joint LElbowYaw: type fixed, parent LBicep, child LElbow, origin xyz=0.1812 0.015 0.00013 rpy=0 -0.157079 0, axis 1.0 0 0, limit lower=-2.08567 upper=2.08567 effort=5.428 velocity=7.33998
- added joint LHand: type fixed, parent l_wrist, child l_hand, origin xyz=0.025 0 0 rpy=0 0 0, axis 1.0 0 0, limit lower=0.02 upper=0.98 effort=0.144 velocity=12.56
- added joint LShoulderPitch: type fixed, parent torso, child LShoulder, origin xyz=-0.057 0.14974 0.22582 rpy=0 0 0, axis 0 1.0 0, limit lower=-2.08567 upper=2.08567 effort=5.428 velocity=7.33998
- added joint LShoulderRoll: type fixed, parent LShoulder, child LBicep, origin xyz=0 0 0 rpy=0 0 0, axis 0 0 1.0, limit lower=0.00872665 upper=1.56207 effort=2.666 velocity=9.22756
- added joint LThumb2: type fixed, parent LThumb1_link, child LThumb2_link, origin xyz=0.022 0 0 rpy=0 0 -1.0472, axis 0 0 1.0, limit lower=0.0 upper=0.872665 effort=0.144 velocity=12.56, mimic joint=LHand multiplier=0.872665 offset=0
- added joint LWristYaw: type fixed, parent LForeArm, child l_wrist, origin xyz=0.15 0 0 rpy=0 0 0, axis 1.0 0 0, limit lower=-1.82387 upper=1.82387 effort=0.2014 velocity=17.3835
- added joint RElbowRoll_rjoint: type revolute, parent RElbow, child RForeArm, origin xyz=0 0 0 rpy=0 0 0, axis 0 0 1.0, limit lower=0.00872665 upper=1.56207 effort=22.666 velocity=19.22756
- added joint RElbowYaw_rjoint: type revolute, parent RBicep, child RElbow, origin xyz=0.19920 -0.015 0.00013 rpy=0 -0.157079 0, axis 1.0 0 0, limit lower=-2.08567 upper=2.08567 effort=25.428 velocity=25.33998
- added joint RFinger21_rjoint: type revolute, parent r_wrist, child RFinger21_link, origin xyz=0.0873 0.0073 0.006 rpy=1.5708 1.0472 0.061086, axis 0 0 1.0, limit lower=0.0 upper=0.872665 effort=0.144 velocity=12.56, mimic joint=RHand multiplier=0.872665 offset=0
- added joint RFinger22_rjoint: type revolute, parent RFinger21_link, child RFinger22_link, origin xyz=0.018 0 0 rpy=0 0 -1.0472, axis 0 0 1.0, limit lower=0.0 upper=0.872665 effort=0.144 velocity=12.56, mimic joint=RHand multiplier=0.872665 offset=0
- added joint RShoulderPitch_rjoint: type revolute, parent torso, child RShoulder, origin xyz=-0.057 -0.14974 0.22582 rpy=0 0 0, axis 0 1.0 0, limit lower=-2.08567 upper=2.08567 effort=5.428 velocity=7.33998
- added joint RShoulderRoll_rjoint: type revolute, parent RShoulder, child RBicep, origin xyz=0 0 0 rpy=0 0 0, axis 0 0 1.0, limit lower=-1.56207 upper=-0.00872665 effort=2.666 velocity=9.22756
- added joint RWristYaw_rjoint: type revolute, parent RForeArm, child r_wrist, origin xyz=0.15 0 0 rpy=0 0 0, axis 1.0 0 0, limit lower=-1.82387 upper=1.82387 effort=0.2014 velocity=17.3835
- added joint endeffector_joint: type fixed, parent RFinger22_link, child endeffector, origin xyz=0.018 0 0 rpy=0 0 -1.0472, axis 0 0 1.0, limit lower=0.0 upper=0.872665 effort=0.144 velocity=12.56, mimic joint=RHand multiplier=0.872665 offset=0
- joint LFinger23: child endeffector -> LFinger23_link
