Commit message: tiago simple.urdf - cleaned

File: myGym/envs/robots/tiago/tiago_simple.urdf (robot description, URDF)
Before this commit: robot tiago, 41 links, 40 joints
Links:
- removed link xtion_depth_frame
- removed link xtion_depth_optical_frame
- removed link xtion_link
- removed link xtion_optical_frame
- removed link xtion_orbbec_aux_joint_frame
- removed link xtion_rgb_frame
- removed link xtion_rgb_optical_frame
Joints:
- removed joint xtion_depth_joint
- removed joint xtion_depth_optical_joint
- removed joint xtion_joint
- removed joint xtion_optical_joint
- removed joint xtion_orbbec_aux_joint
- removed joint xtion_rgb_joint
- removed joint xtion_rgb_optical_joint
- joint arm_1_rjoint: limit lower=0.0 upper=2.74889357189 effort=39.0 velocity=2.7 -> lower=-2.74 upper=2.74889357189 effort=39.0 velocity=2.7
- joint torso_lift_rjoint: limit lower=0 upper=0.35 effort=2000 velocity=0.07 -> lower=0.0 upper=0.55 effort=20 velocity=1

Commit message: fixed tiago_simple

File: myGym/envs/robots/tiago/tiago_simple.urdf (robot description, URDF)
Before this commit: robot tiago, 34 links, 33 joints
Links:
- link arm_1_link: geometry visual mesh filename=meshes/arm/arm_1.stl scale=1 1 1
Joints:
- removed joint torso_lift_rjoint
- added joint torso_lift_joint: type fixed, parent torso_fixed_link, child torso_lift_link, origin xyz=0.0 0.0 0.597 rpy=0.0 0.0 0.0, axis 0 0 1, limit lower=0.0 upper=0.55 effort=20 velocity=1
