Commit message: tiago dual - urdf update

File: myGym/envs/robots/tiago/tiago_dual.urdf (robot description, URDF)
Before this commit: robot tiago_dual, 65 links, 64 joints
Links:
- removed link gripper_right_tool_link
- added link endeffector; visual sphere radius=0.01
- added link gripper, mass 0.0001
- link torso_fixed_column_link: geometry visual box size=0.18 0.2 0.55
- link torso_lift_link: geometry collision mesh filename=package://tiago_description/meshes/torso/torso_lift_collisi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 scale=1 1 1; collision mesh filename=package://tiago_description/meshes/torso/torso_lift_collisi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 scale=1 1 1
Joints:
- removed joint arm_right_1_joint
- removed joint arm_right_2_joint
- removed joint arm_right_3_joint
- removed joint arm_right_4_joint
- removed joint arm_right_5_joint
- removed joint arm_right_6_joint
- removed joint arm_right_7_joint
- removed joint gripper_right_left_finger_joint
- removed joint gripper_right_right_finger_joint
- removed joint head_1_joint
- removed joint head_2_joint
- removed joint torso_lift_joint
- removed joint wheel_left_joint
- removed joint wheel_right_joint
- added joint arm_right_1_rjoint: type revolute, parent torso_lift_link, child arm_right_1_link, origin xyz=0.02556 -0.19 -0.171 rpy=0 0 -1.57079632679, axis 0 0 1, limit lower=-1.1780972451 upper=1.57079632679 effort=43.0 velocity=1.95
- added joint arm_right_2_rjoint: type revolute, parent arm_right_1_link, child arm_right_2_link, origin xyz=0.125 -0.0195 -0.031 rpy=-1.57079632679 0.0 0.0, axis 0 0 1, limit lower=-1.1780972451 upper=1.57079632679 effort=43.0 velocity=1.95
- added joint arm_right_3_rjoint: type revolute, parent arm_right_2_link, child arm_right_3_link, origin xyz=0.0895 0.0 -0.0015 rpy=-1.57079632679 0.0 1.57079632679, axis 0 0 1, limit lower=-0.785398163397 upper=3.92699081699 effort=26 velocity=2.35
- added joint arm_right_4_rjoint: type revolute, parent arm_right_3_link, child arm_right_4_link, origin xyz=-0.02 -0.027 -0.222 rpy=-1.57079632679 -1.57079632679 0.0, axis 0 0 1, limit lower=-0.392699081699 upper=2.35619449019 effort=26 velocity=2.35
- added joint arm_right_5_rjoint: type revolute, parent arm_right_4_link, child arm_right_5_link, origin xyz=-0.162 0.02 0.027 rpy=1.57079632679 -1.57079632679 -1.57079632679, axis 0 0 1, limit lower=-2.09439510239 upper=2.09439510239 effort=3 velocity=1.95
- added joint arm_right_6_rjoint: type revolute, parent arm_right_5_link, child arm_right_6_link, origin xyz=0 0 0.15 rpy=0.0 -1.57079632679 -1.57079632679, axis 0 0 1, limit lower=-1.41371669412 upper=1.41371669412 effort=6.6 velocity=1.76
- added joint arm_right_7_rjoint: type revolute, parent arm_right_6_link, child arm_right_7_link, origin xyz=0 0 0 rpy=1.57079632679 0.0 1.57079632679, axis 0 0 1, limit lower=-2.09439510239 upper=2.09439510239 effort=6.6 velocity=1.76
- added joint endeffector_gjoint: type fixed, parent gripper, child endeffector, origin xyz=0.04 0 0 rpy=0 0 0
- added joint gripper_right_left_finger_gjoint: type prismatic, parent gripper_right_link, child gripper_right_left_finger_link, origin xyz=0. 0 0 rpy=0 0 0, axis -1 0 0, limit lower=0 upper=0.045 effort=16 velocity=0.05
- added joint gripper_right_right_finger_gjoint: type prismatic, parent gripper_right_link, child gripper_right_right_finger_link, origin xyz=0. 0 0 rpy=0 0 0, axis 1 0 0, limit lower=0.0 upper=0.045 effort=16 velocity=0.05
- added joint head_1_rjoint: type revolute, parent torso_lift_link, child head_1_link, origin xyz=0.182 0.0 0.0 rpy=0 0 0, axis 0 0 1, limit lower=-1.308996939 upper=1.308996939 effort=5.197 velocity=3.0
- added joint head_2_rjoint: type revolute, parent head_1_link, child head_2_link, origin xyz=0.005 0.0 0.098 rpy=1.57079632679 0 0, axis 0 0 1, limit lower=-1.0471975512 upper=0.785398163397 effort=2.77 velocity=3.0
- added joint torso_lift_rjoint: type prismatic, parent torso_fixed_link, child torso_lift_link, origin xyz=0.0 0.0 0.597 rpy=0.0 0.0 0.0, axis 0 0 1, limit lower=0 upper=0.35 effort=2000 velocity=5
- added joint wheel_left_rjoint: type continuous, parent ignore_suspension_left_link, child wheel_left_link, origin xyz=0 0.2022 0 rpy=-1.57079632679 0 0, axis 0 0 1, limit effort=6.0 velocity=10.152284264
- added joint wheel_right_rjoint: type continuous, parent ignore_suspension_right_link, child wheel_right_link, origin xyz=0 -0.2022 0 rpy=-1.57079632679 0 0, axis 0 0 1, limit effort=6.0 velocity=10.152284264
- joint arm_left_1_joint: type revolute -> fixed
- joint arm_left_2_joint: type revolute -> fixed
- joint arm_left_3_joint: type revolute -> fixed
- joint arm_left_4_joint: type revolute -> fixed
- joint arm_left_5_joint: type revolute -> fixed
- joint arm_left_6_joint: type revolute -> fixed
- joint arm_left_7_joint: type revolute -> fixed
- joint gripper_right_tool_joint: child gripper_right_tool_link -> gripper
- joint ignore_suspension_left_joint: type prismatic -> fixed
- joint ignore_suspension_right_joint: type prismatic -> fixed

Commit message: tiago_dual fixed - ichores env as table_tiago

File: myGym/envs/robots/tiago/tiago_dual.urdf (robot description, URDF)
Before this commit: robot tiago_dual, 66 links, 65 joints
Joints:
- joint arm_left_1_joint: origin xyz=0.02556 0.19 -0.171 rpy=3.14159265359 0 1.57079632679 -> xyz=0.02556 0.19 -0.171 rpy=3.14159265359 0 2.9
- joint arm_left_2_joint: origin xyz=0.125 -0.0195 0.031 rpy=1.57079632679 0.0 0.0 -> xyz=0.125 -0.0195 0.031 rpy=1.57079632679 -1.57079632679 0.0
- joint arm_left_3_joint: origin xyz=0.0895 0.0 -0.0015 rpy=-1.57079632679 3.14159265359 -1.57079632679 -> xyz=0.0895 0.0 -0.0015 rpy=-1.57079632679 2.9 -1.57079632679
- joint arm_left_4_joint: origin xyz=-0.02 -0.027 0.222 rpy=1.57079632679 -1.57079632679 0.0 -> xyz=-0.02 -0.027 0.222 rpy=1.57079632679 0.785 0.0
- joint torso_lift_rjoint: limit lower=0 upper=0.35 effort=2000 velocity=5 -> lower=0.349 upper=0.35 effort=2000 velocity=5

Commit message: tiago robot update - Tiago base rotated, reach traning created

File: myGym/envs/robots/tiago/tiago_dual.urdf (robot description, URDF)
Before this commit: robot tiago_dual, 66 links, 65 joints
Links:
- link arm_right_1_link: geometry visual mesh filename=package://tiago_description/meshes/arm/arm_1.stl scale=1 -1 1
- link torso_lift_link: geometry visual mesh filename=package://tiago_dual_description/meshes/torso/torso_lift_du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 scale=1 1 1
Joints:
- removed joint head_1_rjoint
- removed joint head_2_rjoint
- removed joint torso_lift_rjoint
- removed joint wheel_left_rjoint
- removed joint wheel_right_rjoint
- added joint head_1_joint: type fixed, parent torso_lift_link, child head_1_link, origin xyz=0.182 0.0 0.0 rpy=0 0 0, axis 0 0 1, limit lower=-1.308996939 upper=1.308996939 effort=5.197 velocity=3.0
- added joint head_2_joint: type fixed, parent head_1_link, child head_2_link, origin xyz=0.005 0.0 0.098 rpy=1.57079632679 0 0, axis 0 0 1, limit lower=-1.0471975512 upper=0.785398163397 effort=2.77 velocity=3.0
- added joint torso_lift_joint: type fixed, parent torso_fixed_link, child torso_lift_link, origin xyz=0.0 0.0 0.95 rpy=0.0 0.0 0.0, axis 0 0 1, limit lower=0.349 upper=0.35 effort=2000 velocity=5
- added joint wheel_left_joint: type fixed, parent ignore_suspension_left_link, child wheel_left_link, origin xyz=0 0.2022 0 rpy=-1.57079632679 0 0, axis 0 0 1, limit effort=6.0 velocity=10.152284264
- added joint wheel_right_joint: type fixed, parent ignore_suspension_right_link, child wheel_right_link, origin xyz=0 -0.2022 0 rpy=-1.57079632679 0 0, axis 0 0 1, limit effort=6.0 velocity=10.152284264
