Commit message: tiago urdf update - ichores reach scripts

File: myGym/envs/robots/tiago/tiago_dual_mygym_rot.urdf (robot description, URDF)
Before this commit: robot tiago_dual_mygym, 37 links, 36 joints
Joints:
- joint arm_right_2_rjoint: limit lower=-1.1780972451 upper=1.57079632679 effort=43.0 velocity=1.95 -> lower=-3.14 upper=0 effort=43.0 velocity=1.95; origin xyz=0.125 -0.0195 -0.031 rpy=-1.57079632679 0.0 0.0 -> xyz=0.125 -0.0195 -0.031 rpy=-1.57079632679 1.57 0.0
- joint arm_right_3_rjoint: origin xyz=0.0895 0.0 -0.0015 rpy=-1.57079632679 0.0 1.57079632679 -> xyz=0.0895 0.0 -0.0015 rpy=-1.57079632679 1.5707 1.57079632679
- joint arm_right_4_rjoint: limit lower=-0.392699081699 upper=2.35619449019 effort=26 velocity=2.35 -> lower=-1.57079632679 upper=0 effort=26 velocity=2.35; origin xyz=-0.02 -0.027 -0.222 rpy=-1.57079632679 -1.57079632679 0.0 -> xyz=-0.02 -0.027 -0.222 rpy=-1.57079632679 0.78 0.0
- joint baseslide_rjoint: type prismatic -> fixed

File: myGym/envs/robots/tiago/tiago_dual_mygym_rotslide.urdf (robot description, URDF)
Before this commit: robot tiago_dual_mygym, 37 links, 36 joints
Joints:
- joint baserot_rjoint: type fixed -> revolute
- joint baseslide_rjoint: limit lower=-0.5 upper=0.5 effort=16 velocity=0.05 -> lower=-0.2 upper=0.2 effort=16 velocity=0.05; type fixed -> prismatic

Commit message: tiago urdf update

File: myGym/envs/robots/tiago/tiago_dual_mygym_rot.urdf (robot description, URDF)
Before this commit: robot tiago_dual_mygym, 37 links, 36 joints
Links:
- link arm_left_1_link: geometry visual mesh filename=package://tiago_description/meshes/arm/arm_1.stl scale=1 -1 -1
- link arm_left_2_link: geometry visual mesh filename=package://tiago_description/meshes/arm/arm_2.stl scale=1 1 -1
- link arm_left_3_link: geometry visual mesh filename=package://tiago_description/meshes/arm/arm_3.stl scale=1 1 -1
- link arm_left_4_link: geometry visual mesh filename=package://tiago_description/meshes/arm/arm_4.stl scale=-1 -1 -1
- link arm_left_5_link: geometry visual mesh filename=package://tiago_description/meshes/arm/arm_5-wrist-2017.stl scale=-1 -1 -1
- link arm_left_6_link: geometry visual mesh filename=package://tiago_description/meshes/arm/arm_6-wrist-2017.stl scale=-1 1 1
- link arm_left_tool_link: geometry visual cylinder length=0.005 radius=0.005
- link base_footprint: mass 1 -> None
- link gripper_left_left_finger_link: geometry visual mesh filename=package://pal_gripper_description/meshes/gripper_finger_lin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
- link gripper_left_link: geometry visual mesh filename=package://pal_gripper_description/meshes/gripper_link.stl
- link gripper_left_right_finger_link: geometry visual mesh filename=package://pal_gripper_description/meshes/gripper_finger_lin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 scale=-1 -1 1
- link torso_lift_link: geometry collision mesh filename=package://tiago_dual_description/meshes/torso/torso_lift_du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 scale=1 1 1; visual mesh filename=package://tiago_dual_description/meshes/torso/torso_lift_du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 scale=1 1 1
- link wrist_left_ft_link: geometry visual cylinder length=0.0157 radius=0.0225
- link wrist_left_ft_tool_link: geometry visual cylinder length=0.00975 radius=0.025
Joints:
- joint baserot_rjoint: limit lower=-1.1780972451 upper=1.57079632679 effort=16 velocity=1.95 -> lower=-1.5780972451 upper=1.57079632679 effort=100 velocity=2; origin xyz=0 0 0.1 rpy=0 0 0 -> xyz=0 0 0 rpy=0 0 0
- joint baseslide_rjoint: limit lower=-0.5 upper=0.5 effort=16 velocity=0.05 -> lower=-0.5 upper=0.5 effort=500 velocity=1

File: myGym/envs/robots/tiago/tiago_dual_mygym_rotslide.urdf (robot description, URDF)
Before this commit: robot tiago_dual_mygym, 37 links, 36 joints
Links:
- link arm_left_1_link: geometry visual mesh filename=package://tiago_description/meshes/arm/arm_1.stl scale=1 -1 -1
- link arm_left_2_link: geometry visual mesh filename=package://tiago_description/meshes/arm/arm_2.stl scale=1 1 -1
- link arm_left_3_link: geometry visual mesh filename=package://tiago_description/meshes/arm/arm_3.stl scale=1 1 -1
- link arm_left_4_link: geometry visual mesh filename=package://tiago_description/meshes/arm/arm_4.stl scale=-1 -1 -1
- link arm_left_5_link: geometry visual mesh filename=package://tiago_description/meshes/arm/arm_5-wrist-2017.stl scale=-1 -1 -1
- link arm_left_6_link: geometry visual mesh filename=package://tiago_description/meshes/arm/arm_6-wrist-2017.stl scale=-1 1 1
- link arm_left_tool_link: geometry visual cylinder length=0.005 radius=0.005
- link base_footprint: mass 1 -> None
- link gripper_left_left_finger_link: geometry visual mesh filename=package://pal_gripper_description/meshes/gripper_finger_lin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
- link gripper_left_link: geometry visual mesh filename=package://pal_gripper_description/meshes/gripper_link.stl
- link gripper_left_right_finger_link: geometry visual mesh filename=package://pal_gripper_description/meshes/gripper_finger_lin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 scale=-1 -1 1
- link torso_lift_link: geometry collision mesh filename=package://tiago_dual_description/meshes/torso/torso_lift_du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 scale=1 1 1; visual mesh filename=package://tiago_dual_description/meshes/torso/torso_lift_du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 scale=1 1 1
- link wrist_left_ft_link: geometry visual cylinder length=0.0157 radius=0.0225
- link wrist_left_ft_tool_link: geometry visual cylinder length=0.00975 radius=0.025
Joints:
- joint baserot_rjoint: limit lower=-1.1780972451 upper=1.57079632679 effort=16 velocity=1.95 -> lower=-1.5780972451 upper=1.57079632679 effort=100 velocity=2; origin xyz=0 0 0.1 rpy=0 0 0 -> xyz=0 0 0 rpy=0 0 0
- joint baseslide_rjoint: limit lower=-0.2 upper=0.2 effort=16 velocity=0.05 -> lower=-0.5 upper=0.5 effort=500 velocity=1

Commit message: tiago bodu update + ycb object + traning script ichores

File: myGym/envs/robots/tiago/tiago_dual_mygym_rot.urdf (robot description, URDF)
Before this commit: robot tiago_dual_mygym, 37 links, 36 joints
Joints:
- joint baserot_rjoint: limit lower=-1.5780972451 upper=1.57079632679 effort=100 velocity=2 -> lower=-1.9780972451 upper=33.14159265359 effort=100 velocity=2
- joint endeffector_gjoint: origin xyz=0.0 0.0 -0.15 rpy=0 0 0 -> xyz=0.0 0.0 -0.23 rpy=0 0 0

File: myGym/envs/robots/tiago/tiago_dual_mygym_rotslide.urdf (robot description, URDF)
Before this commit: robot tiago_dual_mygym, 37 links, 36 joints
Joints:
- joint baserot_rjoint: limit lower=-1.5780972451 upper=1.57079632679 effort=100 velocity=2 -> lower=-1.9780972451 upper=3.14159265359 effort=100 velocity=2
- joint endeffector_gjoint: origin xyz=0.0 0.0 -0.15 rpy=0 0 0 -> xyz=0.0 0.0 -0.23 rpy=0 0 0

Commit message: tiago bodu update + ycb object + traning script ichores
(cherry picked from commit 54e017c740d2f871b5ac1217e67529beae35f71c)

File: myGym/envs/robots/tiago/tiago_dual_mygym_rot.urdf (robot description, URDF)
Before this commit: robot tiago_dual_mygym, 37 links, 36 joints
Joints:
- joint baserot_rjoint: limit lower=-1.9780972451 upper=3.14159265359 effort=100 velocity=2 -> lower=-1.5780972451 upper=1.57079632679 effort=100 velocity=2
- joint endeffector_gjoint: origin xyz=0.0 0.0 -0.23 rpy=0 0 0 -> xyz=0.0 0.0 -0.15 rpy=0 0 0

Commit message: cherrypick bugfies - tiago hardcopy from master

File: myGym/envs/robots/tiago/tiago_dual_mygym_rot.urdf (robot description, URDF)
Before this commit: robot tiago_dual_mygym, 37 links, 36 joints
Joints:
- joint baserot_rjoint: limit lower=-1.5780972451 upper=1.57079632679 effort=100 velocity=2 -> lower=-1.9780972451 upper=3.14159265359 effort=100 velocity=2
- joint endeffector_gjoint: origin xyz=0.0 0.0 -0.15 rpy=0 0 0 -> xyz=0.0 0.0 -0.23 rpy=0 0 0
