Commit message: new tiago robot urdf and new train configs

File: myGym/envs/robots/tiago/tiago_dual_mygym_rotslide2.urdf (robot description, URDF)
Before this commit: robot tiago_dual_mygym, 37 links, 36 joints
Links:
- added link base_footprint2
Joints:
- added joint baseslide2_rjoint: type prismatic, parent base_footprint, child base_footprint2, origin xyz=0. 0 0 rpy=0 0 0, axis 1 0 0, limit lower=-0.5 upper=0.4 effort=500 velocity=1
- joint baserot_rjoint: parent base_footprint -> base_footprint2
- joint baseslide_rjoint: limit lower=-0.5 upper=0.5 effort=500 velocity=1 -> lower=-0.7 upper=0.35 effort=500 velocity=1; type fixed -> prismatic

Commit message: dummy target object added

File: myGym/envs/robots/tiago/tiago_dual_mygym_rotslide2.urdf (robot description, URDF)
Before this commit: robot tiago_dual_mygym, 38 links, 37 joints
Joints:
- joint baseslide_pjoint2: limit lower=-0.5 upper=0.2 effort=16 velocity=0.05 -> lower=-0.5 upper=0.275 effort=16 velocity=0.05

Commit message: update tiago URDF files

File: myGym/envs/robots/tiago/tiago_dual_mygym_rotslide2.urdf (robot description, URDF)
Before this commit: robot tiago_dual_mygym, 38 links, 37 joints
Links:
- link arm_left_1_link: geometry collision mesh filename=package://tiago_description/meshes/arm/arm_1_collision.dae scale=1 -1 -1; visual mesh filename=package://tiago_description/meshes/arm/arm_1.stl scale=1 -1 -1
- link arm_left_2_link: geometry collision mesh filename=package://tiago_description/meshes/arm/arm_2_collision.dae scale=1 1 -1; visual mesh filename=package://tiago_description/meshes/arm/arm_2.stl scale=1 1 -1
- link arm_left_3_link: geometry collision mesh filename=package://tiago_description/meshes/arm/arm_3_collision.dae scale=1 1 -1; visual mesh filename=package://tiago_description/meshes/arm/arm_3.stl scale=1 1 -1
- link arm_left_4_link: geometry collision mesh filename=package://tiago_description/meshes/arm/arm_4_collision.dae scale=-1 -1 -1; visual mesh filename=package://tiago_description/meshes/arm/arm_4.stl scale=-1 -1 -1
- link arm_left_5_link: geometry collision mesh filename=package://tiago_description/meshes/arm/arm_5_collision-wris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 scale=-1 -1 -1; visual mesh filename=package://tiago_description/meshes/arm/arm_5-wrist-2017.stl scale=-1 -1 -1
- link arm_left_6_link: geometry collision mesh filename=package://tiago_description/meshes/arm/arm_6_collision-wris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 scale=-1 1 1; visual mesh filename=package://tiago_description/meshes/arm/arm_6-wrist-2017.stl scale=-1 1 1
- link arm_left_tool_link: geometry collision cylinder length=0.005 radius=0.005; visual cylinder length=0.005 radius=0.005
- link gripper_left_left_finger_link: geometry collision box size=0.01 0.05 0.11; visual mesh filename=package://pal_gripper_description/meshes/gripper_finger_lin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
- link gripper_left_link: geometry collision mesh filename=package://pal_gripper_description/meshes/gripper_link_colli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; visual mesh filename=package://pal_gripper_description/meshes/gripper_link.stl
- link gripper_left_right_finger_link: geometry collision box size=0.01 0.05 0.11; visual mesh filename=package://pal_gripper_description/meshes/gripper_finger_lin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 scale=-1 -1 1
- link torso_fixed_column_link: geometry visual box size=0.18 0.2 0.9
- link torso_lift_link: geometry visual mesh filename=package://tiago_dual_description/meshes/torso/torso_lift_du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 scale=1 1 1
- link wrist_left_ft_link: geometry collision cylinder length=0.0157 radius=0.0225; visual cylinder length=0.0157 radius=0.0225
- link wrist_left_ft_tool_link: geometry collision cylinder length=0.00975 radius=0.025; visual cylinder length=0.00975 radius=0.025
Joints:
- removed joint baseslide2_rjoint
- removed joint baseslide_rjoint
- removed joint torso_lift_joint
- added joint baseslide_pjoint: type prismatic, parent world, child base_footprint, origin xyz=0. 0 0 rpy=0 0 0, axis 0 1 0, limit lower=-0.5 upper=0.5 effort=16 velocity=0.05
- added joint baseslide_pjoint2: type prismatic, parent base_footprint, child base_footprint2, origin xyz=0. 0 0 rpy=0 0 0, axis 1 0 0, limit lower=-0.5 upper=0.275 effort=16 velocity=0.05
- added joint torso_lift_pjoint: type prismatic, parent torso_fixed_link, child torso_lift_link, origin xyz=0.0 0.0 0.95 rpy=0.0 0.0 0.0, axis 0 0 1, limit lower=0.0 upper=0.35 effort=2000 velocity=5
- joint baserot_rjoint: limit lower=-1.9780972451 upper=3.14159265359 effort=100 velocity=2 -> lower=-1.1780972451 upper=1.57079632679 effort=16 velocity=1.95; origin xyz=0 0 0 rpy=0 0 0 -> xyz=0 0 0.1 rpy=0 0 0
- joint endeffector_gjoint: origin xyz=0.0 0.0 -0.23 rpy=0 0 0 -> xyz=0.0 0.0 -0.20 rpy=0 0 -3.14
- joint gripper_right_left_finger_gjoint: limit lower=0.044 upper=0.045 effort=16 velocity=10 -> lower=0.0 upper=0.045 effort=16 velocity=10
- joint gripper_right_right_finger_gjoint: limit lower=0.044 upper=0.045 effort=16 velocity=10 -> lower=0.0 upper=0.045 effort=16 velocity=10

Commit message: slider works for all tiago robots

File: myGym/envs/robots/tiago/tiago_dual_mygym_rotslide2.urdf (robot description, URDF)
Before this commit: robot tiago_dual_mygym, 38 links, 37 joints
Links:
- link arm_left_1_link: geometry collision mesh filename=package://tiago_description/meshes/arm/arm_1_collision.dae scale=1 -1 -1; visual mesh filename=package://tiago_description/meshes/arm/arm_1.stl scale=1 -1 -1
- link arm_right_2_link: geometry collision mesh filename=package://tiago_description/meshes/arm/arm_2_collision.dae scale=1 1 1; visual mesh filename=package://tiago_description/meshes/arm/arm_2.stl scale=1 1 1
- link arm_right_3_link: geometry collision mesh filename=package://tiago_description/meshes/arm/arm_3_collision.dae scale=1 1 1; visual mesh filename=package://tiago_description/meshes/arm/arm_3.stl scale=1 1 1
- link arm_right_4_link: geometry collision mesh filename=package://tiago_description/meshes/arm/arm_4_collision.dae scale=1 1 1; visual mesh filename=package://tiago_description/meshes/arm/arm_4.stl scale=1 1 1
- link arm_right_5_link: mass 1.655819 -> 0.9359143689; geometry collision mesh filename=package://tiago_description/meshes/arm/arm_5_collision-wris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 scale=1 1 1; visual mesh filename=package://tiago_description/meshes/arm/arm_5-wrist-2017.stl scale=1 1 1
- link arm_right_6_link: mass 0.370063 -> 0.30275767222; geometry collision mesh filename=package://tiago_description/meshes/arm/arm_6_collision-wris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 scale=1 1 1; visual mesh filename=package://tiago_description/meshes/arm/arm_6-wrist-2017.stl scale=1 1 1
- link arm_right_7_link: mass 0.234252 -> 0.100
- link arm_right_tool_link: geometry collision cylinder length=0.005 radius=0.005; visual cylinder length=0.005 radius=0.005
- link base_footprint: mass None -> 1
- link base_footprint2: mass None -> 1
- link base_link: mass 20.26649 -> 28.26649
- link gripper_right_left_finger_link: geometry visual mesh filename=package://pal_gripper_description/meshes/gripper_finger_lin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
- link gripper_right_link: geometry collision mesh filename=package://pal_gripper_description/meshes/gripper_link_colli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; visual mesh filename=package://pal_gripper_description/meshes/gripper_link.stl
- link gripper_right_right_finger_link: geometry visual mesh filename=package://pal_gripper_description/meshes/gripper_finger_lin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 scale=-1 -1 1
- link head_1_link: geometry collision mesh filename=package://tiago_description/meshes/head/head_1_collision.dae scale=1 1 1; visual mesh filename=package://tiago_description/meshes/head/head_1.stl scale=1 1 1
- link head_2_link: geometry collision mesh filename=package://tiago_description/meshes/head/head_2_collision.dae scale=1 1 1; visual mesh filename=package://tiago_description/meshes/head/head_2.stl scale=1 1 1
- link torso_fixed_column_link: geometry visual box size=0.18 0.2 0.55
- link torso_lift_link: geometry visual mesh filename=package://tiago_dual_description/meshes/torso/torso_lift_du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 scale=1 1 1
- link wrist_right_ft_link: geometry collision cylinder length=0.0157 radius=0.0225; visual cylinder length=0.0157 radius=0.0225
- link wrist_right_ft_tool_link: geometry collision cylinder length=0.00975 radius=0.025; visual cylinder length=0.00975 radius=0.025
Joints:
- removed joint baseslide2_rjoint
- removed joint torso_lift_rjoint
- added joint baseslide_rjoint2: type prismatic, parent base_footprint, child base_footprint2, origin xyz=0. 0 0 rpy=0 0 0, axis 1 0 0, limit lower=-0.5 upper=0.5 effort=16 velocity=0.05
- added joint torso_lift_gjoint: type prismatic, parent torso_fixed_link, child torso_lift_link, origin xyz=0.0 0.0 0.61 rpy=0.0 0.0 0.0, axis 0 0 1, limit lower=0.0 upper=0.35 effort=2000 velocity=5
- joint arm_left_1_joint: limit lower=-1.1780972451 upper=1.57079632679 effort=43.0 velocity=10 -> lower=-1.1780972451 upper=1.57079632679 effort=43.0 velocity=1.95
- joint arm_right_2_rjoint: limit lower=-1.1780972450961724 upper=1.5707963267948966 effort=43.0 velocity=1.95 -> lower=-1.1780972451 upper=1.57079632679 effort=43.0 velocity=1.95; origin xyz=0.125 -0.0195 -0.031 rpy=-1.5707963267948966 0.0 0.0 -> xyz=0.125 -0.0195 -0.031 rpy=-1.57079632679 0.0 0.0
- joint arm_right_3_rjoint: limit lower=-0.7853981633974483 upper=3.9269908169872414 effort=26 velocity=2.35 -> lower=-0.785398163397 upper=3.92699081699 effort=26 velocity=2.35; origin xyz=0.0895 0.0 -0.0015 rpy=-1.5707963267948966 0.0 1.5707963267948966 -> xyz=0.0895 0.0 -0.0015 rpy=-1.57079632679 0.0 1.57079632679
- joint arm_right_4_rjoint: limit lower=-1.57079632679 upper=0 effort=26 velocity=2.35 -> lower=-0.392699081699 upper=2.35619449019 effort=26 velocity=2.35; origin xyz=-0.02 -0.027 -0.222 rpy=-1.57079632679 0.78 0.0 -> xyz=-0.02 -0.027 -0.222 rpy=-1.57079632679 -1.57079632679 0.0
- joint baserot_rjoint: limit lower=-3.140972451 upper=3.140972451 effort=200 velocity=20 -> lower=-1.1780972451 upper=1.57079632679 effort=16 velocity=1.95
- joint baseslide_rjoint: limit lower=-0.7 upper=0.35 effort=500 velocity=1 -> lower=-0.5 upper=0.5 effort=16 velocity=0.05
- joint endeffector_joint: origin xyz=0.0 0.0 -0.20 rpy=0 0 0 -> xyz=0.0 0.0 -0.20 rpy=0 0 -1.57

File: myGym/envs/robots/tiago/tiago_rotslide2_backup.urdf (robot description, URDF)
Before this commit: robot tiago_dual_mygym, 37 links, 36 joints
Links:
- added link base_footprint2, mass 1
- link arm_left_1_link: geometry visual mesh filename=package://tiago_description/meshes/arm/arm_1.stl scale=1 -1 -1
- link arm_right_2_link: geometry visual mesh filename=package://tiago_description/meshes/arm/arm_2.stl scale=1 1 1
- link arm_right_3_link: geometry visual mesh filename=package://tiago_description/meshes/arm/arm_3.stl scale=1 1 1
- link arm_right_4_link: geometry visual mesh filename=package://tiago_description/meshes/arm/arm_4.stl scale=1 1 1
- link arm_right_5_link: mass 0.9359143689 -> 1.655819; geometry visual mesh filename=package://tiago_description/meshes/arm/arm_5-wrist-2017.stl scale=1 1 1
- link arm_right_6_link: mass 0.30275767222 -> 0.370063; geometry visual mesh filename=package://tiago_description/meshes/arm/arm_6-wrist-2017.stl scale=1 1 1
- link arm_right_7_link: mass 0.100 -> 0.234252
- link arm_right_tool_link: geometry visual cylinder length=0.005 radius=0.005
- link base_link: mass 28.26649 -> 20.26649
- link gripper_right_left_finger_link: geometry collision mesh filename=package://pal_gripper_description/meshes/gripper_finger_lin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; visual mesh filename=package://pal_gripper_description/meshes/gripper_finger_lin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
- link gripper_right_link: geometry visual mesh filename=package://pal_gripper_description/meshes/gripper_link.stl
- link gripper_right_right_finger_link: geometry collision mesh filename=package://pal_gripper_description/meshes/gripper_finger_lin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 scale=-1 -1 1; visual mesh filename=package://pal_gripper_description/meshes/gripper_finger_lin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 scale=-1 -1 1
- link head_1_link: geometry visual mesh filename=package://tiago_description/meshes/head/head_1.stl scale=1 1 1
- link head_2_link: geometry visual mesh filename=package://tiago_description/meshes/head/head_2.stl scale=1 1 1
- link torso_fixed_column_link: geometry visual box size=0.18 0.2 0.60
- link torso_lift_link: geometry collision mesh filename=package://tiago_dual_description/meshes/torso/torso_lift_du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 scale=1 1 1; visual mesh filename=package://tiago_dual_description/meshes/torso/torso_lift_du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 scale=1 1 1
- link wrist_right_ft_link: geometry visual cylinder length=0.0157 radius=0.0225
- link wrist_right_ft_tool_link: geometry visual cylinder length=0.00975 radius=0.025
Joints:
- removed joint torso_lift_gjoint
- added joint baseslide2_rjoint: type prismatic, parent base_footprint, child base_footprint2, origin xyz=0. 0 0 rpy=0 0 0, axis 1 0 0, limit lower=-0.5 upper=0.4 effort=500 velocity=1
- added joint torso_lift_rjoint: type prismatic, parent torso_fixed_link, child torso_lift_link, origin xyz=0.0 0.0 0.61 rpy=0.0 0.0 0.0, axis 0 0 1, limit lower=0.0 upper=0.35 effort=2000 velocity=5
- joint arm_left_1_joint: limit lower=-1.1780972451 upper=1.57079632679 effort=43.0 velocity=1.95 -> lower=-1.1780972451 upper=1.57079632679 effort=43.0 velocity=10
- joint arm_right_2_rjoint: limit lower=-1.1780972451 upper=1.57079632679 effort=43.0 velocity=1.95 -> lower=-1.1780972450961724 upper=1.5707963267948966 effort=43.0 velocity=1.95; origin xyz=0.125 -0.0195 -0.031 rpy=-1.57079632679 0.0 0.0 -> xyz=0.125 -0.0195 -0.031 rpy=-1.5707963267948966 0.0 0.0
- joint arm_right_3_rjoint: limit lower=-0.785398163397 upper=3.92699081699 effort=26 velocity=2.35 -> lower=-0.7853981633974483 upper=3.9269908169872414 effort=26 velocity=2.35; origin xyz=0.0895 0.0 -0.0015 rpy=-1.57079632679 0.0 1.57079632679 -> xyz=0.0895 0.0 -0.0015 rpy=-1.5707963267948966 0.0 1.5707963267948966
- joint arm_right_4_rjoint: limit lower=-0.392699081699 upper=2.35619449019 effort=26 velocity=2.35 -> lower=-1.57079632679 upper=0 effort=26 velocity=2.35; origin xyz=-0.02 -0.027 -0.222 rpy=-1.57079632679 -1.57079632679 0.0 -> xyz=-0.02 -0.027 -0.222 rpy=-1.57079632679 0.78 0.0
- joint baserot_rjoint: limit lower=-1.1780972451 upper=1.57079632679 effort=16 velocity=1.95 -> lower=-3.140972451 upper=3.140972451 effort=200 velocity=20; parent base_footprint -> base_footprint2
- joint baseslide_rjoint: limit lower=-0.5 upper=0.5 effort=16 velocity=0.05 -> lower=-0.7 upper=0.35 effort=500 velocity=1
- joint endeffector_joint: origin xyz=0.0 0.0 -0.20 rpy=0 0 -1.57 -> xyz=0.0 0.0 -0.20 rpy=0 0 0

File: myGym/envs/robots/tiago/tiago_rotslide_old.urdf (robot description, URDF)
Before this commit: robot tiago_dual_mygym, 37 links, 36 joints
Links:
- added link base_footprint2
- link arm_left_1_link: geometry visual mesh filename=package://tiago_description/meshes/arm/arm_1.stl scale=1 -1 -1
- link arm_right_2_link: geometry visual mesh filename=package://tiago_description/meshes/arm/arm_2.stl scale=1 1 1
- link arm_right_3_link: geometry visual mesh filename=package://tiago_description/meshes/arm/arm_3.stl scale=1 1 1
- link arm_right_4_link: geometry visual mesh filename=package://tiago_description/meshes/arm/arm_4.stl scale=1 1 1
- link arm_right_5_link: mass 0.9359143689 -> 1.655819; geometry visual mesh filename=package://tiago_description/meshes/arm/arm_5-wrist-2017.stl scale=1 1 1
- link arm_right_6_link: mass 0.30275767222 -> 0.370063; geometry visual mesh filename=package://tiago_description/meshes/arm/arm_6-wrist-2017.stl scale=1 1 1
- link arm_right_7_link: mass 0.100 -> 0.234252
- link arm_right_tool_link: geometry visual cylinder length=0.005 radius=0.005
- link base_footprint: mass 1 -> None
- link base_link: mass 28.26649 -> 20.26649
- link endeffector: mass 0.0000332 -> None; geometry visual sphere radius=0.01
- link gripper_right_left_finger_link: geometry collision mesh filename=package://pal_gripper_description/meshes/gripper_finger_lin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; visual mesh filename=package://pal_gripper_description/meshes/gripper_finger_lin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
- link gripper_right_link: geometry visual mesh filename=package://pal_gripper_description/meshes/gripper_link.stl
- link gripper_right_right_finger_link: geometry collision mesh filename=package://pal_gripper_description/meshes/gripper_finger_lin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 scale=-1 -1 1; visual mesh filename=package://pal_gripper_description/meshes/gripper_finger_lin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 scale=-1 -1 1
- link head_1_link: geometry visual mesh filename=package://tiago_description/meshes/head/head_1.stl scale=1 1 1
- link head_2_link: geometry visual mesh filename=package://tiago_description/meshes/head/head_2.stl scale=1 1 1
- link torso_fixed_column_link: geometry visual box size=0.18 0.2 0.60
- link torso_lift_link: geometry collision mesh filename=package://tiago_dual_description/meshes/torso/torso_lift_du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 scale=1 1 1; visual mesh filename=package://tiago_dual_description/meshes/torso/torso_lift_du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 scale=1 1 1
- link wrist_right_ft_link: geometry visual cylinder length=0.0157 radius=0.0225
- link wrist_right_ft_tool_link: geometry visual cylinder length=0.00975 radius=0.025
Joints:
- removed joint endeffector_joint
- removed joint torso_lift_gjoint
- added joint baseslide2_rjoint: type fixed, parent base_footprint, child base_footprint2, origin xyz=0. 0 0 rpy=0 0 0, axis 1 0 0, limit lower=-0.5 upper=0.4 effort=500 velocity=1
- added joint endeffector_gjoint: type fixed, parent gripper, child endeffector, origin xyz=0.0 0.0 -0.20 rpy=0 0 -1.57079632679
- added joint torso_lift_joint: type prismatic, parent torso_fixed_link, child torso_lift_link, origin xyz=0.0 0.0 0.61 rpy=0.0 0.0 0.0, axis 0 0 1, limit lower=0.0 upper=0.35 effort=2000 velocity=5
- joint arm_left_1_joint: limit lower=-1.1780972451 upper=1.57079632679 effort=43.0 velocity=1.95 -> lower=-1.1780972451 upper=1.57079632679 effort=43.0 velocity=10
- joint arm_right_2_rjoint: limit lower=-1.1780972451 upper=1.57079632679 effort=43.0 velocity=1.95 -> lower=-1.1780972450961724 upper=1.5707963267948966 effort=43.0 velocity=1.95; origin xyz=0.125 -0.0195 -0.031 rpy=-1.57079632679 0.0 0.0 -> xyz=0.125 -0.0195 -0.031 rpy=-1.5707963267948966 0.0 0.0
- joint arm_right_3_rjoint: limit lower=-0.785398163397 upper=3.92699081699 effort=26 velocity=2.35 -> lower=-0.7853981633974483 upper=3.9269908169872414 effort=26 velocity=2.35; origin xyz=0.0895 0.0 -0.0015 rpy=-1.57079632679 0.0 1.57079632679 -> xyz=0.0895 0.0 -0.0015 rpy=-1.5707963267948966 0.0 1.5707963267948966
- joint arm_right_4_rjoint: limit lower=-0.392699081699 upper=2.35619449019 effort=26 velocity=2.35 -> lower=-1.57079632679 upper=0 effort=26 velocity=2.35; origin xyz=-0.02 -0.027 -0.222 rpy=-1.57079632679 -1.57079632679 0.0 -> xyz=-0.02 -0.027 -0.222 rpy=-1.57079632679 0.78 0.0
- joint baserot_rjoint: limit lower=-1.1780972451 upper=1.57079632679 effort=16 velocity=1.95 -> lower=-3.140972451 upper=3.140972451 effort=200 velocity=20
- joint baseslide_rjoint: limit lower=-0.5 upper=0.5 effort=16 velocity=0.05 -> lower=-0.7 upper=0.35 effort=500 velocity=1
