Commit message: first RDDL configs (up to AGMDW), Tiago gripper update, new YCB objects

File: myGym/envs/robots/tiago/tiago_dual_mygym.urdf (robot description, URDF)
Before this commit: robot tiago_dual_mygym, 37 links, 36 joints
Joints:
- joint gripper_right_left_finger_gjoint: limit lower=0.044 upper=0.045 effort=16 velocity=10 -> lower=0.0 upper=0.045 effort=16 velocity=10
- joint gripper_right_right_finger_gjoint: limit lower=0.044 upper=0.045 effort=16 velocity=10 -> lower=0.0 upper=0.045 effort=16 velocity=10

Commit message: protorewards - AGM -WIP

File: myGym/envs/robots/tiago/tiago_dual_mygym.urdf (robot description, URDF)
Before this commit: robot tiago_dual_mygym, 37 links, 36 joints
Joints:
- joint endeffector_gjoint: origin xyz=0.0 0.0 -0.15 rpy=0 0 0 -> xyz=0.0 0.0 -0.20 rpy=0 0 0

Commit message: copied additions from RDDL to master, test and train wo configs working

File: myGym/envs/robots/tiago/tiago_dual_mygym.urdf (robot description, URDF)
Before this commit: robot tiago_dual_mygym, 37 links, 36 joints
Joints:
- joint endeffector_gjoint: origin xyz=0.0 0.0 -0.15 rpy=0 0 0 -> xyz=0.0 0.0 -0.20 rpy=0 0 0
- joint gripper_right_left_finger_gjoint: limit lower=0.044 upper=0.045 effort=16 velocity=10 -> lower=0.0 upper=0.045 effort=16 velocity=10
- joint gripper_right_right_finger_gjoint: limit lower=0.044 upper=0.045 effort=16 velocity=10 -> lower=0.0 upper=0.045 effort=16 velocity=10

Commit message: verbosity bugfix - robot and table urdf missing inertia fixed, robot summary converted to self.debug mode

File: myGym/envs/robots/tiago/tiago_dual_mygym.urdf (robot description, URDF)
Before this commit: robot tiago_dual_mygym, 37 links, 36 joints
Links:
- link endeffector: mass None -> 0.00

File: myGym/envs/robots/tiago/tiago_dual_mygym_rot.urdf (robot description, URDF)
Before this commit: robot tiago_dual_mygym, 37 links, 36 joints
Links:
- link base_footprint: mass None -> 1
- link endeffector: mass None -> 0.00

File: myGym/envs/robots/tiago/tiago_dual_mygym_rotslide.urdf (robot description, URDF)
Before this commit: robot tiago_dual_mygym, 37 links, 36 joints
Links:
- link base_footprint: mass None -> 1
- link endeffector: mass None -> 0.00

File: myGym/envs/robots/tiago/tiago_dual_mygym_rotslide2.urdf (robot description, URDF)
Before this commit: robot tiago_dual_mygym, 38 links, 37 joints
Links:
- link base_footprint: mass None -> 1
- link base_footprint2: mass None -> 1
- link endeffector: mass None -> 0.00

Commit message: tiago rot oraculum working v1

File: myGym/envs/robots/tiago/tiago_dual_mygym.urdf (robot description, URDF)
Before this commit: robot tiago_dual_mygym, 37 links, 36 joints
Links:
- link torso_fixed_column_link: geometry visual box size=0.18 0.2 0.9
Joints:
- removed joint torso_lift_joint
- added joint torso_lift_pjoint: type prismatic, parent torso_fixed_link, child torso_lift_link, origin xyz=0.0 0.0 0.95 rpy=0.0 0.0 0.0, axis 0 0 1, limit lower=0.0 upper=0.35 effort=2000 velocity=5
- joint endeffector_gjoint: origin xyz=0.0 0.0 -0.20 rpy=0 0 0 -> xyz=0.0 0.0 -0.20 rpy=0 0 -3.1415

File: myGym/envs/robots/tiago/tiago_dual_mygym_rot.urdf (robot description, URDF)
Before this commit: robot tiago_dual_mygym, 37 links, 36 joints
Links:
- link arm_left_1_link: geometry collision mesh filename=package://tiago_description/meshes/arm/arm_1_collision.dae scale=1 -1 -1; visual mesh filename=package://tiago_description/meshes/arm/arm_1.stl scale=1 -1 -1
- link arm_left_2_link: geometry collision mesh filename=package://tiago_description/meshes/arm/arm_2_collision.dae scale=1 1 -1; visual mesh filename=package://tiago_description/meshes/arm/arm_2.stl scale=1 1 -1
- link arm_left_3_link: geometry collision mesh filename=package://tiago_description/meshes/arm/arm_3_collision.dae scale=1 1 -1; visual mesh filename=package://tiago_description/meshes/arm/arm_3.stl scale=1 1 -1
- link arm_left_4_link: geometry collision mesh filename=package://tiago_description/meshes/arm/arm_4_collision.dae scale=-1 -1 -1; visual mesh filename=package://tiago_description/meshes/arm/arm_4.stl scale=-1 -1 -1
- link arm_left_5_link: geometry collision mesh filename=package://tiago_description/meshes/arm/arm_5_collision-wris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 scale=-1 -1 -1; visual mesh filename=package://tiago_description/meshes/arm/arm_5-wrist-2017.stl scale=-1 -1 -1
- link arm_left_6_link: geometry collision mesh filename=package://tiago_description/meshes/arm/arm_6_collision-wris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 scale=-1 1 1; visual mesh filename=package://tiago_description/meshes/arm/arm_6-wrist-2017.stl scale=-1 1 1
- link arm_left_tool_link: geometry collision cylinder length=0.005 radius=0.005; visual cylinder length=0.005 radius=0.005
- link gripper_left_left_finger_link: geometry collision box size=0.01 0.05 0.11; visual mesh filename=package://pal_gripper_description/meshes/gripper_finger_lin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
- link gripper_left_link: geometry collision mesh filename=package://pal_gripper_description/meshes/gripper_link_colli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; visual mesh filename=package://pal_gripper_description/meshes/gripper_link.stl
- link gripper_left_right_finger_link: geometry collision box size=0.01 0.05 0.11; visual mesh filename=package://pal_gripper_description/meshes/gripper_finger_lin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 scale=-1 -1 1
- link torso_fixed_column_link: geometry visual box size=0.18 0.2 0.9
- link torso_lift_link: geometry visual mesh filename=package://tiago_dual_description/meshes/torso/torso_lift_du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 scale=1 1 1
- link wrist_left_ft_link: geometry collision cylinder length=0.0157 radius=0.0225; visual cylinder length=0.0157 radius=0.0225
- link wrist_left_ft_tool_link: geometry collision cylinder length=0.00975 radius=0.025; visual cylinder length=0.00975 radius=0.025
Joints:
- removed joint torso_lift_joint
- added joint torso_lift_pjoint: type prismatic, parent torso_fixed_link, child torso_lift_link, origin xyz=0.0 0.0 0.95 rpy=0.0 0.0 0.0, axis 0 0 1, limit lower=0.0 upper=0.35 effort=2000 velocity=5
- joint baserot_rjoint: limit lower=-1.9780972451 upper=3.14159265359 effort=100 velocity=2 -> lower=-1.1780972451 upper=1.57079632679 effort=16 velocity=1.95; origin xyz=0 0 0 rpy=0 0 0 -> xyz=0 0 0.1 rpy=0 0 0
- joint baseslide_rjoint: limit lower=-0.5 upper=0.5 effort=500 velocity=1 -> lower=-0.5 upper=0.5 effort=16 velocity=0.05
- joint endeffector_gjoint: origin xyz=0.0 0.0 -0.23 rpy=0 0 0 -> xyz=0.0 0.0 -0.20 rpy=0 0 -3.14
- joint gripper_right_left_finger_gjoint: limit lower=0.044 upper=0.045 effort=16 velocity=10 -> lower=0.0 upper=0.045 effort=16 velocity=10
- joint gripper_right_right_finger_gjoint: limit lower=0.044 upper=0.045 effort=16 velocity=10 -> lower=0.0 upper=0.045 effort=16 velocity=10

File: myGym/envs/robots/tiago/tiago_dual_mygym_rotslide.urdf (robot description, URDF)
Before this commit: robot tiago_dual_mygym, 37 links, 36 joints
Links:
- link arm_left_1_link: geometry collision mesh filename=package://tiago_description/meshes/arm/arm_1_collision.dae scale=1 -1 -1; visual mesh filename=package://tiago_description/meshes/arm/arm_1.stl scale=1 -1 -1
- link arm_left_2_link: geometry collision mesh filename=package://tiago_description/meshes/arm/arm_2_collision.dae scale=1 1 -1; visual mesh filename=package://tiago_description/meshes/arm/arm_2.stl scale=1 1 -1
- link arm_left_3_link: geometry collision mesh filename=package://tiago_description/meshes/arm/arm_3_collision.dae scale=1 1 -1; visual mesh filename=package://tiago_description/meshes/arm/arm_3.stl scale=1 1 -1
- link arm_left_4_link: geometry collision mesh filename=package://tiago_description/meshes/arm/arm_4_collision.dae scale=-1 -1 -1; visual mesh filename=package://tiago_description/meshes/arm/arm_4.stl scale=-1 -1 -1
- link arm_left_5_link: geometry collision mesh filename=package://tiago_description/meshes/arm/arm_5_collision-wris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 scale=-1 -1 -1; visual mesh filename=package://tiago_description/meshes/arm/arm_5-wrist-2017.stl scale=-1 -1 -1
- link arm_left_6_link: geometry collision mesh filename=package://tiago_description/meshes/arm/arm_6_collision-wris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 scale=-1 1 1; visual mesh filename=package://tiago_description/meshes/arm/arm_6-wrist-2017.stl scale=-1 1 1
- link arm_left_tool_link: geometry collision cylinder length=0.005 radius=0.005; visual cylinder length=0.005 radius=0.005
- link gripper_left_left_finger_link: geometry collision box size=0.01 0.05 0.11; visual mesh filename=package://pal_gripper_description/meshes/gripper_finger_lin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
- link gripper_left_link: geometry collision mesh filename=package://pal_gripper_description/meshes/gripper_link_colli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; visual mesh filename=package://pal_gripper_description/meshes/gripper_link.stl
- link gripper_left_right_finger_link: geometry collision box size=0.01 0.05 0.11; visual mesh filename=package://pal_gripper_description/meshes/gripper_finger_lin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 scale=-1 -1 1
- link torso_fixed_column_link: geometry visual box size=0.18 0.2 0.9
- link torso_lift_link: geometry visual mesh filename=package://tiago_dual_description/meshes/torso/torso_lift_du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 scale=1 1 1
- link wrist_left_ft_link: geometry collision cylinder length=0.0157 radius=0.0225; visual cylinder length=0.0157 radius=0.0225
- link wrist_left_ft_tool_link: geometry collision cylinder length=0.00975 radius=0.025; visual cylinder length=0.00975 radius=0.025
Joints:
- removed joint baseslide_rjoint
- removed joint torso_lift_joint
- added joint baseslide_pjoint: type prismatic, parent world, child base_footprint, origin xyz=0. 0 0 rpy=0 0 0, axis 0 1 0, limit lower=-0.5 upper=0.5 effort=16 velocity=0.05
- added joint torso_lift_pjoint: type prismatic, parent torso_fixed_link, child torso_lift_link, origin xyz=0.0 0.0 0.95 rpy=0.0 0.0 0.0, axis 0 0 1, limit lower=0.0 upper=0.35 effort=2000 velocity=5
- joint baserot_rjoint: limit lower=-1.9780972451 upper=3.14159265359 effort=100 velocity=2 -> lower=-1.1780972451 upper=1.57079632679 effort=16 velocity=1.95; origin xyz=0 0 0 rpy=0 0 0 -> xyz=0 0 0.1 rpy=0 0 0
- joint endeffector_gjoint: origin xyz=0.0 0.0 -0.23 rpy=0 0 0 -> xyz=0.0 0.0 -0.20 rpy=0 0 -3.14
- joint gripper_right_left_finger_gjoint: limit lower=0.044 upper=0.045 effort=16 velocity=10 -> lower=0.0 upper=0.045 effort=16 velocity=10
- joint gripper_right_right_finger_gjoint: limit lower=0.044 upper=0.045 effort=16 velocity=10 -> lower=0.0 upper=0.045 effort=16 velocity=10

File: myGym/envs/robots/tiago/tiago_dual_mygym_rotslide2.urdf (robot description, URDF)
Before this commit: robot tiago_dual_mygym, 38 links, 37 joints
Links:
- link arm_left_1_link: geometry collision mesh filename=package://tiago_description/meshes/arm/arm_1_collision.dae scale=1 -1 -1; visual mesh filename=package://tiago_description/meshes/arm/arm_1.stl scale=1 -1 -1
- link arm_left_2_link: geometry collision mesh filename=package://tiago_description/meshes/arm/arm_2_collision.dae scale=1 1 -1; visual mesh filename=package://tiago_description/meshes/arm/arm_2.stl scale=1 1 -1
- link arm_left_3_link: geometry collision mesh filename=package://tiago_description/meshes/arm/arm_3_collision.dae scale=1 1 -1; visual mesh filename=package://tiago_description/meshes/arm/arm_3.stl scale=1 1 -1
- link arm_left_4_link: geometry collision mesh filename=package://tiago_description/meshes/arm/arm_4_collision.dae scale=-1 -1 -1; visual mesh filename=package://tiago_description/meshes/arm/arm_4.stl scale=-1 -1 -1
- link arm_left_5_link: geometry collision mesh filename=package://tiago_description/meshes/arm/arm_5_collision-wris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 scale=-1 -1 -1; visual mesh filename=package://tiago_description/meshes/arm/arm_5-wrist-2017.stl scale=-1 -1 -1
- link arm_left_6_link: geometry collision mesh filename=package://tiago_description/meshes/arm/arm_6_collision-wris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 scale=-1 1 1; visual mesh filename=package://tiago_description/meshes/arm/arm_6-wrist-2017.stl scale=-1 1 1
- link arm_left_tool_link: geometry collision cylinder length=0.005 radius=0.005; visual cylinder length=0.005 radius=0.005
- link gripper_left_left_finger_link: geometry collision box size=0.01 0.05 0.11; visual mesh filename=package://pal_gripper_description/meshes/gripper_finger_lin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
- link gripper_left_link: geometry collision mesh filename=package://pal_gripper_description/meshes/gripper_link_colli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; visual mesh filename=package://pal_gripper_description/meshes/gripper_link.stl
- link gripper_left_right_finger_link: geometry collision box size=0.01 0.05 0.11; visual mesh filename=package://pal_gripper_description/meshes/gripper_finger_lin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 scale=-1 -1 1
- link torso_fixed_column_link: geometry visual box size=0.18 0.2 0.9
- link torso_lift_link: geometry visual mesh filename=package://tiago_dual_description/meshes/torso/torso_lift_du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 scale=1 1 1
- link wrist_left_ft_link: geometry collision cylinder length=0.0157 radius=0.0225; visual cylinder length=0.0157 radius=0.0225
- link wrist_left_ft_tool_link: geometry collision cylinder length=0.00975 radius=0.025; visual cylinder length=0.00975 radius=0.025
Joints:
- removed joint baseslide2_rjoint
- removed joint baseslide_rjoint
- removed joint torso_lift_joint
- added joint baseslide_pjoint: type prismatic, parent world, child base_footprint, origin xyz=0. 0 0 rpy=0 0 0, axis 0 1 0, limit lower=-0.5 upper=0.5 effort=16 velocity=0.05
- added joint baseslide_pjoint2: type prismatic, parent base_footprint, child base_footprint2, origin xyz=0. 0 0 rpy=0 0 0, axis 1 0 0, limit lower=-0.5 upper=0.2 effort=16 velocity=0.05
- added joint torso_lift_pjoint: type prismatic, parent torso_fixed_link, child torso_lift_link, origin xyz=0.0 0.0 0.95 rpy=0.0 0.0 0.0, axis 0 0 1, limit lower=0.0 upper=0.35 effort=2000 velocity=5
- joint baserot_rjoint: limit lower=-1.9780972451 upper=3.14159265359 effort=100 velocity=2 -> lower=-1.1780972451 upper=1.57079632679 effort=16 velocity=1.95; origin xyz=0 0 0 rpy=0 0 0 -> xyz=0 0 0.1 rpy=0 0 0
- joint endeffector_gjoint: origin xyz=0.0 0.0 -0.23 rpy=0 0 0 -> xyz=0.0 0.0 -0.20 rpy=0 0 -3.14
- joint gripper_right_left_finger_gjoint: limit lower=0.044 upper=0.045 effort=16 velocity=10 -> lower=0.0 upper=0.045 effort=16 velocity=10
- joint gripper_right_right_finger_gjoint: limit lower=0.044 upper=0.045 effort=16 velocity=10 -> lower=0.0 upper=0.045 effort=16 velocity=10

Commit message: oraculum update, tiago urdf change

File: myGym/envs/robots/tiago/tiago_dual_mygym.urdf (robot description, URDF)
Before this commit: robot tiago_dual_mygym, 37 links, 36 joints
Links:
- link endeffector: geometry visual cylinder length=0.07 radius=0.01
Joints:
- removed joint endeffector_gjoint
- added joint endeffector: type fixed, parent gripper, child endeffector, origin xyz=0.0 0.0 -0.20 rpy=0 0 -3.1415

File: myGym/envs/robots/tiago/tiago_dual_mygym_rotslide.urdf (robot description, URDF)
Before this commit: robot tiago_dual_mygym, 37 links, 36 joints
Links:
- link endeffector: geometry visual cylinder length=0.07 radius=0.01
Joints:
- removed joint endeffector_gjoint
- added joint endeffector: type fixed, parent gripper, child endeffector, origin xyz=0.0 0.0 -0.20 rpy=0 0 -3.14

File: myGym/envs/robots/tiago/tiago_dual_mygym_rotslide2.urdf (robot description, URDF)
Before this commit: robot tiago_dual_mygym, 38 links, 37 joints
Links:
- link endeffector: geometry visual cylinder length=0.07 radius=0.01
Joints:
- removed joint endeffector_gjoint
- added joint endeffector: type fixed, parent gripper, child endeffector, origin xyz=0.0 0.0 -0.20 rpy=0 0 -3.14
