Commit message: tiago urdf updates - lift joint position and Rado fix the joint limits

File: myGym/envs/robots/tiago/tiago_dual_mygym.urdf (robot description, URDF)
Before this commit: robot tiago_dual_mygym, 37 links, 36 joints
Links:
- added link base_footprint2
- link arm_left_1_link: geometry visual mesh filename=package://tiago_description/meshes/arm/arm_1.stl scale=1 -1 -1
- link arm_right_2_link: geometry visual mesh filename=package://tiago_description/meshes/arm/arm_2.stl scale=1 1 1
- link arm_right_3_link: geometry visual mesh filename=package://tiago_description/meshes/arm/arm_3.stl scale=1 1 1
- link arm_right_4_link: geometry visual mesh filename=package://tiago_description/meshes/arm/arm_4.stl scale=1 1 1
- link arm_right_5_link: geometry visual mesh filename=package://tiago_description/meshes/arm/arm_5-wrist-2017.stl scale=1 1 1
- link arm_right_6_link: geometry visual mesh filename=package://tiago_description/meshes/arm/arm_6-wrist-2017.stl scale=1 1 1
- link arm_right_tool_link: geometry visual cylinder length=0.005 radius=0.005
- link base_footprint: mass 1 -> None
- link base_link: mass 28.26649 -> 20.26649
- link endeffector: mass 0.00 -> None
- link gripper_right_left_finger_link: geometry collision mesh filename=package://pal_gripper_description/meshes/gripper_finger_lin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; visual mesh filename=package://pal_gripper_description/meshes/gripper_finger_lin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
- link gripper_right_link: geometry visual mesh filename=package://pal_gripper_description/meshes/gripper_link.stl
- link gripper_right_right_finger_link: geometry collision mesh filename=package://pal_gripper_description/meshes/gripper_finger_lin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 scale=-1 -1 1; visual mesh filename=package://pal_gripper_description/meshes/gripper_finger_lin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 scale=-1 -1 1
- link head_1_link: geometry visual mesh filename=package://tiago_description/meshes/head/head_1.stl scale=1 1 1
- link head_2_link: geometry visual mesh filename=package://tiago_description/meshes/head/head_2.stl scale=1 1 1
- link torso_fixed_column_link: geometry visual box size=0.18 0.2 0.60
- link torso_lift_link: geometry collision mesh filename=package://tiago_dual_description/meshes/torso/torso_lift_du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 scale=1 1 1; visual mesh filename=package://tiago_dual_description/meshes/torso/torso_lift_du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 scale=1 1 1
- link wrist_right_ft_link: geometry visual cylinder length=0.0157 radius=0.0225
- link wrist_right_ft_tool_link: geometry visual cylinder length=0.00975 radius=0.025
Joints:
- removed joint torso_lift_pjoint
- added joint baseslide2_rjoint: type fixed, parent base_footprint, child base_footprint2, origin xyz=0. 0 0 rpy=0 0 0, axis 1 0 0, limit lower=-0.5 upper=0.4 effort=500 velocity=1
- added joint torso_lift_joint: type prismatic, parent torso_fixed_link, child torso_lift_link, origin xyz=0.0 0.0 0.61 rpy=0.0 0.0 0.0, axis 0 0 1, limit lower=0.0 upper=0.35 effort=2000 velocity=5
- joint arm_left_1_joint: limit lower=-1.1780972451 upper=1.57079632679 effort=43.0 velocity=1.95 -> lower=-1.1780972451 upper=1.57079632679 effort=43.0 velocity=10
- joint arm_right_2_rjoint: limit lower=-3.14 upper=0 effort=43.0 velocity=1.95 -> lower=-1.1780972450961724 upper=1.5707963267948966 effort=43.0 velocity=1.95; origin xyz=0.125 -0.0195 -0.031 rpy=-1.57079632679 1.57 0.0 -> xyz=0.125 -0.0195 -0.031 rpy=-1.5707963267948966 0.0 0.0
- joint arm_right_3_rjoint: limit lower=-0.785398163397 upper=3.92699081699 effort=26 velocity=2.35 -> lower=-0.7853981633974483 upper=3.9269908169872414 effort=26 velocity=2.35; origin xyz=0.0895 0.0 -0.0015 rpy=-1.57079632679 1.5707 1.57079632679 -> xyz=0.0895 0.0 -0.0015 rpy=-1.5707963267948966 0.0 1.5707963267948966
- joint baserot_rjoint: limit lower=-1.1780972451 upper=1.57079632679 effort=16 velocity=1.95 -> lower=-1.1780972451 upper=1.57079632679 effort=200 velocity=20
- joint baseslide_rjoint: limit lower=-0.5 upper=0.5 effort=16 velocity=0.05 -> lower=-0.7 upper=0.35 effort=500 velocity=1
- joint endeffector_gjoint: origin xyz=0.0 0.0 -0.20 rpy=0 0 -3.1415 -> xyz=0.0 0.0 -0.20 rpy=0 0 -1.57079632679

File: myGym/envs/robots/tiago/tiago_dual_mygym_rot.urdf (robot description, URDF)
Before this commit: robot tiago_dual_mygym, 37 links, 36 joints
Links:
- added link base_footprint2
- link arm_left_1_link: geometry visual mesh filename=package://tiago_description/meshes/arm/arm_1.stl scale=1 -1 -1
- link arm_right_2_link: geometry visual mesh filename=package://tiago_description/meshes/arm/arm_2.stl scale=1 1 1
- link arm_right_3_link: geometry visual mesh filename=package://tiago_description/meshes/arm/arm_3.stl scale=1 1 1
- link arm_right_4_link: geometry visual mesh filename=package://tiago_description/meshes/arm/arm_4.stl scale=1 1 1
- link arm_right_5_link: geometry visual mesh filename=package://tiago_description/meshes/arm/arm_5-wrist-2017.stl scale=1 1 1
- link arm_right_6_link: geometry visual mesh filename=package://tiago_description/meshes/arm/arm_6-wrist-2017.stl scale=1 1 1
- link arm_right_tool_link: geometry visual cylinder length=0.005 radius=0.005
- link base_footprint: mass 1 -> None
- link base_link: mass 28.26649 -> 20.26649
- link endeffector: mass 0.00 -> None
- link gripper_right_left_finger_link: geometry collision mesh filename=package://pal_gripper_description/meshes/gripper_finger_lin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; visual mesh filename=package://pal_gripper_description/meshes/gripper_finger_lin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
- link gripper_right_link: geometry visual mesh filename=package://pal_gripper_description/meshes/gripper_link.stl
- link gripper_right_right_finger_link: geometry collision mesh filename=package://pal_gripper_description/meshes/gripper_finger_lin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 scale=-1 -1 1; visual mesh filename=package://pal_gripper_description/meshes/gripper_finger_lin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 scale=-1 -1 1
- link head_1_link: geometry visual mesh filename=package://tiago_description/meshes/head/head_1.stl scale=1 1 1
- link head_2_link: geometry visual mesh filename=package://tiago_description/meshes/head/head_2.stl scale=1 1 1
- link torso_fixed_column_link: geometry visual box size=0.18 0.2 0.60
- link torso_lift_link: geometry collision mesh filename=package://tiago_dual_description/meshes/torso/torso_lift_du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 scale=1 1 1; visual mesh filename=package://tiago_dual_description/meshes/torso/torso_lift_du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 scale=1 1 1
- link wrist_right_ft_link: geometry visual cylinder length=0.0157 radius=0.0225
- link wrist_right_ft_tool_link: geometry visual cylinder length=0.00975 radius=0.025
Joints:
- removed joint torso_lift_pjoint
- added joint baseslide2_rjoint: type fixed, parent base_footprint, child base_footprint2, origin xyz=0. 0 0 rpy=0 0 0, axis 1 0 0, limit lower=-0.5 upper=0.4 effort=500 velocity=1
- added joint torso_lift_joint: type prismatic, parent torso_fixed_link, child torso_lift_link, origin xyz=0.0 0.0 0.61 rpy=0.0 0.0 0.0, axis 0 0 1, limit lower=0.0 upper=0.35 effort=2000 velocity=5
- joint arm_left_1_joint: limit lower=-1.1780972451 upper=1.57079632679 effort=43.0 velocity=1.95 -> lower=-1.1780972451 upper=1.57079632679 effort=43.0 velocity=10
- joint arm_right_2_rjoint: limit lower=-3.14 upper=0 effort=43.0 velocity=1.95 -> lower=-1.1780972450961724 upper=1.5707963267948966 effort=43.0 velocity=1.95; origin xyz=0.125 -0.0195 -0.031 rpy=-1.57079632679 1.57 0.0 -> xyz=0.125 -0.0195 -0.031 rpy=-1.5707963267948966 0.0 0.0
- joint arm_right_3_rjoint: limit lower=-0.785398163397 upper=3.92699081699 effort=26 velocity=2.35 -> lower=-0.7853981633974483 upper=3.9269908169872414 effort=26 velocity=2.35; origin xyz=0.0895 0.0 -0.0015 rpy=-1.57079632679 1.5707 1.57079632679 -> xyz=0.0895 0.0 -0.0015 rpy=-1.5707963267948966 0.0 1.5707963267948966
- joint baserot_rjoint: limit lower=-1.1780972451 upper=1.57079632679 effort=16 velocity=1.95 -> lower=-3.140972451 upper=3.140972451 effort=200 velocity=20
- joint baseslide_rjoint: limit lower=-0.5 upper=0.5 effort=16 velocity=0.05 -> lower=-0.7 upper=0.35 effort=500 velocity=1
- joint endeffector_gjoint: origin xyz=0.0 0.0 -0.20 rpy=0 0 -3.14 -> xyz=0.0 0.0 -0.20 rpy=0 0 -1.57079632679

File: myGym/envs/robots/tiago/tiago_dual_mygym_rotslide2.urdf (robot description, URDF)
Before this commit: robot tiago_dual_mygym, 38 links, 37 joints
Links:
- link arm_left_1_link: geometry visual mesh filename=package://tiago_description/meshes/arm/arm_1.stl scale=1 -1 -1
- link arm_right_2_link: geometry visual mesh filename=package://tiago_description/meshes/arm/arm_2.stl scale=1 1 1
- link arm_right_3_link: geometry visual mesh filename=package://tiago_description/meshes/arm/arm_3.stl scale=1 1 1
- link arm_right_4_link: geometry visual mesh filename=package://tiago_description/meshes/arm/arm_4.stl scale=1 1 1
- link arm_right_5_link: geometry visual mesh filename=package://tiago_description/meshes/arm/arm_5-wrist-2017.stl scale=1 1 1
- link arm_right_6_link: geometry visual mesh filename=package://tiago_description/meshes/arm/arm_6-wrist-2017.stl scale=1 1 1
- link arm_right_tool_link: geometry visual cylinder length=0.005 radius=0.005
- link base_footprint: mass 1 -> None
- link base_footprint2: mass 1 -> None
- link base_link: mass 28.26649 -> 20.26649
- link endeffector: mass 0.00 -> None
- link gripper_right_left_finger_link: geometry collision mesh filename=package://pal_gripper_description/meshes/gripper_finger_lin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; visual mesh filename=package://pal_gripper_description/meshes/gripper_finger_lin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
- link gripper_right_link: geometry visual mesh filename=package://pal_gripper_description/meshes/gripper_link.stl
- link gripper_right_right_finger_link: geometry collision mesh filename=package://pal_gripper_description/meshes/gripper_finger_lin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 scale=-1 -1 1; visual mesh filename=package://pal_gripper_description/meshes/gripper_finger_lin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 scale=-1 -1 1
- link head_1_link: geometry visual mesh filename=package://tiago_description/meshes/head/head_1.stl scale=1 1 1
- link head_2_link: geometry visual mesh filename=package://tiago_description/meshes/head/head_2.stl scale=1 1 1
- link torso_fixed_column_link: geometry visual box size=0.18 0.2 0.60
- link torso_lift_link: geometry collision mesh filename=package://tiago_dual_description/meshes/torso/torso_lift_du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 scale=1 1 1; visual mesh filename=package://tiago_dual_description/meshes/torso/torso_lift_du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 scale=1 1 1
- link wrist_right_ft_link: geometry visual cylinder length=0.0157 radius=0.0225
- link wrist_right_ft_tool_link: geometry visual cylinder length=0.00975 radius=0.025
Joints:
- removed joint baseslide_pjoint
- removed joint baseslide_pjoint2
- removed joint torso_lift_pjoint
- added joint baseslide2_rjoint: type prismatic, parent base_footprint, child base_footprint2, origin xyz=0. 0 0 rpy=0 0 0, axis 1 0 0, limit lower=-0.5 upper=0.4 effort=500 velocity=1
- added joint baseslide_rjoint: type prismatic, parent world, child base_footprint, origin xyz=0. 0 0 rpy=0 0 0, axis 0 1 0, limit lower=-0.7 upper=0.35 effort=500 velocity=1
- added joint torso_lift_joint: type prismatic, parent torso_fixed_link, child torso_lift_link, origin xyz=0.0 0.0 0.61 rpy=0.0 0.0 0.0, axis 0 0 1, limit lower=0.0 upper=0.35 effort=2000 velocity=5
- joint arm_left_1_joint: limit lower=-1.1780972451 upper=1.57079632679 effort=43.0 velocity=1.95 -> lower=-1.1780972451 upper=1.57079632679 effort=43.0 velocity=10
- joint arm_right_2_rjoint: limit lower=-3.14 upper=0 effort=43.0 velocity=1.95 -> lower=-1.1780972450961724 upper=1.5707963267948966 effort=43.0 velocity=1.95; origin xyz=0.125 -0.0195 -0.031 rpy=-1.57079632679 1.57 0.0 -> xyz=0.125 -0.0195 -0.031 rpy=-1.5707963267948966 0.0 0.0
- joint arm_right_3_rjoint: limit lower=-0.785398163397 upper=3.92699081699 effort=26 velocity=2.35 -> lower=-0.7853981633974483 upper=3.9269908169872414 effort=26 velocity=2.35; origin xyz=0.0895 0.0 -0.0015 rpy=-1.57079632679 1.5707 1.57079632679 -> xyz=0.0895 0.0 -0.0015 rpy=-1.5707963267948966 0.0 1.5707963267948966
- joint baserot_rjoint: limit lower=-1.1780972451 upper=1.57079632679 effort=16 velocity=1.95 -> lower=-3.140972451 upper=3.140972451 effort=200 velocity=20
- joint endeffector_gjoint: origin xyz=0.0 0.0 -0.20 rpy=0 0 -3.14 -> xyz=0.0 0.0 -0.20 rpy=0 0 -1.57079632679

Commit message: Fixed URDF for tiago dual

File: myGym/envs/robots/tiago/tiago_dual_mygym.urdf (robot description, URDF)
Before this commit: robot tiago_dual_mygym, 37 links, 36 joints
Joints:
- joint arm_right_2_rjoint: limit lower=-3.14 upper=0 effort=43.0 velocity=1.95 -> lower=-1.1780972450961724 upper=1.5707963267948966 effort=43.0 velocity=1.95; origin xyz=0.125 -0.0195 -0.031 rpy=-1.57079632679 1.57 0.0 -> xyz=0.125 -0.0195 -0.031 rpy=-1.5707963267948966 0.0 0.0
- joint arm_right_3_rjoint: limit lower=-0.785398163397 upper=3.92699081699 effort=26 velocity=2.35 -> lower=-0.7853981633974483 upper=3.9269908169872414 effort=26 velocity=2.35; origin xyz=0.0895 0.0 -0.0015 rpy=-1.57079632679 1.5707 1.57079632679 -> xyz=0.0895 0.0 -0.0015 rpy=-1.5707963267948966 0.0 1.5707963267948966
