Commit message: Merge branch 'PRAG' into ros

File: myGym/envs/robots/tiago/tiago_dual_mygym.urdf (robot description, URDF)
Before this commit: robot tiago_dual_mygym, 37 links, 36 joints
Links:
- added link base_footprint2
- link arm_left_1_link: geometry visual mesh filename=package://tiago_description/meshes/arm/arm_1.stl scale=1 -1 -1
- link arm_right_2_link: geometry visual mesh filename=package://tiago_description/meshes/arm/arm_2.stl scale=1 1 1
- link arm_right_3_link: geometry visual mesh filename=package://tiago_description/meshes/arm/arm_3.stl scale=1 1 1
- link arm_right_4_link: geometry visual mesh filename=package://tiago_description/meshes/arm/arm_4.stl scale=1 1 1
- link arm_right_5_link: geometry visual mesh filename=package://tiago_description/meshes/arm/arm_5-wrist-2017.stl scale=1 1 1
- link arm_right_6_link: geometry visual mesh filename=package://tiago_description/meshes/arm/arm_6-wrist-2017.stl scale=1 1 1
- link arm_right_tool_link: geometry visual cylinder length=0.005 radius=0.005
- link base_footprint: mass 1 -> None
- link base_link: mass 28.26649 -> 20.26649
- link endeffector: mass 0.00 -> None
- link gripper_right_left_finger_link: geometry collision mesh filename=package://pal_gripper_description/meshes/gripper_finger_lin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; visual mesh filename=package://pal_gripper_description/meshes/gripper_finger_lin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
- link gripper_right_link: geometry visual mesh filename=package://pal_gripper_description/meshes/gripper_link.stl
- link gripper_right_right_finger_link: geometry collision mesh filename=package://pal_gripper_description/meshes/gripper_finger_lin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 scale=-1 -1 1; visual mesh filename=package://pal_gripper_description/meshes/gripper_finger_lin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 scale=-1 -1 1
- link head_1_link: geometry visual mesh filename=package://tiago_description/meshes/head/head_1.stl scale=1 1 1
- link head_2_link: geometry visual mesh filename=package://tiago_description/meshes/head/head_2.stl scale=1 1 1
- link torso_fixed_column_link: geometry visual box size=0.18 0.2 0.60
- link torso_lift_link: geometry collision mesh filename=package://tiago_dual_description/meshes/torso/torso_lift_du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 scale=1 1 1; visual mesh filename=package://tiago_dual_description/meshes/torso/torso_lift_du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 scale=1 1 1
- link wrist_right_ft_link: geometry visual cylinder length=0.0157 radius=0.0225
- link wrist_right_ft_tool_link: geometry visual cylinder length=0.00975 radius=0.025
Joints:
- added joint baseslide2_rjoint: type fixed, parent base_footprint, child base_footprint2, origin xyz=0. 0 0 rpy=0 0 0, axis 1 0 0, limit lower=-0.5 upper=0.4 effort=500 velocity=1
- joint arm_left_1_joint: limit lower=-1.1780972451 upper=1.57079632679 effort=43.0 velocity=1.95 -> lower=-1.1780972451 upper=1.57079632679 effort=43.0 velocity=10
- joint baserot_rjoint: limit lower=-1.1780972451 upper=1.57079632679 effort=16 velocity=1.95 -> lower=-1.1780972451 upper=1.57079632679 effort=200 velocity=20
- joint baseslide_rjoint: limit lower=-0.5 upper=0.5 effort=16 velocity=0.05 -> lower=-0.7 upper=0.35 effort=500 velocity=1
- joint endeffector_gjoint: origin xyz=0.0 0.0 -0.20 rpy=0 0 0 -> xyz=0.0 0.0 -0.20 rpy=0 0 -1.57079632679
- joint torso_lift_joint: limit lower=0.349 upper=0.35 effort=2000 velocity=5 -> lower=0.0 upper=0.35 effort=2000 velocity=5; origin xyz=0.0 0.0 0.95 rpy=0.0 0.0 0.0 -> xyz=0.0 0.0 0.61 rpy=0.0 0.0 0.0; type fixed -> prismatic

File: myGym/envs/robots/tiago/tiago_dual_mygym_rot.urdf (robot description, URDF)
Before this commit: robot tiago_dual_mygym, 37 links, 36 joints
Links:
- added link base_footprint2
- link arm_left_2_link: geometry collision mesh filename=package://tiago_description/meshes/arm/arm_2_collision.dae scale=1 1 -1; visual mesh filename=package://tiago_description/meshes/arm/arm_2.stl scale=1 1 -1
- link arm_left_3_link: geometry collision mesh filename=package://tiago_description/meshes/arm/arm_3_collision.dae scale=1 1 -1; visual mesh filename=package://tiago_description/meshes/arm/arm_3.stl scale=1 1 -1
- link arm_left_4_link: geometry collision mesh filename=package://tiago_description/meshes/arm/arm_4_collision.dae scale=-1 -1 -1; visual mesh filename=package://tiago_description/meshes/arm/arm_4.stl scale=-1 -1 -1
- link arm_left_5_link: geometry collision mesh filename=package://tiago_description/meshes/arm/arm_5_collision-wris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 scale=-1 -1 -1; visual mesh filename=package://tiago_description/meshes/arm/arm_5-wrist-2017.stl scale=-1 -1 -1
- link arm_left_6_link: geometry collision mesh filename=package://tiago_description/meshes/arm/arm_6_collision-wris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 scale=-1 1 1; visual mesh filename=package://tiago_description/meshes/arm/arm_6-wrist-2017.stl scale=-1 1 1
- link arm_left_tool_link: geometry collision cylinder length=0.005 radius=0.005; visual cylinder length=0.005 radius=0.005
- link arm_right_2_link: geometry visual mesh filename=package://tiago_description/meshes/arm/arm_2.stl scale=1 1 1
- link arm_right_3_link: geometry visual mesh filename=package://tiago_description/meshes/arm/arm_3.stl scale=1 1 1
- link arm_right_4_link: geometry visual mesh filename=package://tiago_description/meshes/arm/arm_4.stl scale=1 1 1
- link arm_right_5_link: geometry visual mesh filename=package://tiago_description/meshes/arm/arm_5-wrist-2017.stl scale=1 1 1
- link arm_right_6_link: geometry visual mesh filename=package://tiago_description/meshes/arm/arm_6-wrist-2017.stl scale=1 1 1
- link arm_right_tool_link: geometry visual cylinder length=0.005 radius=0.005
- link base_footprint: mass 1 -> None
- link base_link: mass 28.26649 -> 20.26649
- link endeffector: mass 0.00 -> None
- link gripper_left_left_finger_link: geometry collision box size=0.01 0.05 0.11; visual mesh filename=package://pal_gripper_description/meshes/gripper_finger_lin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
- link gripper_left_link: geometry collision mesh filename=package://pal_gripper_description/meshes/gripper_link_colli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; visual mesh filename=package://pal_gripper_description/meshes/gripper_link.stl
- link gripper_left_right_finger_link: geometry collision box size=0.01 0.05 0.11; visual mesh filename=package://pal_gripper_description/meshes/gripper_finger_lin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 scale=-1 -1 1
- link gripper_right_left_finger_link: geometry collision mesh filename=package://pal_gripper_description/meshes/gripper_finger_lin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; visual mesh filename=package://pal_gripper_description/meshes/gripper_finger_lin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
- link gripper_right_link: geometry visual mesh filename=package://pal_gripper_description/meshes/gripper_link.stl
- link gripper_right_right_finger_link: geometry collision mesh filename=package://pal_gripper_description/meshes/gripper_finger_lin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 scale=-1 -1 1; visual mesh filename=package://pal_gripper_description/meshes/gripper_finger_lin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 scale=-1 -1 1
- link head_1_link: geometry visual mesh filename=package://tiago_description/meshes/head/head_1.stl scale=1 1 1
- link head_2_link: geometry visual mesh filename=package://tiago_description/meshes/head/head_2.stl scale=1 1 1
- link torso_fixed_column_link: geometry visual box size=0.18 0.2 0.60
- link wrist_left_ft_link: geometry collision cylinder length=0.0157 radius=0.0225; visual cylinder length=0.0157 radius=0.0225
- link wrist_left_ft_tool_link: geometry collision cylinder length=0.00975 radius=0.025; visual cylinder length=0.00975 radius=0.025
- link wrist_right_ft_link: geometry visual cylinder length=0.0157 radius=0.0225
- link wrist_right_ft_tool_link: geometry visual cylinder length=0.00975 radius=0.025
Joints:
- added joint baseslide2_rjoint: type fixed, parent base_footprint, child base_footprint2, origin xyz=0. 0 0 rpy=0 0 0, axis 1 0 0, limit lower=-0.5 upper=0.4 effort=500 velocity=1
- joint arm_left_1_joint: limit lower=-1.1780972451 upper=1.57079632679 effort=43.0 velocity=1.95 -> lower=-1.1780972451 upper=1.57079632679 effort=43.0 velocity=10
- joint arm_right_2_rjoint: limit lower=-3.14 upper=0 effort=43.0 velocity=1.95 -> lower=-1.1780972450961724 upper=1.5707963267948966 effort=43.0 velocity=1.95; origin xyz=0.125 -0.0195 -0.031 rpy=-1.57079632679 1.57 0.0 -> xyz=0.125 -0.0195 -0.031 rpy=-1.5707963267948966 0.0 0.0
- joint arm_right_3_rjoint: limit lower=-0.785398163397 upper=3.92699081699 effort=26 velocity=2.35 -> lower=-0.7853981633974483 upper=3.9269908169872414 effort=26 velocity=2.35; origin xyz=0.0895 0.0 -0.0015 rpy=-1.57079632679 1.5707 1.57079632679 -> xyz=0.0895 0.0 -0.0015 rpy=-1.5707963267948966 0.0 1.5707963267948966
- joint baserot_rjoint: limit lower=-1.9780972451 upper=3.14159265359 effort=100 velocity=2 -> lower=-3.140972451 upper=3.140972451 effort=200 velocity=20; origin xyz=0 0 0 rpy=0 0 0 -> xyz=0 0 0.1 rpy=0 0 0
- joint baseslide_rjoint: limit lower=-0.5 upper=0.5 effort=500 velocity=1 -> lower=-0.7 upper=0.35 effort=500 velocity=1
- joint endeffector_gjoint: origin xyz=0.0 0.0 -0.23 rpy=0 0 0 -> xyz=0.0 0.0 -0.20 rpy=0 0 -1.57079632679
- joint gripper_right_left_finger_gjoint: limit lower=0.044 upper=0.045 effort=16 velocity=10 -> lower=0.0 upper=0.045 effort=16 velocity=10
- joint gripper_right_right_finger_gjoint: limit lower=0.044 upper=0.045 effort=16 velocity=10 -> lower=0.0 upper=0.045 effort=16 velocity=10
- joint torso_lift_joint: limit lower=0.349 upper=0.35 effort=2000 velocity=5 -> lower=0.0 upper=0.35 effort=2000 velocity=5; origin xyz=0.0 0.0 0.95 rpy=0.0 0.0 0.0 -> xyz=0.0 0.0 0.61 rpy=0.0 0.0 0.0; type fixed -> prismatic

File: myGym/envs/robots/tiago/tiago_dual_mygym_rotslide.urdf (robot description, URDF)
Before this commit: robot tiago_dual_mygym, 37 links, 36 joints
Links:
- added link base_footprint2
- link arm_left_2_link: geometry collision mesh filename=package://tiago_description/meshes/arm/arm_2_collision.dae scale=1 1 -1; visual mesh filename=package://tiago_description/meshes/arm/arm_2.stl scale=1 1 -1
- link arm_left_3_link: geometry collision mesh filename=package://tiago_description/meshes/arm/arm_3_collision.dae scale=1 1 -1; visual mesh filename=package://tiago_description/meshes/arm/arm_3.stl scale=1 1 -1
- link arm_left_4_link: geometry collision mesh filename=package://tiago_description/meshes/arm/arm_4_collision.dae scale=-1 -1 -1; visual mesh filename=package://tiago_description/meshes/arm/arm_4.stl scale=-1 -1 -1
- link arm_left_5_link: geometry collision mesh filename=package://tiago_description/meshes/arm/arm_5_collision-wris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 scale=-1 -1 -1; visual mesh filename=package://tiago_description/meshes/arm/arm_5-wrist-2017.stl scale=-1 -1 -1
- link arm_left_6_link: geometry collision mesh filename=package://tiago_description/meshes/arm/arm_6_collision-wris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 scale=-1 1 1; visual mesh filename=package://tiago_description/meshes/arm/arm_6-wrist-2017.stl scale=-1 1 1
- link arm_left_tool_link: geometry collision cylinder length=0.005 radius=0.005; visual cylinder length=0.005 radius=0.005
- link arm_right_2_link: geometry visual mesh filename=package://tiago_description/meshes/arm/arm_2.stl scale=1 1 1
- link arm_right_3_link: geometry visual mesh filename=package://tiago_description/meshes/arm/arm_3.stl scale=1 1 1
- link arm_right_4_link: geometry visual mesh filename=package://tiago_description/meshes/arm/arm_4.stl scale=1 1 1
- link arm_right_5_link: geometry visual mesh filename=package://tiago_description/meshes/arm/arm_5-wrist-2017.stl scale=1 1 1
- link arm_right_6_link: geometry visual mesh filename=package://tiago_description/meshes/arm/arm_6-wrist-2017.stl scale=1 1 1
- link arm_right_tool_link: geometry visual cylinder length=0.005 radius=0.005
- link base_footprint: mass 1 -> None
- link base_link: mass 28.26649 -> 20.26649
- link endeffector: mass 0.00 -> None
- link gripper_left_left_finger_link: geometry collision box size=0.01 0.05 0.11; visual mesh filename=package://pal_gripper_description/meshes/gripper_finger_lin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
- link gripper_left_link: geometry collision mesh filename=package://pal_gripper_description/meshes/gripper_link_colli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; visual mesh filename=package://pal_gripper_description/meshes/gripper_link.stl
- link gripper_left_right_finger_link: geometry collision box size=0.01 0.05 0.11; visual mesh filename=package://pal_gripper_description/meshes/gripper_finger_lin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 scale=-1 -1 1
- link gripper_right_left_finger_link: geometry collision mesh filename=package://pal_gripper_description/meshes/gripper_finger_lin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; visual mesh filename=package://pal_gripper_description/meshes/gripper_finger_lin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
- link gripper_right_link: geometry visual mesh filename=package://pal_gripper_description/meshes/gripper_link.stl
- link gripper_right_right_finger_link: geometry collision mesh filename=package://pal_gripper_description/meshes/gripper_finger_lin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 scale=-1 -1 1; visual mesh filename=package://pal_gripper_description/meshes/gripper_finger_lin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 scale=-1 -1 1
- link head_1_link: geometry visual mesh filename=package://tiago_description/meshes/head/head_1.stl scale=1 1 1
- link head_2_link: geometry visual mesh filename=package://tiago_description/meshes/head/head_2.stl scale=1 1 1
- link torso_fixed_column_link: geometry visual box size=0.18 0.2 0.60
- link wrist_left_ft_link: geometry collision cylinder length=0.0157 radius=0.0225; visual cylinder length=0.0157 radius=0.0225
- link wrist_left_ft_tool_link: geometry collision cylinder length=0.00975 radius=0.025; visual cylinder length=0.00975 radius=0.025
- link wrist_right_ft_link: geometry visual cylinder length=0.0157 radius=0.0225
- link wrist_right_ft_tool_link: geometry visual cylinder length=0.00975 radius=0.025
Joints:
- added joint baseslide2_rjoint: type fixed, parent base_footprint, child base_footprint2, origin xyz=0. 0 0 rpy=0 0 0, axis 1 0 0, limit lower=-0.5 upper=0.4 effort=500 velocity=1
- joint arm_left_1_joint: limit lower=-1.1780972451 upper=1.57079632679 effort=43.0 velocity=1.95 -> lower=-1.1780972451 upper=1.57079632679 effort=43.0 velocity=10
- joint arm_right_2_rjoint: limit lower=-3.14 upper=0 effort=43.0 velocity=1.95 -> lower=-1.1780972450961724 upper=1.5707963267948966 effort=43.0 velocity=1.95; origin xyz=0.125 -0.0195 -0.031 rpy=-1.57079632679 1.57 0.0 -> xyz=0.125 -0.0195 -0.031 rpy=-1.5707963267948966 0.0 0.0
- joint arm_right_3_rjoint: limit lower=-0.785398163397 upper=3.92699081699 effort=26 velocity=2.35 -> lower=-0.7853981633974483 upper=3.9269908169872414 effort=26 velocity=2.35; origin xyz=0.0895 0.0 -0.0015 rpy=-1.57079632679 1.5707 1.57079632679 -> xyz=0.0895 0.0 -0.0015 rpy=-1.5707963267948966 0.0 1.5707963267948966
- joint baserot_rjoint: limit lower=-1.9780972451 upper=3.14159265359 effort=100 velocity=2 -> lower=-3.140972451 upper=3.140972451 effort=200 velocity=20; origin xyz=0 0 0 rpy=0 0 0 -> xyz=0 0 0.1 rpy=0 0 0
- joint baseslide_rjoint: limit lower=-0.5 upper=0.5 effort=500 velocity=1 -> lower=-0.7 upper=0.35 effort=500 velocity=1
- joint endeffector_gjoint: origin xyz=0.0 0.0 -0.23 rpy=0 0 0 -> xyz=0.0 0.0 -0.20 rpy=0 0 -1.57079632679
- joint gripper_right_left_finger_gjoint: limit lower=0.044 upper=0.045 effort=16 velocity=10 -> lower=0.0 upper=0.045 effort=16 velocity=10
- joint gripper_right_right_finger_gjoint: limit lower=0.044 upper=0.045 effort=16 velocity=10 -> lower=0.0 upper=0.045 effort=16 velocity=10
- joint torso_lift_joint: limit lower=0.349 upper=0.35 effort=2000 velocity=5 -> lower=0.0 upper=0.35 effort=2000 velocity=5; origin xyz=0.0 0.0 0.95 rpy=0.0 0.0 0.0 -> xyz=0.0 0.0 0.61 rpy=0.0 0.0 0.0; type fixed -> prismatic

File: myGym/envs/robots/tiago/tiago_dual_mygym_rotslide2.urdf (robot description, URDF)
Before this commit: robot tiago_dual_mygym, 38 links, 37 joints
Links:
- link arm_left_2_link: geometry collision mesh filename=package://tiago_description/meshes/arm/arm_2_collision.dae scale=1 1 -1; visual mesh filename=package://tiago_description/meshes/arm/arm_2.stl scale=1 1 -1
- link arm_left_3_link: geometry collision mesh filename=package://tiago_description/meshes/arm/arm_3_collision.dae scale=1 1 -1; visual mesh filename=package://tiago_description/meshes/arm/arm_3.stl scale=1 1 -1
- link arm_left_4_link: geometry collision mesh filename=package://tiago_description/meshes/arm/arm_4_collision.dae scale=-1 -1 -1; visual mesh filename=package://tiago_description/meshes/arm/arm_4.stl scale=-1 -1 -1
- link arm_left_5_link: geometry collision mesh filename=package://tiago_description/meshes/arm/arm_5_collision-wris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 scale=-1 -1 -1; visual mesh filename=package://tiago_description/meshes/arm/arm_5-wrist-2017.stl scale=-1 -1 -1
- link arm_left_6_link: geometry collision mesh filename=package://tiago_description/meshes/arm/arm_6_collision-wris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 scale=-1 1 1; visual mesh filename=package://tiago_description/meshes/arm/arm_6-wrist-2017.stl scale=-1 1 1
- link arm_left_tool_link: geometry collision cylinder length=0.005 radius=0.005; visual cylinder length=0.005 radius=0.005
- link arm_right_2_link: geometry visual mesh filename=package://tiago_description/meshes/arm/arm_2.stl scale=1 1 1
- link arm_right_3_link: geometry visual mesh filename=package://tiago_description/meshes/arm/arm_3.stl scale=1 1 1
- link arm_right_4_link: geometry visual mesh filename=package://tiago_description/meshes/arm/arm_4.stl scale=1 1 1
- link arm_right_5_link: geometry visual mesh filename=package://tiago_description/meshes/arm/arm_5-wrist-2017.stl scale=1 1 1
- link arm_right_6_link: geometry visual mesh filename=package://tiago_description/meshes/arm/arm_6-wrist-2017.stl scale=1 1 1
- link arm_right_tool_link: geometry visual cylinder length=0.005 radius=0.005
- link base_footprint: mass 1 -> None
- link base_footprint2: mass 1 -> None
- link base_link: mass 28.26649 -> 20.26649
- link endeffector: mass 0.00 -> None
- link gripper_left_left_finger_link: geometry collision box size=0.01 0.05 0.11; visual mesh filename=package://pal_gripper_description/meshes/gripper_finger_lin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
- link gripper_left_link: geometry collision mesh filename=package://pal_gripper_description/meshes/gripper_link_colli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; visual mesh filename=package://pal_gripper_description/meshes/gripper_link.stl
- link gripper_left_right_finger_link: geometry collision box size=0.01 0.05 0.11; visual mesh filename=package://pal_gripper_description/meshes/gripper_finger_lin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 scale=-1 -1 1
- link gripper_right_left_finger_link: geometry collision mesh filename=package://pal_gripper_description/meshes/gripper_finger_lin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; visual mesh filename=package://pal_gripper_description/meshes/gripper_finger_lin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
- link gripper_right_link: geometry visual mesh filename=package://pal_gripper_description/meshes/gripper_link.stl
- link gripper_right_right_finger_link: geometry collision mesh filename=package://pal_gripper_description/meshes/gripper_finger_lin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 scale=-1 -1 1; visual mesh filename=package://pal_gripper_description/meshes/gripper_finger_lin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 scale=-1 -1 1
- link head_1_link: geometry visual mesh filename=package://tiago_description/meshes/head/head_1.stl scale=1 1 1
- link head_2_link: geometry visual mesh filename=package://tiago_description/meshes/head/head_2.stl scale=1 1 1
- link torso_fixed_column_link: geometry visual box size=0.18 0.2 0.60
- link wrist_left_ft_link: geometry collision cylinder length=0.0157 radius=0.0225; visual cylinder length=0.0157 radius=0.0225
- link wrist_left_ft_tool_link: geometry collision cylinder length=0.00975 radius=0.025; visual cylinder length=0.00975 radius=0.025
- link wrist_right_ft_link: geometry visual cylinder length=0.0157 radius=0.0225
- link wrist_right_ft_tool_link: geometry visual cylinder length=0.00975 radius=0.025
Joints:
- joint arm_left_1_joint: limit lower=-1.1780972451 upper=1.57079632679 effort=43.0 velocity=1.95 -> lower=-1.1780972451 upper=1.57079632679 effort=43.0 velocity=10
- joint arm_right_2_rjoint: limit lower=-3.14 upper=0 effort=43.0 velocity=1.95 -> lower=-1.1780972450961724 upper=1.5707963267948966 effort=43.0 velocity=1.95; origin xyz=0.125 -0.0195 -0.031 rpy=-1.57079632679 1.57 0.0 -> xyz=0.125 -0.0195 -0.031 rpy=-1.5707963267948966 0.0 0.0
- joint arm_right_3_rjoint: limit lower=-0.785398163397 upper=3.92699081699 effort=26 velocity=2.35 -> lower=-0.7853981633974483 upper=3.9269908169872414 effort=26 velocity=2.35; origin xyz=0.0895 0.0 -0.0015 rpy=-1.57079632679 1.5707 1.57079632679 -> xyz=0.0895 0.0 -0.0015 rpy=-1.5707963267948966 0.0 1.5707963267948966
- joint baserot_rjoint: limit lower=-1.9780972451 upper=3.14159265359 effort=100 velocity=2 -> lower=-3.140972451 upper=3.140972451 effort=200 velocity=20; origin xyz=0 0 0 rpy=0 0 0 -> xyz=0 0 0.1 rpy=0 0 0
- joint endeffector_gjoint: origin xyz=0.0 0.0 -0.23 rpy=0 0 0 -> xyz=0.0 0.0 -0.20 rpy=0 0 -1.57079632679
- joint gripper_right_left_finger_gjoint: limit lower=0.044 upper=0.045 effort=16 velocity=10 -> lower=0.0 upper=0.045 effort=16 velocity=10
- joint gripper_right_right_finger_gjoint: limit lower=0.044 upper=0.045 effort=16 velocity=10 -> lower=0.0 upper=0.045 effort=16 velocity=10
- joint torso_lift_joint: limit lower=0.349 upper=0.35 effort=2000 velocity=5 -> lower=0.0 upper=0.35 effort=2000 velocity=5; origin xyz=0.0 0.0 0.95 rpy=0.0 0.0 0.0 -> xyz=0.0 0.0 0.61 rpy=0.0 0.0 0.0; type fixed -> prismatic

Commit message: tiago end effoctor poitioning - WIP

File: myGym/envs/robots/tiago/tiago_dual_mygym.urdf (robot description, URDF)
Before this commit: robot tiago_dual_mygym, 38 links, 37 joints
Links:
- link endeffector: mass None -> 0.0000332; geometry visual cylinder length=0.05 radius=0.002
Joints:
- removed joint endeffector_gjoint
- added joint endeffector_joint: type fixed, parent gripper, child endeffector, origin xyz=0.0 0.0 -0.20 rpy=0 0 -1.57

File: myGym/envs/robots/tiago/tiago_dual_mygym_rotslide2.urdf (robot description, URDF)
Before this commit: robot tiago_dual_mygym, 38 links, 37 joints
Links:
- link endeffector: mass None -> 0.0000332; geometry visual cylinder length=0.05 radius=0.002
Joints:
- removed joint endeffector_gjoint
- added joint endeffector_joint: type fixed, parent gripper, child endeffector, origin xyz=0.0 0.0 -0.20 rpy=0 0 0
