Commit message: oraculum on new tiago urdfs works
(cherry picked from commit d98c6fe710e93667a83947f9b26ce4e8e675f7a0)

File: myGym/envs/robots/tiago/tiago_dual_mygym.urdf (robot description, URDF)
Before this commit: robot tiago_dual_mygym, 38 links, 37 joints
Joints:
- removed joint torso_lift_joint
- added joint torso_lift_rjoint: type prismatic, parent torso_fixed_link, child torso_lift_link, origin xyz=0.0 0.0 0.61 rpy=0.0 0.0 0.0, axis 0 0 1, limit lower=0.0 upper=0.35 effort=2000 velocity=5
- joint endeffector_joint: origin xyz=0.0 0.0 -0.20 rpy=0 0 -1.57 -> xyz=0.0 0.0 -0.20 rpy=0 0 -3.1415

File: myGym/envs/robots/tiago/tiago_dual_mygym_rot.urdf (robot description, URDF)
Before this commit: robot tiago_dual_mygym, 38 links, 37 joints
Joints:
- removed joint torso_lift_joint
- added joint endeffector_joint: type fixed, parent gripper, child endeffector, origin xyz=0.0 0.0 -0.20 rpy=0 0 -3.1415
- added joint torso_lift_rjoint: type prismatic, parent torso_fixed_link, child torso_lift_link, origin xyz=0.0 0.0 0.61 rpy=0.0 0.0 0.0, axis 0 0 1, limit lower=0.0 upper=0.35 effort=2000 velocity=5

File: myGym/envs/robots/tiago/tiago_dual_mygym_rotslide.urdf (robot description, URDF)
Before this commit: robot tiago_dual_mygym, 38 links, 37 joints
Joints:
- removed joint torso_lift_joint
- added joint endeffector_joint: type fixed, parent gripper, child endeffector, origin xyz=0.0 0.0 -0.20 rpy=0 0 -3.1415
- added joint torso_lift_rjoint: type prismatic, parent torso_fixed_link, child torso_lift_link, origin xyz=0.0 0.0 0.61 rpy=0.0 0.0 0.0, axis 0 0 1, limit lower=0.0 upper=0.35 effort=2000 velocity=5

File: myGym/envs/robots/tiago/tiago_dual_mygym_rotslide2.urdf (robot description, URDF)
Before this commit: robot tiago_dual_mygym, 38 links, 37 joints
Joints:
- removed joint torso_lift_joint
- added joint torso_lift_rjoint: type prismatic, parent torso_fixed_link, child torso_lift_link, origin xyz=0.0 0.0 0.61 rpy=0.0 0.0 0.0, axis 0 0 1, limit lower=0.0 upper=0.35 effort=2000 velocity=5
- joint endeffector_joint: origin xyz=0.0 0.0 -0.20 rpy=0 0 0 -> xyz=0.0 0.0 -0.20 rpy=0 0 -3.1415
