Commit message: absolute gripper bug in test.py fixed

File: myGym/envs/robots/tiago/tiago_dual_mygym_fix.urdf (robot description, URDF)
Before this commit: robot tiago_dual_mygym, 37 links, 36 joints
Joints:
- joint torso_lift_rjoint: limit lower=0.175 upper=0.175 effort=2000 velocity=5 -> lower=0.175 upper=0.1751 effort=2000 velocity=5

Commit message: camera origin for tiago fix

File: myGym/envs/robots/tiago/tiago_dual_mygym_fix.urdf (robot description, URDF)
Before this commit: robot tiago_dual_mygym, 40 links, 39 joints
Links:
- added link camera_origin; visual sphere radius=0.005
Joints:
- added joint camera_origin_joint: type fixed, parent head_2_link, child camera_origin, origin xyz=0.11 0.08 0.0 rpy=0 0 0
