Commit message: tiago reach with joints working

File: myGym/envs/robots/tiago/tiago_pal_gripper.urdf (robot description, URDF)
Before this commit: robot tiago, 49 links, 48 joints
Links:
- removed link xtion_orbbec_aux_joint_frame
- added link xtion_orbbec_aux_rjoint_frame, mass 0.001
Joints:
- removed joint arm_1_joint
- removed joint arm_2_joint
- removed joint arm_3_joint
- removed joint arm_4_joint
- removed joint arm_5_joint
- removed joint arm_6_joint
- removed joint arm_7_joint
- removed joint arm_tool_joint
- removed joint base_antenna_left_joint
- removed joint base_antenna_right_joint
- removed joint base_footprint_joint
- removed joint base_imu_joint
- removed joint base_laser_joint
- removed joint base_sonar_01_joint
- removed joint base_sonar_02_joint
- removed joint base_sonar_03_joint
- removed joint caster_back_left_1_joint
- removed joint caster_back_left_2_joint
- removed joint caster_back_right_1_joint
- removed joint caster_back_right_2_joint
- removed joint caster_front_left_1_joint
- removed joint caster_front_left_2_joint
- removed joint caster_front_right_1_joint
- removed joint caster_front_right_2_joint
- removed joint cover_joint
- removed joint endeffector_joint
- removed joint gripper_grasping_frame_joint
- removed joint gripper_joint
- removed joint gripper_left_finger_joint
- removed joint gripper_right_finger_joint
- removed joint gripper_tool_joint
- removed joint head_1_joint
- removed joint head_2_joint
- removed joint rgbd_laser_joint
- removed joint suspension_left_joint
- removed joint suspension_right_joint
- removed joint torso_fixed_column_joint
- removed joint torso_fixed_joint
- removed joint torso_lift_joint
- removed joint wheel_left_joint
- removed joint wheel_right_joint
- removed joint xtion_depth_joint
- removed joint xtion_depth_optical_joint
- removed joint xtion_joint
- removed joint xtion_optical_joint
- removed joint xtion_orbbec_aux_joint
- removed joint xtion_rgb_joint
- removed joint xtion_rgb_optical_joint
- added joint arm_1_rjoint: type revolute, parent torso_lift_link, child arm_1_link, origin xyz=0.15505 0.014 -0.151 rpy=0 0 -1.57079632679, axis 0 0 1, limit lower=0.0 upper=2.74889357189 effort=43.0 velocity=1.95
- added joint arm_2_rjoint: type revolute, parent arm_1_link, child arm_2_link, origin xyz=0.125 0.0195 -0.031 rpy=1.57079632679 0.0 0.0, axis 0 0 1, limit lower=-1.57079632679 upper=1.0908307825 effort=43.0 velocity=1.95
- added joint arm_3_rjoint: type revolute, parent arm_2_link, child arm_3_link, origin xyz=0.0895 0.0 -0.0015 rpy=-1.57079632679 0.0 1.57079632679, axis 0 0 1, limit lower=-3.53429173529 upper=1.57079632679 effort=26 velocity=2.35
- added joint arm_4_rjoint: type revolute, parent arm_3_link, child arm_4_link, origin xyz=-0.02 -0.027 -0.222 rpy=-1.57079632679 -1.57079632679 0.0, axis 0 0 1, limit lower=-0.392699081699 upper=2.35619449019 effort=26 velocity=2.35
- added joint arm_5_rjoint: type revolute, parent arm_4_link, child arm_5_link, origin xyz=-0.162 0.02 0.027 rpy=1.57079632679 -1.57079632679 -1.57079632679, axis 0 0 1, limit lower=-2.09439510239 upper=2.09439510239 effort=3 velocity=1.95
- added joint arm_6_rjoint: type revolute, parent arm_5_link, child arm_6_link, origin xyz=0 0 0.15 rpy=0.0 -1.57079632679 -1.57079632679, axis 0 0 1, limit lower=-1.41371669412 upper=1.41371669412 effort=6.6 velocity=1.76
- added joint arm_7_rjoint: type revolute, parent arm_6_link, child arm_7_link, origin xyz=0 0 0 rpy=1.57079632679 0.0 1.57079632679, axis 0 0 1, limit lower=-2.09439510239 upper=2.09439510239 effort=6.6 velocity=1.76
- added joint arm_tool_rjoint: type fixed, parent arm_7_link, child arm_tool_link, origin xyz=0 0 0.0573 rpy=1.57079632679 -1.57079632679 3.14159265359
- added joint base_antenna_left_rjoint: type fixed, parent base_link, child base_antenna_left_link, origin xyz=-0.201 0.1062 0.195 rpy=0 0 0
- added joint base_antenna_right_rjoint: type fixed, parent base_link, child base_antenna_right_link, origin xyz=-0.201 -0.1062 0.195 rpy=0 0 0
- added joint base_footprint_rjoint: type fixed, parent base_footprint, child base_link, origin xyz=0 0 0.0985 rpy=0 0 0
- added joint base_imu_rjoint: type fixed, parent base_link, child base_imu_link, origin xyz=0.10171 0 0.11282 rpy=0 0 -1.57079632679
- added joint base_laser_gjoint: type fixed, parent base_link, child base_laser_link, origin xyz=0.202 0.0 -0.004 rpy=0 0 0, axis 0 1 0
- added joint base_sonar_01_rjoint: type fixed, parent base_link, child base_sonar_01_link, origin xyz=-0.183 -0.183 0.173 rpy=0 0 3.92699081699, axis 0 0 1
- added joint base_sonar_02_rjoint: type fixed, parent base_link, child base_sonar_02_link, origin xyz=-0.259 0.0 0.173 rpy=0 0 3.14159265359, axis 0 0 1
- added joint base_sonar_03_rjoint: type fixed, parent base_link, child base_sonar_03_link, origin xyz=-0.183 0.183 0.173 rpy=0 0 2.35619449019, axis 0 0 1
- added joint caster_back_left_1_rjoint: type fixed, parent base_link, child caster_back_left_1_link, origin xyz=-0.1735 0.102 -0.0335 rpy=0 0 0, axis 0 0 1
- added joint caster_back_left_2_rjoint: type fixed, parent caster_back_left_1_link, child caster_back_left_2_link, origin xyz=-0.016 0.0000 -0.040 rpy=-1.57079632679 0 0, axis 0 0 1
- added joint caster_back_right_1_rjoint: type fixed, parent base_link, child caster_back_right_1_link, origin xyz=-0.1735 -0.102 -0.0335 rpy=0 0 0, axis 0 0 1
- added joint caster_back_right_2_rjoint: type fixed, parent caster_back_right_1_link, child caster_back_right_2_link, origin xyz=-0.016 0.0000 -0.040 rpy=-1.57079632679 0 0, axis 0 0 1
- added joint caster_front_left_1_rjoint: type fixed, parent base_link, child caster_front_left_1_link, origin xyz=0.1695 0.102 -0.0335 rpy=0 0 0, axis 0 0 1
- added joint caster_front_left_2_rjoint: type fixed, parent caster_front_left_1_link, child caster_front_left_2_link, origin xyz=-0.016 0.0000 -0.040 rpy=-1.57079632679 0 0, axis 0 0 1
- added joint caster_front_right_1_rjoint: type fixed, parent base_link, child caster_front_right_1_link, origin xyz=0.1695 -0.102 -0.0335 rpy=0 0 0, axis 0 0 1
- added joint caster_front_right_2_rjoint: type fixed, parent caster_front_right_1_link, child caster_front_right_2_link, origin xyz=-0.016 0.0000 -0.040 rpy=-1.57079632679 0 0, axis 0 0 1
- added joint cover_rjoint: type fixed, parent base_footprint, child base_cover_link, origin xyz=0 0 0.13 rpy=0 0 0
- added joint endeffector_gjoint: type fixed, parent gripper, child endeffector, origin xyz=0 0.0 0.1 rpy=0 0 0
- added joint gripper_grasping_frame_rjoint: type fixed, parent gripper, child gripper_grasping_frame, origin xyz=0 0 -0.12 rpy=-1.5708 1.5708 0
- added joint gripper_left_finger_rjoint: type prismatic, parent gripper, child gripper_left_finger_link, origin xyz=0. 0 0 rpy=0 0 0, axis -1 0 0, limit lower=0 upper=0.045 effort=16 velocity=0.05
- added joint gripper_right_finger_rjoint: type prismatic, parent gripper, child gripper_right_finger_link, origin xyz=0. 0 0 rpy=0 0 0, axis 1 0 0, limit lower=0.0 upper=0.045 effort=16 velocity=0.05
- added joint gripper_rjoint: type fixed, parent arm_tool_link, child gripper, origin xyz=0.01 0 0 rpy=1.57079632679 1.57079632679 -1.57079632679, axis 0 0 0
- added joint gripper_tool_rjoint: type fixed, parent arm_tool_link, child gripper_tool_link, origin xyz=0.01 0 0 rpy=1.57079632679 1.57079632679 -1.57079632679, axis 0 0 0
- added joint head_1_rjoint: type fixed, parent torso_lift_link, child head_1_link, origin xyz=0.182 0.0 0.0 rpy=0 0 0, axis 0 0 1, limit lower=-1.308996939 upper=1.308996939 effort=5.197 velocity=3.0
- added joint head_2_rjoint: type fixed, parent head_1_link, child head_2_link, origin xyz=0.005 0.0 0.098 rpy=1.57079632679 0 0, axis 0 0 1, limit lower=-1.0471975512 upper=0.785398163397 effort=2.77 velocity=3.0
- added joint rgbd_laser_rjoint: type fixed, parent base_footprint, child rgbd_laser_link, origin xyz=-0.9 0 0 rpy=0 0 0
- added joint suspension_left_rjoint: type fixed, parent base_link, child suspension_left_link, origin xyz=0 0 0 rpy=0 0 0, axis 0 0 1, limit lower=-0.005 upper=0.005 effort=100.0 velocity=1.0
- added joint suspension_right_rjoint: type fixed, parent base_link, child suspension_right_link, origin xyz=0 0 0 rpy=0 0 0, axis 0 0 1, limit lower=-0.005 upper=0.005 effort=100.0 velocity=1.0
- added joint torso_fixed_column_rjoint: type fixed, parent base_link, child torso_fixed_column_link, origin xyz=-0.062 0 0.195 rpy=0 0 0, axis 0 0 0
- added joint torso_fixed_rjoint: type fixed, parent base_link, child torso_fixed_link, origin xyz=-0.062 0.0 0.193 rpy=0 0 0, axis 0 0 0
- added joint torso_lift_rjoint: type fixed, parent torso_fixed_link, child torso_lift_link, origin xyz=0.0 0.0 0.597 rpy=0.0 0.0 0.0, axis 0 0 1, limit lower=0 upper=0.35 effort=2000 velocity=0.07
- added joint wheel_left_rjoint: type fixed, parent suspension_left_link, child wheel_left_link, origin xyz=0 0.2022 0.0 rpy=-1.57079632679 0 0, axis 0 0 1, limit effort=6.0 velocity=10.152284264
- added joint wheel_right_rjoint: type fixed, parent suspension_right_link, child wheel_right_link, origin xyz=0 -0.2022 0.0 rpy=-1.57079632679 0 0, axis 0 0 1, limit effort=6.0 velocity=10.152284264
- added joint xtion_depth_optical_rjoint: type fixed, parent xtion_depth_frame, child xtion_depth_optical_frame, origin xyz=0 0 0 rpy=-1.57079632679 0.0 -1.57079632679
- added joint xtion_depth_rjoint: type fixed, parent xtion_rgb_frame, child xtion_depth_frame, origin xyz=0.0 0.047 0.0 rpy=0 0 0
- added joint xtion_optical_gjoint: type fixed, parent xtion_link, child xtion_optical_frame, origin xyz=0 0 0 rpy=-1.57079632679 0.0 -1.57079632679
- added joint xtion_orbbec_aux_rjoint: type fixed, parent xtion_link, child xtion_orbbec_aux_rjoint_frame, origin xyz=0 0 0 rpy=0 0 0
- added joint xtion_rgb_optical_rjoint: type fixed, parent xtion_rgb_frame, child xtion_rgb_optical_frame, origin xyz=0 0 0 rpy=-1.57079632679 0.0 -1.57079632679
- added joint xtion_rgb_rjoint: type fixed, parent xtion_orbbec_aux_rjoint_frame, child xtion_rgb_frame, origin xyz=0.0 0.022 0.0 rpy=0 0 0
- added joint xtion_rjoint: type fixed, parent head_2_link, child xtion_link, origin xyz=0.080815 0.0822042 0.00658015 rpy=-1.57629 0.0197082 -0.000892242

Commit message: fixes

File: myGym/envs/robots/tiago/tiago_pal_gripper.urdf (robot description, URDF)
Before this commit: robot tiago, 49 links, 48 joints
Links:
- removed link gripper_grasping_frame
- removed link rgbd_laser_link
- added link gripper_link, mass 0.602660; collision mesh filename=meshes/gripper/gripper_link_collision.stl; visual mesh filename=meshes/gripper/gripper_link.stl
- link arm_1_link: mass 1.563428 -> 2.31325
- link arm_2_link: mass 1.800397 -> 1.10224
- link arm_3_link: mass 2.343502 -> 2.42460
- link arm_4_link: mass 1.432697 -> 1.45429
- link arm_5_link: mass 0.9359143689 -> 1.07424; geometry collision mesh filename=meshes/arm/arm_5_collision.dae scale=1 1 1; visual mesh filename=meshes/arm/arm_5.stl scale=1 1 1
- link arm_6_link: mass 0.30275767222 -> 0.28722; geometry collision mesh filename=meshes/arm/arm_6_collision.dae scale=1 1 1; visual mesh filename=meshes/arm/arm_6.stl scale=1 1 1
- link arm_7_link: mass 0.100 -> 0.05935
- link gripper: mass 0.602660 -> 0.0001; geometry 
Joints:
- removed joint rgbd_laser_rjoint
- joint arm_1_rjoint: limit lower=0.0 upper=2.74889357189 effort=43.0 velocity=1.95 -> lower=0.0 upper=2.74889357189 effort=39.0 velocity=2.7
- joint arm_2_rjoint: limit lower=-1.57079632679 upper=1.0908307825 effort=43.0 velocity=1.95 -> lower=-1.57079632679 upper=1.0908307825 effort=39.0 velocity=3.66; origin xyz=0.125 0.0195 -0.031 rpy=1.57079632679 0.0 0.0 -> xyz=0.125 0.0165 -0.031 rpy=1.57079632679 0.0 0.0
- joint arm_3_rjoint: limit lower=-3.53429173529 upper=1.57079632679 effort=26 velocity=2.35 -> lower=-3.53429173529 upper=1.57079632679 effort=17.86 velocity=4.58; origin xyz=0.0895 0.0 -0.0015 rpy=-1.57079632679 0.0 1.57079632679 -> xyz=0.0895 0.0 0.0015 rpy=-1.57079632679 0.0 1.57079632679
- joint arm_4_rjoint: limit lower=-0.392699081699 upper=2.35619449019 effort=26 velocity=2.35 -> lower=-0.392699081699 upper=2.35619449019 effort=17.86 velocity=4.58
- joint arm_5_rjoint: origin xyz=-0.162 0.02 0.027 rpy=1.57079632679 -1.57079632679 -1.57079632679 -> xyz=-0.162 0.02 0.027 rpy=0.0 -1.57079632679 0.0
- joint arm_6_rjoint: limit lower=-1.41371669412 upper=1.41371669412 effort=6.6 velocity=1.76 -> lower=-1.57079632679 upper=1.57079632679 effort=6.6 velocity=1.76
- joint arm_tool_rjoint: origin xyz=0 0 0.0573 rpy=1.57079632679 -1.57079632679 3.14159265359 -> xyz=0 0 0.046 rpy=1.57079632679 -1.57079632679 3.14159265359
- joint endeffector_gjoint: origin xyz=0 0.0 0.1 rpy=0 0 0 -> xyz=0 0 0 rpy=0 0 0
- joint gripper_grasping_frame_rjoint: child gripper_grasping_frame -> gripper; parent gripper -> gripper_link
- joint gripper_left_finger_rjoint: parent gripper -> gripper_link
- joint gripper_right_finger_rjoint: parent gripper -> gripper_link
- joint gripper_rjoint: child gripper -> gripper_link

File: myGym/envs/robots/tiago_dualhand/tiago_dual_hey5.urdf (robot description, URDF)
Before this commit: robot tiago_dual, 128 links, 127 joints
Joints:
- joint endeffector_gjoint: origin xyz=0.12 0.03 0.0 rpy=0 0 0 -> xyz=0.0 0.0 0.0 rpy=0 0 0

Commit message: tiago_singlehand fixed

File: myGym/envs/robots/tiago/tiago_pal_gripper.urdf (robot description, URDF)
Before this commit: robot tiago, 48 links, 47 joints
Links:
- removed link xtion_orbbec_aux_rjoint_frame
- added link xtion_orbbec_aux_joint_frame, mass 0.001
Joints:
- removed joint base_antenna_left_rjoint
- removed joint base_antenna_right_rjoint
- removed joint base_footprint_rjoint
- removed joint base_imu_rjoint
- removed joint base_laser_gjoint
- removed joint base_sonar_01_rjoint
- removed joint base_sonar_02_rjoint
- removed joint base_sonar_03_rjoint
- removed joint caster_back_left_1_rjoint
- removed joint caster_back_left_2_rjoint
- removed joint caster_back_right_1_rjoint
- removed joint caster_back_right_2_rjoint
- removed joint caster_front_left_1_rjoint
- removed joint caster_front_left_2_rjoint
- removed joint caster_front_right_1_rjoint
- removed joint caster_front_right_2_rjoint
- removed joint cover_rjoint
- removed joint gripper_grasping_frame_rjoint
- removed joint gripper_left_finger_rjoint
- removed joint gripper_right_finger_rjoint
- removed joint gripper_rjoint
- removed joint gripper_tool_rjoint
- removed joint head_1_rjoint
- removed joint head_2_rjoint
- removed joint suspension_left_rjoint
- removed joint suspension_right_rjoint
- removed joint torso_fixed_column_rjoint
- removed joint torso_fixed_rjoint
- removed joint torso_lift_rjoint
- removed joint wheel_left_rjoint
- removed joint wheel_right_rjoint
- removed joint xtion_depth_optical_rjoint
- removed joint xtion_depth_rjoint
- removed joint xtion_optical_gjoint
- removed joint xtion_orbbec_aux_rjoint
- removed joint xtion_rgb_optical_rjoint
- removed joint xtion_rgb_rjoint
- removed joint xtion_rjoint
- added joint base_antenna_left_joint: type fixed, parent base_link, child base_antenna_left_link, origin xyz=-0.201 0.1062 0.195 rpy=0 0 0
- added joint base_antenna_right_joint: type fixed, parent base_link, child base_antenna_right_link, origin xyz=-0.201 -0.1062 0.195 rpy=0 0 0
- added joint base_footprint_joint: type fixed, parent base_footprint, child base_link, origin xyz=0 0 0.0985 rpy=0 0 0
- added joint base_imu_joint: type fixed, parent base_link, child base_imu_link, origin xyz=0.10171 0 0.11282 rpy=0 0 -1.57079632679
- added joint base_laser_joint: type fixed, parent base_link, child base_laser_link, origin xyz=0.202 0.0 -0.004 rpy=0 0 0, axis 0 1 0
- added joint base_sonar_01_joint: type fixed, parent base_link, child base_sonar_01_link, origin xyz=-0.183 -0.183 0.173 rpy=0 0 3.92699081699, axis 0 0 1
- added joint base_sonar_02_joint: type fixed, parent base_link, child base_sonar_02_link, origin xyz=-0.259 0.0 0.173 rpy=0 0 3.14159265359, axis 0 0 1
- added joint base_sonar_03_joint: type fixed, parent base_link, child base_sonar_03_link, origin xyz=-0.183 0.183 0.173 rpy=0 0 2.35619449019, axis 0 0 1
- added joint caster_back_left_1_joint: type fixed, parent base_link, child caster_back_left_1_link, origin xyz=-0.1735 0.102 -0.0335 rpy=0 0 0, axis 0 0 1
- added joint caster_back_left_2_joint: type fixed, parent caster_back_left_1_link, child caster_back_left_2_link, origin xyz=-0.016 0.0000 -0.040 rpy=-1.57079632679 0 0, axis 0 0 1
- added joint caster_back_right_1_joint: type fixed, parent base_link, child caster_back_right_1_link, origin xyz=-0.1735 -0.102 -0.0335 rpy=0 0 0, axis 0 0 1
- added joint caster_back_right_2_joint: type fixed, parent caster_back_right_1_link, child caster_back_right_2_link, origin xyz=-0.016 0.0000 -0.040 rpy=-1.57079632679 0 0, axis 0 0 1
- added joint caster_front_left_1_joint: type fixed, parent base_link, child caster_front_left_1_link, origin xyz=0.1695 0.102 -0.0335 rpy=0 0 0, axis 0 0 1
- added joint caster_front_left_2_joint: type fixed, parent caster_front_left_1_link, child caster_front_left_2_link, origin xyz=-0.016 0.0000 -0.040 rpy=-1.57079632679 0 0, axis 0 0 1
- added joint caster_front_right_1_joint: type fixed, parent base_link, child caster_front_right_1_link, origin xyz=0.1695 -0.102 -0.0335 rpy=0 0 0, axis 0 0 1
- added joint caster_front_right_2_joint: type fixed, parent caster_front_right_1_link, child caster_front_right_2_link, origin xyz=-0.016 0.0000 -0.040 rpy=-1.57079632679 0 0, axis 0 0 1
- added joint cover_joint: type fixed, parent base_footprint, child base_cover_link, origin xyz=0 0 0.13 rpy=0 0 0
- added joint gripper_gjoint: type fixed, parent arm_tool_link, child gripper_link, origin xyz=0.01 0 0 rpy=1.57079632679 1.57079632679 -1.57079632679, axis 0 0 0
- added joint gripper_grasping_frame_gjoint: type fixed, parent gripper_link, child gripper, origin xyz=0 0 -0.12 rpy=-1.5708 1.5708 0
- added joint gripper_left_finger_gjoint: type prismatic, parent gripper_link, child gripper_left_finger_link, origin xyz=0. 0 0 rpy=0 0 0, axis -1 0 0, limit lower=0 upper=0.045 effort=16 velocity=0.05
- added joint gripper_right_finger_gjoint: type prismatic, parent gripper_link, child gripper_right_finger_link, origin xyz=0. 0 0 rpy=0 0 0, axis 1 0 0, limit lower=0.0 upper=0.045 effort=16 velocity=0.05
- added joint gripper_tool_gjoint: type fixed, parent arm_tool_link, child gripper_tool_link, origin xyz=0.01 0 0 rpy=1.57079632679 1.57079632679 -1.57079632679, axis 0 0 0
- added joint head_1_joint: type fixed, parent torso_lift_link, child head_1_link, origin xyz=0.182 0.0 0.0 rpy=0 0 0, axis 0 0 1, limit lower=-1.308996939 upper=1.308996939 effort=5.197 velocity=3.0
- added joint head_2_joint: type fixed, parent head_1_link, child head_2_link, origin xyz=0.005 0.0 0.098 rpy=1.57079632679 0 0, axis 0 0 1, limit lower=-1.0471975512 upper=0.785398163397 effort=2.77 velocity=3.0
- added joint suspension_left_joint: type fixed, parent base_link, child suspension_left_link, origin xyz=0 0 0 rpy=0 0 0, axis 0 0 1, limit lower=-0.005 upper=0.005 effort=100.0 velocity=1.0
- added joint suspension_right_joint: type fixed, parent base_link, child suspension_right_link, origin xyz=0 0 0 rpy=0 0 0, axis 0 0 1, limit lower=-0.005 upper=0.005 effort=100.0 velocity=1.0
- added joint torso_fixed_column_joint: type fixed, parent base_link, child torso_fixed_column_link, origin xyz=-0.062 0 0.195 rpy=0 0 0, axis 0 0 0
- added joint torso_fixed_joint: type fixed, parent base_link, child torso_fixed_link, origin xyz=-0.062 0.0 0.193 rpy=0 0 0, axis 0 0 0
- added joint torso_lift_joint: type fixed, parent torso_fixed_link, child torso_lift_link, origin xyz=0.0 0.0 0.597 rpy=0.0 0.0 0.0, axis 0 0 1, limit lower=0 upper=0.35 effort=2000 velocity=0.07
- added joint wheel_left_joint: type fixed, parent suspension_left_link, child wheel_left_link, origin xyz=0 0.2022 0.0 rpy=-1.57079632679 0 0, axis 0 0 1, limit effort=6.0 velocity=10.152284264
- added joint wheel_right_joint: type fixed, parent suspension_right_link, child wheel_right_link, origin xyz=0 -0.2022 0.0 rpy=-1.57079632679 0 0, axis 0 0 1, limit effort=6.0 velocity=10.152284264
- added joint xtion_depth_joint: type fixed, parent xtion_rgb_frame, child xtion_depth_frame, origin xyz=0.0 0.047 0.0 rpy=0 0 0
- added joint xtion_depth_optical_joint: type fixed, parent xtion_depth_frame, child xtion_depth_optical_frame, origin xyz=0 0 0 rpy=-1.57079632679 0.0 -1.57079632679
- added joint xtion_joint: type fixed, parent head_2_link, child xtion_link, origin xyz=0.080815 0.0822042 0.00658015 rpy=-1.57629 0.0197082 -0.000892242
- added joint xtion_optical_joint: type fixed, parent xtion_link, child xtion_optical_frame, origin xyz=0 0 0 rpy=-1.57079632679 0.0 -1.57079632679
- added joint xtion_orbbec_aux_joint: type fixed, parent xtion_link, child xtion_orbbec_aux_joint_frame, origin xyz=0 0 0 rpy=0 0 0
- added joint xtion_rgb_joint: type fixed, parent xtion_orbbec_aux_joint_frame, child xtion_rgb_frame, origin xyz=0.0 0.022 0.0 rpy=0 0 0
- added joint xtion_rgb_optical_joint: type fixed, parent xtion_rgb_frame, child xtion_rgb_optical_frame, origin xyz=0 0 0 rpy=-1.57079632679 0.0 -1.57079632679
- joint endeffector_gjoint: origin xyz=0 0 0 rpy=0 0 0 -> xyz=0.04 0 0 rpy=0 0 0

Commit message: open/close positions update in helpers.py

File: myGym/envs/robots/tiago/tiago_pal_gripper.urdf (robot description, URDF)
Before this commit: robot tiago, 51 links, 50 joints
Joints:
- removed joint gripper_gjoint
- removed joint gripper_grasping_frame_gjoint
- removed joint gripper_tool_gjoint
- added joint gripper_grasping_frame_joint: type fixed, parent gripper_link, child gripper, origin xyz=0 0 -0.12 rpy=-1.5708 1.5708 0
- added joint gripper_joint: type fixed, parent arm_tool_link, child gripper_link, origin xyz=0.01 0 0 rpy=1.57079632679 1.57079632679 -1.57079632679, axis 0 0 0
- added joint gripper_tool_joint: type fixed, parent arm_tool_link, child gripper_tool_link, origin xyz=0.01 0 0 rpy=1.57079632679 1.57079632679 -1.57079632679, axis 0 0 0
