Commit message: Creation of dice throw feature branch by J.Picha

File: myGym/envs/robots/kuka_magnetic_gripper_sdf/kuka_push.urdf (robot description, URDF)
Before this commit: robot lbr_iiwa, 13 links, 12 joints
Links:
- link slider: geometry collision mesh filename=meshes/dice_paddle.stl scale=.002 .002 .002; visual mesh filename=meshes/dice_paddle.stl scale=.002 .002 .002
