Commit message: pre-submit

File: myGym/envs/robots/kuka_magnetic_gripper_sdf/kuka_magnetic.urdf (robot description, URDF)
Before this commit: robot lbr_iiwa, 13 links, 12 joints
Links:
- link collet: geometry 
- link endeffector: geometry 
- link gripper: geometry 
- link lbr_iiwa_link_0: geometry 
- link lbr_iiwa_link_1: geometry 
- link lbr_iiwa_link_2: geometry 
- link lbr_iiwa_link_3: geometry 
- link lbr_iiwa_link_4: geometry 
- link lbr_iiwa_link_5: geometry 
- link lbr_iiwa_link_6: geometry 
- link lbr_iiwa_link_7: geometry 
- link sensor: geometry 
- link slider: geometry 

File: myGym/envs/robots/pepper/pepper.urdf (robot description, URDF)
Before this commit: robot JulietteY20MP, 99 links, 98 joints
Links:
- link Head: geometry collision mesh filename=meshes/pepper/HeadPitch_0.10.stl scale=1 1 1
- link HeadPitch_1: geometry 
- link HeadPitch_2: geometry 
- link HeadPitch_3: geometry 
- link HeadPitch_4: geometry 
- link Hip: geometry collision mesh filename=meshes/pepper/HipRoll_0.10.stl scale=1 1 1
- link HipPitch_1: geometry 
- link KneePitch_1: geometry 
- link LBicep: geometry collision mesh filename=meshes/pepper/LShoulderRoll_0.10.stl scale=1 1 1
- link LElbow: geometry collision mesh filename=meshes/pepper/LElbowYaw_0.10.stl scale=1 1 1
- link LElbowRoll_1: geometry 
- link LFinger11_link: geometry collision mesh filename=meshes/pepper/Phalax.obj scale=1 1 1
- link LFinger12_link: geometry collision mesh filename=meshes/pepper/Phalax.obj scale=1 1 1
- link LFinger13_link: geometry collision mesh filename=meshes/pepper/PhalaxEnd.obj scale=1 1 1
- link LFinger21_link: geometry collision mesh filename=meshes/pepper/Phalax.obj scale=1 1 1
- link LFinger22_link: geometry collision mesh filename=meshes/pepper/Phalax.obj scale=1 1 1
- link LFinger23_link: geometry collision mesh filename=meshes/pepper/PhalaxEnd.obj scale=1 1 1
- link LFinger31_link: geometry collision mesh filename=meshes/pepper/Phalax.obj scale=1 1 1
- link LFinger32_link: geometry collision mesh filename=meshes/pepper/Phalax.obj scale=1 1 1
- link LFinger33_link: geometry collision mesh filename=meshes/pepper/PhalaxEnd.obj scale=1 1 1
- link LFinger41_link: geometry collision mesh filename=meshes/pepper/Phalax.obj scale=1 1 1
- link LFinger42_link: geometry collision mesh filename=meshes/pepper/Phalax.obj scale=1 1 1
- link LFinger43_link: geometry collision mesh filename=meshes/pepper/PhalaxEnd.obj scale=1 1 1
- link LForeArm: geometry collision mesh filename=meshes/pepper/LElbowRoll_0.10.stl scale=1 1 1
- link LShoulder: geometry collision mesh filename=meshes/pepper/LShoulderPitch_0.10.stl scale=1 1 1
- link LShoulderRoll_1: geometry 
- link LThumb1_link: geometry collision mesh filename=meshes/pepper/Phalax.obj scale=1 1 1
- link LThumb2_link: geometry collision mesh filename=meshes/pepper/PhalaxEnd.obj scale=1 1 1
- link Neck: geometry collision mesh filename=meshes/pepper/HeadYaw_0.10.stl scale=1 1 1
- link Pelvis: geometry collision mesh filename=meshes/pepper/HipPitch_0.10.stl scale=1 1 1
- link RBicep: geometry collision mesh filename=meshes/pepper/RShoulderRoll_0.10.stl scale=1 1 1
- link RElbow: geometry collision mesh filename=meshes/pepper/RElbowYaw_0.10.stl scale=1 1 1
- link RElbowRoll_1: geometry 
- link RFinger11_link: geometry collision mesh filename=meshes/pepper/Phalax.obj scale=1 1 1
- link RFinger12_link: geometry collision mesh filename=meshes/pepper/Phalax.obj scale=1 1 1
- link RFinger13_link: geometry collision mesh filename=meshes/pepper/PhalaxEnd.obj scale=1 1 1
- link RFinger21_link: geometry collision mesh filename=meshes/pepper/Phalax.obj scale=1 1 1
- link RFinger22_link: geometry collision mesh filename=meshes/pepper/Phalax.obj scale=1 1 1
- link RFinger31_link: geometry collision mesh filename=meshes/pepper/Phalax.obj scale=1 1 1
- link RFinger32_link: geometry collision mesh filename=meshes/pepper/Phalax.obj scale=1 1 1
- link RFinger33_link: geometry collision mesh filename=meshes/pepper/PhalaxEnd.obj scale=1 1 1
- link RFinger41_link: geometry collision mesh filename=meshes/pepper/Phalax.obj scale=1 1 1
- link RFinger42_link: geometry collision mesh filename=meshes/pepper/Phalax.obj scale=1 1 1
- link RFinger43_link: geometry collision mesh filename=meshes/pepper/PhalaxEnd.obj scale=1 1 1
- link RForeArm: geometry collision mesh filename=meshes/pepper/RElbowRoll_0.10.stl scale=1 1 1
- link RShoulder: geometry collision mesh filename=meshes/pepper/RShoulderPitch_0.10.stl scale=1 1 1
- link RShoulderRoll_1: geometry 
- link RThumb1_link: geometry collision mesh filename=meshes/pepper/Phalax.obj scale=1 1 1
- link RThumb2_link: geometry collision mesh filename=meshes/pepper/PhalaxEnd.obj scale=1 1 1
- link Tibia: geometry collision mesh filename=meshes/pepper/KneePitch_0.10.stl scale=1 1 1
- link Torso_1: geometry 
- link Torso_2: geometry 
- link Torso_3: geometry 
- link Torso_4: geometry 
- link WheelB_link: geometry collision mesh filename=meshes/pepper/Wheel_0.10.stl scale=1 1 1
- link WheelFL_link: geometry collision mesh filename=meshes/pepper/Wheel_0.10.stl scale=1 1 1
- link WheelFR_link: geometry collision mesh filename=meshes/pepper/Wheel_0.10.stl scale=1 1 1
- link endeffector: geometry collision mesh filename=meshes/pepper/PhalaxEnd.obj scale=1 1 1
- link l_wrist: geometry collision mesh filename=meshes/pepper/LWristYaw_vhacd.obj scale=1 1 1
- link r_wrist: geometry collision mesh filename=meshes/pepper/RWristYaw_vhacd.obj scale=1 1 1
- link torso: geometry collision mesh filename=meshes/pepper/Torso_0.10.stl scale=0 0 0
