Commit message: New commit

File: myGym/envs/objects/furniture/urdf/table.urdf (robot description, URDF)
Before this commit: robot table, 1 links, 0 joints
Links:
- link baseLink: geometry collision mesh filename=../obj/table.obj scale=0.2 0.2 0.2; visual mesh filename=../obj/table.obj scale=0.2 0.2 0.2

File: myGym/envs/objects/toys/urdf/dice.urdf (robot description, URDF)
Before this commit: robot dice.urdf, 1 links, 0 joints
Links:
- link baseLink: mass 0.113 -> 1.001; geometry collision box size=0.1 0.1 0.1; visual box size=0.1 0.1 0.1
