Commit message: robots urdf update

File: myGym/envs/robots/franka_emika/panda_moveit/urdf/panda2.urdf (robot description, URDF)
Before this commit: robot panda, 13 links, 12 joints
Joints:
- joint panda_finger_gjoint2: mimic joint=panda_finger_joint1 -> joint=panda_finger_gjoint1

File: myGym/envs/robots/hsr/hsrb4s.urdf (robot description, URDF)
Before this commit: robot hsrb, 45 links, 44 joints
Joints:
- joint hand_l_mimic_distal_gjoint: mimic joint=hand_l_spring_proximal_rjoint multiplier=-1.0 -> joint=hand_l_proximal_gjoint multiplier=-1.0
- joint hand_l_proximal_gjoint: mimic joint=hand_motor_rjoint -> joint=hand_motor_gjoint
- joint hand_r_mimic_distal_gjoint: mimic joint=hand_r_spring_proximal_rjoint multiplier=-1.0 -> joint=hand_r_spring_proximal_gjoint multiplier=-1.0
- joint torso_lift_rjoint: mimic joint=arm_lift_rjoint multiplier=0.5 -> joint=arm_lift_gjoint multiplier=0.5

File: myGym/envs/robots/kuka_gripper/kuka_gripper.urdf (robot description, URDF)
Before this commit: robot kuka_gripper, 18 links, 17 joints
Links:
- link finger_00: geometry collision mesh filename=meshes/finger_0.obj scale=1 0.7 0.7; visual mesh filename=meshes/finger_0.obj scale=1 0.7 0.7
- link finger_01: geometry collision mesh filename=meshes/finger_1.obj scale=1 0.7 0.7; visual mesh filename=meshes/finger_1.obj scale=1 0.7 0.7
- link finger_10: geometry collision mesh filename=meshes/finger_0.obj scale=1 0.7 0.7; visual mesh filename=meshes/finger_0.obj scale=1 0.7 0.7
- link finger_11: geometry collision mesh filename=meshes/finger_1.obj scale=1 0.7 0.7; visual mesh filename=meshes/finger_1.obj scale=1 0.7 0.7
- link gripper: geometry collision mesh filename=meshes/base.obj; visual mesh filename=meshes/base.obj
- link lbr_iiwa_link_0: geometry collision mesh filename=meshes/link_0.obj; visual mesh filename=meshes/link_0.obj
- link lbr_iiwa_link_1: geometry collision mesh filename=meshes/link_1.obj; visual mesh filename=meshes/link_1.obj
- link lbr_iiwa_link_2: geometry collision mesh filename=meshes/link_2.obj; visual mesh filename=meshes/link_2.obj
- link lbr_iiwa_link_3: geometry collision mesh filename=meshes/link_3.obj; visual mesh filename=meshes/link_3.obj
- link lbr_iiwa_link_4: geometry collision mesh filename=meshes/link_4.obj; visual mesh filename=meshes/link_4.obj
- link lbr_iiwa_link_5: geometry collision mesh filename=meshes/link_5.obj; visual mesh filename=meshes/link_5.obj
- link lbr_iiwa_link_6: geometry collision mesh filename=meshes/link_6.obj; visual mesh filename=meshes/link_6.obj
- link lbr_iiwa_link_7: geometry collision mesh filename=meshes/link_7.obj; visual mesh filename=meshes/link_7.obj
- link skin_00: geometry collision mesh filename=meshes/skin_0.obj scale=1 0.3 0.7; visual mesh filename=meshes/skin_0.obj scale=1 0.3 0.7
- link skin_01: geometry collision mesh filename=meshes/skin_0.obj scale=1 0.3 0.3; visual mesh filename=meshes/skin_0.obj scale=1 0.3 0.3
- link skin_10: geometry collision mesh filename=meshes/skin_0.obj scale=1 0.3 0.7; visual mesh filename=meshes/skin_0.obj scale=1 0.3 0.7
- link skin_11: geometry collision mesh filename=meshes/skin_0.obj scale=1 0.3 0.3; visual mesh filename=meshes/skin_0.obj scale=1 0.3 0.3
Joints:
- joint finger00_to_finger01_gjoint: limit lower=0 upper=-1.5707963267948966 effort=30 velocity=1 -> lower=-1.5707963267948966 upper=0 effort=30 velocity=1
- joint finger10_to_finger11_gjoint: limit lower=0 upper=-1.5707963267948966 effort=30 velocity=1 -> lower=-1.5707963267948966 upper=0 effort=30 velocity=1

File: myGym/envs/robots/nico/nico_upper_rh6d_copy.urdf (robot description, URDF)
Before this commit: robot nico_upper, 33 links, 32 joints
Links:
- removed link finger_segment:11
- removed link finger_segment:12
- removed link finger_segment:13
- removed link finger_segment:21
- removed link finger_segment:23
- removed link fingertip:11
- removed link fingertip:12
- removed link fingertip:13
- removed link neck:11
- removed link torso:11
- added link neck; collision mesh filename=meshes/neck_long_new.stl; visual mesh filename=meshes/neck_long_new.stl
- added link torso; visual mesh filename=meshes/torso_merged_new.stl
- added link world
- link endeffector: mass 0.000009 -> None; geometry visual sphere radius=0.005
- link gripper: geometry collision mesh filename=meshes/right_palm_simple.stl scale=0.001 0.001 0.001; visual mesh filename=meshes/rh6d_palm_simple.stl scale=0.001 0.001 0.001
- link head:21: geometry collision mesh filename=meshes/head_half_simple.stl scale=0.001 0.001 0.001; visual mesh filename=meshes/headfbx.stl scale=1 1 1
- link right_wrist:11: geometry collision mesh filename=meshes/rh6d_shell_simple.stl scale=0.001 0.001 0.001; visual mesh filename=meshes/rh6d_shell_simple.stl scale=0.001 0.001 0.001
Joints:
- removed joint endeffector_gjoint
- removed joint head_z
- removed joint r_indexfinger_1st_gjoint
- removed joint r_indexfingers_x_rjoint
- removed joint r_ringfinger_1st_x_gjoint
- removed joint r_ringfinger_2nd_x_gjoint
- removed joint r_ringfingers_x_gjoint
- removed joint r_thumb_1st_x_gjoint
- removed joint r_thumb_2nd_x_gjoint
- removed joint r_thumb_x_gjoint
- removed joint r_wrist_x_gjoint
- added joint endeffector_joint: type fixed, parent gripper, child endeffector, origin xyz=-0.025 0.00 -0.14 rpy=0 0 0
- added joint head_z_rjoint: type fixed, parent torso, child neck, origin xyz=-0.02 0.0 0.23 rpy=0 0 0, axis 0 0 1, limit lower=-3.124 upper=3.142 effort=30 velocity=1
- added joint r_wrist_x_rjoint: type revolute, parent right_wrist:11, child gripper, origin xyz=0.023416 0.006052 -0.070337 rpy=-0.433097 0 0, axis 1 0 0, limit lower=0 upper=0.872665 effort=30 velocity=1
- added joint world_to_base_link: type fixed, parent world, child torso
- joint head_y: origin xyz=0 0.023001 0.0745 rpy=0 0 0 -> xyz=0 0.0 0.40 rpy=0 0 0
- joint l_shoulder_z: parent torso:11 -> torso
- joint r_shoulder_z_rjoint: parent torso:11 -> torso
