Commit message: turn off collisions for panda_sgripper's fingers

File: myGym/envs/robots/franka_emika/panda_moveit/urdf/panda2.urdf (robot description, URDF)
Before this commit: robot panda, 16 links, 15 joints
Links:
- link panda_leftfinger: geometry visual mesh filename=meshes/visual/finger.dae
- link panda_rightfinger: geometry visual mesh filename=meshes/visual/finger.dae
