Commit message: nico mesh and urdf cleaning - working joints

File: myGym/envs/robots/nico/nico_upper.urdf (robot description, URDF)
Before this commit: robot nico_upper, 33 links, 32 joints
Links:
- link head:21: geometry collision mesh filename=meshes/head_half_simple.stl scale=0.001 0.001 0.001; visual mesh filename=meshes/head_half_simple.stl scale=0.001 0.001 0.001
- link torso:11: geometry collision mesh filename=meshes/torso_simple.stl scale=0.001 0.001 0.001; visual mesh filename=meshes/torso_simple.stl scale=0.001 0.001 0.001

Commit message: nico model update

File: myGym/envs/robots/nico/nico_upper.urdf (robot description, URDF)
Before this commit: robot nico_upper, 33 links, 32 joints
Links:
- link gripper: geometry collision mesh filename=meshes/right_palm_simple.stl scale=0.001 0.001 0.001; visual mesh filename=meshes/right_palm_simple.stl scale=0.001 0.001 0.001
- link left_collarbone:11: geometry collision mesh filename=meshes/left_upper_arm_simple.stl scale=0.001 0.001 0.001; visual mesh filename=meshes/left_upper_arm_simple.stl scale=0.001 0.001 0.001
- link left_lower_arm:11: geometry visual mesh filename=meshes/left_lowerarm_simple.stl scale=0.001 0.001 0.001
- link left_palm:11: geometry collision mesh filename=meshes/left_palm_simple.stl scale=0.001 0.001 0.001; visual mesh filename=meshes/left_palm_simple.stl scale=0.001 0.001 0.001
- link left_shoulder:11: geometry collision mesh filename=meshes/left_shoulder_simple.stl scale=0.001 0.001 0.001; visual mesh filename=meshes/left_shoulder_simple.stl scale=0.001 0.001 0.001
- link left_upper_arm:11: geometry visual mesh filename=meshes/left_lower_arm_simple.stl scale=0.001 0.001 0.001
- link left_wrist:11: geometry collision mesh filename=meshes/left_wrist_simple.stl scale=0.001 0.001 0.001; visual mesh filename=meshes/left_wrist_simple.stl scale=0.001 0.001 0.001
- link neck:11: geometry collision mesh filename=meshes/neck_simple.stl scale=0.001 0.001 0.001; visual mesh filename=meshes/neck_simple.stl scale=0.001 0.001 0.001
- link right_collarbone:11: geometry collision mesh filename=meshes/right_upper_arm_simple.stl scale=0.001 0.001 0.001; visual mesh filename=meshes/right_upper_arm_simple.stl scale=0.001 0.001 0.001
- link right_lower_arm:11: geometry collision mesh filename=meshes/right_lowerarm_simple.stl scale=0.001 0.001 0.001; visual mesh filename=meshes/right_lowerarm_simple.stl scale=0.001 0.001 0.001
- link right_shoulder:11: geometry collision mesh filename=meshes/right_shoulder_simple.stl scale=0.001 0.001 0.001; visual mesh filename=meshes/right_shoulder_simple.stl scale=0.001 0.001 0.001
- link right_upper_arm:11: geometry collision mesh filename=meshes/right_lower_arm_simple.stl scale=0.001 0.001 0.001; visual mesh filename=meshes/right_lower_arm_simple.stl scale=0.001 0.001 0.001
- link right_wrist:11: geometry collision mesh filename=meshes/right_wrist_simple.stl scale=0.001 0.001 0.001; visual mesh filename=meshes/right_wrist_simple.stl scale=0.001 0.001 0.001
Joints:
- removed joint endeffector_joint
- removed joint r_indexfinger_1st_x
- removed joint r_ringfinger_1st_x
- removed joint r_ringfinger_2nd_x
- removed joint r_ringfingers_x
- removed joint r_thumb_1st_x
- removed joint r_thumb_2nd_x
- removed joint r_thumb_x
- added joint endeffector_gjoint: type revolute, parent finger_segment:13, child fingertip:13, origin xyz=0 -0 -0.016 rpy=-0.109614 0 0, axis 0.998022 0.00962907 0.0621208, limit lower=-1.309 upper=0 effort=30 velocity=1
- added joint r_indexfinger_1st_gjoint: type revolute, parent finger_segment:23, child finger_segment:13, origin xyz=-0.0005 0 -0.015999 rpy=-0.095246 0 0, axis 0.998022 0.00962907 0.0621208, limit lower=-1.309 upper=0 effort=30 velocity=1
- added joint r_ringfinger_1st_x_gjoint: type revolute, parent endeffector, child finger_segment:12, origin xyz=-0.0005 0 -0.016 rpy=-0.095245 0 0, axis 0.998022 -0.00962907 -0.0621208, limit lower=-1.309 upper=0 effort=30 velocity=1
- added joint r_ringfinger_2nd_x_gjoint: type revolute, parent finger_segment:12, child fingertip:12, origin xyz=0 -0 -0.016 rpy=-0.109614 0 0, axis 0.998022 -0.00962907 -0.0621208, limit lower=-1.309 upper=0 effort=30 velocity=1
- added joint r_ringfingers_x_gjoint: type revolute, parent gripper, child endeffector, origin xyz=-0.035879 0.006226 -0.040569 rpy=-0.569851 -0.062904 -3.141593, axis 0.998022 -0.00962907 -0.0621208, limit lower=-1.309 upper=0 effort=30 velocity=1
- added joint r_thumb_1st_x_gjoint: type revolute, parent finger_segment:21, child finger_segment:11, origin xyz=-0.0005 -0.000001 -0.016001 rpy=-0.095246 0 0, axis 1 0 0, limit lower=-1.309 upper=0 effort=30 velocity=1
- added joint r_thumb_2nd_x_gjoint: type revolute, parent finger_segment:11, child fingertip:11, origin xyz=0 0.000001 -0.015999 rpy=-0.109614 0 0, axis 1 0 0, limit lower=-1.309 upper=0 effort=30 velocity=1
- added joint r_thumb_x_gjoint: type revolute, parent gripper, child finger_segment:21, origin xyz=-0.0275 0.0199 -0.00842 rpy=1.915504 0 0, axis 1 0 0, limit lower=-1.309 upper=0 effort=30 velocity=1
- joint l_elbow_y: limit lower=-1.745 upper=1.745 effort=30 velocity=1 -> lower=1.545 upper=1.745 effort=30 velocity=1; origin xyz=-0.034583 0.023066 -0.169859 rpy=0 0.055976 0 -> xyz=-0.034583 0.023066 -0.169859 rpy=0 -1.405976 0

Commit message: nico urdf update

File: myGym/envs/robots/nico/nico_upper.urdf (robot description, URDF)
Before this commit: robot nico_upper, 33 links, 32 joints
Links:
- link right_collarbone:11: geometry collision mesh filename=meshes/right_upper_arm_simple.stl scale=0.001 0.001 0.001; visual mesh filename=meshes/right_collar_simple.stl scale=0.001 0.001 0.001

File: myGym/envs/robots/nico/nico_upper_rh6d.urdf (robot description, URDF)
Before this commit: robot nico_upper, 26 links, 25 joints
Links:
- removed link head:21
- removed link neck:11
- removed link right_collarbone:11
- removed link right_lower_arm:11
- removed link right_shoulder:11
- removed link right_upper_arm:11
- removed link torso:11
- added link head, mass 0.294137; collision mesh filename=mesh/head.stl; visual mesh filename=mesh/head.stl
- added link neck, mass 0.090439; collision mesh filename=mesh/neck.stl; visual mesh filename=mesh/neck.stl
- added link right_collarbone, mass 0.024811; collision mesh filename=mesh/right_collar.stl; visual mesh filename=mesh/right_collar.stl
- added link right_lower_arm, mass 0.076793; collision mesh filename=mesh/right_lower_arm.stl; visual mesh filename=mesh/right_lower_arm.stl
- added link right_shoulder, mass 0.084038; collision mesh filename=mesh/right_shoulder.stl; visual mesh filename=mesh/right_shoulder.stl
- added link right_upper_arm, mass 0.189729; collision mesh filename=mesh/right_upper_arm.stl; visual mesh filename=mesh/right_upper_arm.stl
- added link torso; visual mesh filename=mesh/torso.stl
Joints:
- removed joint head_y
- removed joint head_z
- removed joint r_arm_x_rjoint
- added joint head_y_rjoint: type revolute, parent neck, child head, origin xyz=0 0.0 0.10 rpy=0 0 0, axis 0 1 0, limit lower=-1.553 upper=1.379 effort=30 velocity=1
- added joint head_z_rjoint: type revolute, parent torso, child neck, origin xyz=-0.02 0.0 0.23 rpy=0 0 0, axis 0 0 1, limit lower=-3.124 upper=3.142 effort=30 velocity=1
- added joint r_upperarm_x_rjoint: type revolute, parent right_collarbone, child right_upper_arm, origin xyz=0.00 -0.073 -0.023 rpy=0 0 0, axis 1 0 0, limit lower=-3.002 upper=1.8675 effort=30 velocity=1
- joint l_shoulder_z: parent torso:11 -> torso
- joint r_elbow_y_rjoint: child right_lower_arm:11 -> right_lower_arm; origin xyz=-0.023001 -0.024001 -0.1732 rpy=0 0 0 -> xyz=0.0 0 -0.17 rpy=0 0 0; parent right_upper_arm:11 -> right_upper_arm
- joint r_shoulder_y_rjoint: child right_collarbone:11 -> right_collarbone; origin xyz=0.026211 -0.018056 0.037 rpy=0 0 0.20444 -> xyz=-0.021 -0.023 0.033 rpy=0 0 0; parent right_shoulder:11 -> right_shoulder
- joint r_shoulder_z_rjoint: child right_shoulder:11 -> right_shoulder; parent torso:11 -> torso
- joint r_wrist_z_rjoint: parent right_lower_arm:11 -> right_lower_arm
- joint world_to_base_link: child torso:11 -> torso
