Commit message: nico robot update

File: myGym/envs/robots/nico/nico_upper_rh6d.urdf (robot description, URDF)
Before this commit: robot nico_upper, 33 links, 32 joints
Links:
- removed link finger_segment:11
- removed link finger_segment:12
- removed link finger_segment:13
- removed link finger_segment:21
- removed link finger_segment:23
- removed link fingertip:11
- removed link fingertip:12
- removed link fingertip:13
- link endeffector: mass 0.000009 -> None; geometry visual sphere radius=0.005
- link gripper: geometry collision mesh filename=meshes/right_palm_simple.stl scale=0.001 0.001 0.001; visual mesh filename=meshes/rh6d_palm_simple.stl scale=0.001 0.001 0.001
- link right_wrist:11: geometry collision mesh filename=meshes/rh6d_shell_simple.stl scale=0.001 0.001 0.001; visual mesh filename=meshes/rh6d_shell_simple.stl scale=0.001 0.001 0.001
Joints:
- removed joint endeffector
- removed joint r_indexfinger_1st
- removed joint r_indexfingers_x_rjoint
- removed joint r_ringfinger_1st_x
- removed joint r_ringfinger_2nd_x
- removed joint r_ringfingers_x
- removed joint r_thumb_1st_x
- removed joint r_thumb_2nd_x
- removed joint r_thumb_x
- added joint endeffector_joint: type fixed, parent gripper, child endeffector, origin xyz=-0.025 0.05 -0.04 rpy=0 0 0

Commit message: Rewards extesion (FM and FMOM), Nico body update

File: myGym/envs/robots/nico/nico_upper_rh6d.urdf (robot description, URDF)
Before this commit: robot nico_upper, 25 links, 24 joints
Links:
- link torso:11: geometry visual mesh filename=meshes/torso_fbx.stl scale=0.01 0.01 0.01
Joints:
- joint endeffector_joint: origin xyz=-0.025 0.05 -0.04 rpy=0 0 0 -> xyz=-0.025 0.00 -0.14 rpy=0 0 0

Commit message: robot urdf update

File: myGym/envs/robots/nico/nico_upper_rh6d.urdf (robot description, URDF)
Before this commit: robot nico_upper, 25 links, 24 joints
Links:
- added link world
- link head:21: geometry collision mesh filename=meshes/headfbx.stl; visual mesh filename=meshes/headfbx.stl
- link neck:11: geometry collision mesh filename=meshes/neck_long_new.stl; visual mesh filename=meshes/neck_long_new.stl
- link right_collarbone:11: geometry collision mesh filename=meshes/right_collar_simple.stl scale=0.001 0.001 0.001; visual mesh filename=meshes/right_collar_simple.stl scale=0.001 0.001 0.001
- link right_upper_arm:11: geometry collision mesh filename=meshes/right_upper_arm_fbx.stl scale=0.001 0.001 0.001; visual mesh filename=meshes/right_upper_arm_fbx.stl scale=0.001 0.001 0.001
- link torso:11: geometry visual mesh filename=meshes/torso_merged_new.stl
Joints:
- added joint world_to_base_link: type fixed, parent world, child torso:11
- joint head_y: origin xyz=0 0.023001 0.0745 rpy=0 0 0 -> xyz=0 0.0 0.11 rpy=0 0 0
- joint head_z: origin xyz=0.001283 -0.000212 0.756309 rpy=0 0 0 -> xyz=-0.02 0.0 0.23 rpy=0 0 0
- joint l_shoulder_z: origin xyz=0.026783 0.049488 0.748809 rpy=0 0 0.019617 -> xyz=0.0 0.045 0.23 rpy=0 0 0.019617
- joint r_shoulder_z_rjoint: origin xyz=0.026783 -0.049912 0.748809 rpy=0 0 -0.20444 -> xyz=0.0 -0.045 0.23 rpy=0 0 0

Commit message: nico urdf update

File: myGym/envs/robots/nico/nico_upper_rh6d.urdf (robot description, URDF)
Before this commit: robot nico_upper_rh6d, 26 links, 25 joints
Links:
- removed link right_wrist:11
- added link indexfinger, mass 0.000009; collision mesh filename=mesh/finger.stl; visual mesh filename=mesh/finger.stl
- added link littlefinger, mass 0.000009; collision mesh filename=mesh/finger.stl; visual mesh filename=mesh/finger.stl
- added link middlefinger, mass 0.000009; collision mesh filename=mesh/finger.stl; visual mesh filename=mesh/finger.stl
- added link right_wrist, mass 0.028397; collision mesh filename=mesh/right_wrist.stl; visual mesh filename=mesh/right_wrist.stl
- link gripper: geometry collision mesh filename=mesh/right_palm.stl; visual mesh filename=mesh/right_palm.stl
Joints:
- added joint indexfinger_rjoint: type revolute, parent gripper, child indexfinger, origin xyz=0.00 -0.02 -0.06 rpy=0 0 0, axis 0 1 0, limit lower=-1.57 upper=0 effort=30 velocity=1
- added joint litlefinger_rjoint: type revolute, parent gripper, child littlefinger, origin xyz=0.00 0.02 -0.06 rpy=0 0 0, axis 0 1 0, limit lower=-1.57 upper=0 effort=30 velocity=1
- added joint middlefinger_rjoint: type revolute, parent gripper, child middlefinger, origin xyz=0 0 -0.06 rpy=0 0 0, axis 0 1 0, limit lower=-1.57 upper=0 effort=30 velocity=1
- joint endeffector_joint: origin xyz=-0.025 0.00 -0.14 rpy=0 0 0 -> xyz=0.03 0.00 -0.03 rpy=0 0 0
- joint head_y_rjoint: origin xyz=0 0.0 0.10 rpy=0 0 0 -> xyz=0 0.0 0.105 rpy=0 0 0
- joint r_wrist_x_rjoint: axis 1 0 0 -> 0 1 0; limit lower=0 upper=0.872665 effort=30 velocity=1 -> lower=-.5 upper=0.5 effort=30 velocity=1; origin xyz=0.023416 0.006052 -0.070337 rpy=-0.433097 0 0 -> xyz=0 0 -0.10 rpy=0 0 0; parent right_wrist:11 -> right_wrist
- joint r_wrist_z_rjoint: child right_wrist:11 -> right_wrist; origin xyz=0 0.0102 -0.12605 rpy=0 0 0.028946 -> xyz=0 0 -0.105 rpy=0 0 0

Commit message: nico update

File: myGym/envs/robots/nico/nico_upper_rh6d.urdf (robot description, URDF)
Before this commit: robot nico_upper_rh6d, 29 links, 28 joints
Links:
- removed link left_shoulder:11
- added link left_shoulder, mass 0.084038; collision mesh filename=mesh/right_shoulder.stl; visual mesh filename=mesh/right_shoulder.stl
Joints:
- removed joint l_shoulder_z
- added joint l_shoulder_z_rjoint: type revolute, parent torso, child left_shoulder, origin xyz=0.0 0.045 0.23 rpy=0 0 0, axis 0 0 1, limit lower=-1.745 upper=2.182 effort=30 velocity=1
- joint l_shoulder_y: parent left_shoulder:11 -> left_shoulder
- joint r_shoulder_z_rjoint: origin xyz=0.0 -0.045 0.23 rpy=0 0 0 -> xyz=0.005 -0.045 0.23 rpy=0 0 0

Commit message: urdf update  - sim2real  nico initial

File: myGym/envs/robots/nico/nico_upper_rh6d.urdf (robot description, URDF)
Before this commit: robot nico_upper_rh6d, 29 links, 28 joints
Joints:
- joint head_y_rjoint: limit lower=-1.553 upper=1.379 effort=30 velocity=1 -> lower=-0.8726 upper=0.4363 effort=30 velocity=1
- joint head_z_rjoint: limit lower=-3.124 upper=3.142 effort=30 velocity=1 -> lower=-1.5708 upper=1.5708 effort=30 velocity=1
- joint indexfinger_rjoint: limit lower=-1.57 upper=0 effort=30 velocity=1 -> lower=-2.57 upper=0 effort=30 velocity=1
- joint litlefinger_rjoint: limit lower=-1.57 upper=0 effort=30 velocity=1 -> lower=-2.57 upper=0 effort=30 velocity=1
- joint middlefinger_rjoint: limit lower=-1.57 upper=0 effort=30 velocity=1 -> lower=-2.57 upper=0 effort=30 velocity=1
- joint r_elbow_y_rjoint: limit lower=-1.745 upper=1.745 effort=30 velocity=1 -> lower=-1.57 upper=0 effort=30 velocity=1
- joint r_shoulder_y_rjoint: limit lower=-3.142 upper=3.124 effort=30 velocity=1 -> lower=-0.5236 upper=3.1416 effort=30 velocity=1
- joint r_shoulder_z_rjoint: limit lower=-1.745 upper=2.182 effort=30 velocity=1 -> lower=-0.4363 upper=1.3963 effort=30 velocity=1
- joint r_upperarm_x_rjoint: limit lower=-3.002 upper=1.8675 effort=30 velocity=1 -> lower=0 upper=1.2217 effort=30 velocity=1

Commit message: sim to real tests - two joints working

File: myGym/envs/robots/nico/nico_upper_rh6d.urdf (robot description, URDF)
Before this commit: robot nico_upper_rh6d, 29 links, 28 joints
Joints:
- joint head_y_rjoint: type revolute -> fixed
- joint head_z_rjoint: type revolute -> fixed
- joint indexfinger_rjoint: type revolute -> fixed
- joint l_shoulder_z_rjoint: type revolute -> fixed
- joint litlefinger_rjoint: type revolute -> fixed
- joint middlefinger_rjoint: type revolute -> fixed

Commit message: sim2real WORKING - 6 joints on right arm

File: myGym/envs/robots/nico/nico_upper_rh6d.urdf (robot description, URDF)
Before this commit: robot nico_upper_rh6d, 29 links, 28 joints
Joints:
- joint r_elbow_y_rjoint: limit lower=-1.57 upper=0 effort=30 velocity=1 -> lower=0.8726 upper=3.1416 effort=30 velocity=1; origin xyz=0.0 0 -0.17 rpy=0 0 0 -> xyz=0.0 0 -0.17 rpy=0 3.14 0
- joint r_upperarm_x_rjoint: axis 1 0 0 -> -1 0 0
- joint r_wrist_x_rjoint: limit lower=-.5 upper=0.5 effort=30 velocity=1 -> lower=-.78 upper=0.78 effort=30 velocity=1
- joint r_wrist_z_rjoint: origin xyz=0 0 -0.105 rpy=0 0 0 -> xyz=0 0 -0.105 rpy=0 0 1.57

Commit message: nico config update - reach task

File: myGym/envs/robots/nico/nico_upper_rh6d.urdf (robot description, URDF)
Before this commit: robot nico_upper_rh6d, 29 links, 28 joints
Links:
- link endeffector: geometry visual sphere radius=0.01
Joints:
- joint endeffector_joint: origin xyz=0.03 0.00 -0.03 rpy=0 0 0 -> xyz=0.00 -0.02 -0.11 rpy=0 0 0

Commit message: nico update - urdf for reaching

File: myGym/envs/robots/nico/nico_upper_rh6d.urdf (robot description, URDF)
Before this commit: robot nico_upper_rh6d, 29 links, 28 joints
Links:
- removed link indexfinger
- removed link littlefinger
- removed link middlefinger
- added link r_palm, mass 0.005332; collision mesh filename=mesh/right_palm.stl; visual mesh filename=mesh/right_palm.stl
- link gripper: mass 0.005332 -> 0.000009; geometry collision mesh filename=mesh/finger.stl; visual mesh filename=mesh/finger.stl
Joints:
- removed joint indexfinger_rjoint
- removed joint litlefinger_rjoint
- removed joint middlefinger_rjoint
- added joint gripper_rjoint: type revolute, parent r_palm, child gripper, origin xyz=0.00 -0.02 -0.06 rpy=0 0 0, axis 0 1 0, limit lower=-2.57 upper=0 effort=30 velocity=1
- joint endeffector_joint: origin xyz=0.00 -0.02 -0.11 rpy=0 0 0 -> xyz=0.00 -0.0 -0.05 rpy=0 0 0
- joint r_wrist_x_rjoint: child gripper -> r_palm

Commit message: nico reach update

File: myGym/envs/robots/nico/nico_upper_rh6d.urdf (robot description, URDF)
Before this commit: robot nico_upper_rh6d, 27 links, 26 joints
Joints:
- joint l_elbow_y: origin xyz=-0.034583 0.023066 -0.169859 rpy=0 -1.405976 0 -> xyz=-0.034583 0.023066 -0.169859 rpy=0 -1.695976 0
