Commit message: ik solver update

File: myGym/envs/robots/nico/nico_ik.urdf (robot description, URDF)
Before this commit: robot nico_upper_rh6d, 8 links, 7 joints
Links:
- added link world
Joints:
- added joint world_to_base_link: type fixed, parent world, child base_link
- joint r_elbow_y_rjoint: limit lower=0.0 upper=3.1416 effort=30 velocity=1 -> lower=-0.5 upper=3.1416 effort=30 velocity=1
