Commit message: nico urdf intetia update

File: myGym/envs/robots/nico/nico_grasp.urdf (robot description, URDF)
Before this commit: robot nico_upper_rh6d, 25 links, 24 joints
Links:
- link endeffectol: mass None -> 0.000009
- link endeffector: mass None -> 0.000009

Commit message: adaptive gripper thresholds - calculated from URDF joint limits and ranges.

File: myGym/envs/robots/nico/nico_grasp.urdf (robot description, URDF)
Before this commit: robot nico_upper_rh6d, 25 links, 24 joints
Joints:
- joint r_indexfinger_x_gjoint: limit lower=-2.57 upper=0 effort=30 velocity=5 -> lower=0 upper=2 effort=30 velocity=0; origin xyz=0.00 -0.02 -0.06 rpy=0 0 0 -> xyz=0.00 -0.02 -0.06 rpy=0 -2. 0
- joint r_litlefinger_x_gjoint: limit lower=-2.57 upper=0 effort=30 velocity=5 -> lower=0 upper=2 effort=30 velocity=10; origin xyz=0.00 0.02 -0.06 rpy=0 0 0 -> xyz=0.00 0.02 -0.06 rpy=0 -2 0

Commit message: nico traning update

File: myGym/envs/robots/nico/nico_grasp.urdf (robot description, URDF)
Before this commit: robot nico_upper_rh6d, 25 links, 24 joints
Links:
- link sight: geometry 

Commit message: oraculum gripper control update wip

File: myGym/envs/robots/nico/nico_grasp.urdf (robot description, URDF)
Before this commit: robot nico_upper_rh6d, 25 links, 24 joints
Links:
- link r_indexfinger: mass 0.000009 -> 0.01
- link r_littlefinger: mass 0.000009 -> 0.01
Joints:
- removed joint r_middlefinger_x
- added joint r_middlefinger_x_gjoint: type revolute, parent gripper, child r_middlefinger, origin xyz=0 0 -0.06 rpy=0 0 0, axis 0 1 0, limit lower=-2.57 upper=0 effort=30 velocity=5

File: myGym/envs/robots/nico/nico_grasper.urdf (robot description, URDF)
Before this commit: robot nico_upper_rh6d, 29 links, 28 joints
Links:
- link r_indexfinger: mass 0.000009 -> 0.01
- link r_littlefinger: mass 0.000009 -> 0.01
- link r_middlefinger: mass 0.000009 -> 0.01
- link right_thumb: mass 0.000009 -> 0.01
