Commit message: minor bugfixes

File: myGym/envs/robots/nico/nico_grasper.urdf (robot description, URDF)
Before this commit: robot nico_upper_rh6d, 29 links, 28 joints
Joints:
- removed joint r_thumb_x
- added joint r_thumb_x_joint: type revolute, parent gripper, child thumb_intermediate_link, origin xyz=0.008 -0.020 -0.028 rpy=-0.3 1 1.4, axis 2 1 0, limit lower=-2.57 upper=0 effort=30 velocity=100
- joint r_indexfinger_x_gjoint: limit lower=-2.57 upper=0 effort=30 velocity=1 -> lower=-2.57 upper=0 effort=30 velocity=10
- joint r_litlefinger_x_gjoint: limit lower=-2.57 upper=0 effort=30 velocity=1 -> lower=-2.57 upper=0 effort=30 velocity=10
- joint r_middlefingers_x_gjoint: limit lower=-2.57 upper=0 effort=30 velocity=1 -> lower=-2.57 upper=0 effort=30 velocity=10
- joint r_thumb_z_gjoint: limit lower=-2.57 upper=0 effort=30 velocity=1 -> lower=-2.57 upper=0 effort=70 velocity=100

Commit message: nico urdf repaired

File: myGym/envs/robots/nico/nico_grasper.urdf (robot description, URDF)
Before this commit: robot nico_upper_rh6d, 29 links, 28 joints
Joints:
- joint head_y: type revolute -> fixed
- joint head_z: type revolute -> fixed
- joint l_arm_x: type revolute -> fixed
- joint l_elbow_y: type revolute -> fixed
- joint l_indexfinger_x: type revolute -> fixed
- joint l_litlefinger_x: type revolute -> fixed
- joint l_middlefingers_x: type revolute -> fixed
- joint l_shoulder_y: type revolute -> fixed
- joint l_shoulder_z: type revolute -> fixed
- joint l_thumb_x: type revolute -> fixed
- joint l_thumb_z: type revolute -> fixed
- joint l_wrist_x: type revolute -> fixed
- joint l_wrist_z: type revolute -> fixed
- joint r_thumb_x_joint: type revolute -> fixed

Commit message: added gripper open/close thresholds for all robots based on gjoints limits

File: myGym/envs/robots/nico/nico_grasper.urdf (robot description, URDF)
Before this commit: robot nico_upper_rh6d, 29 links, 28 joints
Joints:
- joint r_thumb_z_gjoint: type revolute -> fixed

Commit message: nico oraculum works w/o topgrasp, testing model bug fixed

File: myGym/envs/robots/nico/nico_grasper.urdf (robot description, URDF)
Before this commit: robot nico_upper_rh6d, 29 links, 28 joints
Links:
- link r_indexfinger: geometry visual mesh filename=mesh/finger.stl
- link r_littlefinger: geometry visual mesh filename=mesh/finger.stl
- link r_middlefinger: geometry visual mesh filename=mesh/finger.stl

Commit message: update from master

File: myGym/envs/robots/nico/nico_grasper.urdf (robot description, URDF)
Before this commit: robot nico_upper_rh6d, 29 links, 28 joints
Links:
- link r_indexfinger: mass 0.000009 -> 0.01; geometry visual mesh filename=mesh/finger.stl
- link r_littlefinger: mass 0.000009 -> 0.01; geometry visual mesh filename=mesh/finger.stl
- link r_middlefinger: mass 0.000009 -> 0.01; geometry visual mesh filename=mesh/finger.stl
- link right_thumb: mass 0.000009 -> 0.01
Joints:
- removed joint r_thumb_x
- added joint r_thumb_x_joint: type fixed, parent gripper, child thumb_intermediate_link, origin xyz=0.008 -0.020 -0.028 rpy=-0.3 1 1.4, axis 2 1 0, limit lower=-2.57 upper=0 effort=30 velocity=100
- joint head_y: type revolute -> fixed
- joint head_z: type revolute -> fixed
- joint l_arm_x: type revolute -> fixed
- joint l_elbow_y: type revolute -> fixed
- joint l_indexfinger_x: type revolute -> fixed
- joint l_litlefinger_x: type revolute -> fixed
- joint l_middlefingers_x: type revolute -> fixed
- joint l_shoulder_y: type revolute -> fixed
- joint l_shoulder_z: type revolute -> fixed
- joint l_thumb_x: type revolute -> fixed
- joint l_thumb_z: type revolute -> fixed
- joint l_wrist_x: type revolute -> fixed
- joint l_wrist_z: type revolute -> fixed
- joint r_indexfinger_x_gjoint: limit lower=-2.57 upper=0 effort=30 velocity=1 -> lower=-2.57 upper=0 effort=30 velocity=10
- joint r_litlefinger_x_gjoint: limit lower=-2.57 upper=0 effort=30 velocity=1 -> lower=-2.57 upper=0 effort=30 velocity=10
- joint r_middlefingers_x_gjoint: limit lower=-2.57 upper=0 effort=30 velocity=1 -> lower=-2.57 upper=0 effort=30 velocity=10
- joint r_thumb_z_gjoint: limit lower=-2.57 upper=0 effort=30 velocity=1 -> lower=-2.57 upper=0 effort=70 velocity=100; type revolute -> fixed

Commit message: urf downgrad to old model - needs new training

File: myGym/envs/robots/nico/nico_grasper.urdf (robot description, URDF)
Before this commit: robot nico_upper_rh6d, 29 links, 28 joints
Links:
- link r_indexfinger: geometry collision mesh filename=mesh/finger.stl; visual mesh filename=mesh/finger.stl
- link r_littlefinger: geometry collision mesh filename=mesh/finger.stl; visual mesh filename=mesh/finger.stl
- link r_middlefinger: geometry collision mesh filename=mesh/finger.stl; visual mesh filename=mesh/finger.stl
Joints:
- joint r_thumb_z_gjoint: type fixed -> revolute

Commit message: oraculum works for g1, nico

File: myGym/envs/robots/nico/nico_grasper.urdf (robot description, URDF)
Before this commit: robot nico_upper_rh6d, 29 links, 28 joints
Links:
- link gripper: geometry visual mesh filename=mesh/right_palm.stl
- link right_thumb: geometry visual mesh filename=mesh/finger.stl

File: myGym/envs/robots/unitree/g1_mygym.urdf (robot description, URDF)
Before this commit: robot g1_29dof_with_hand_rev_1_0, 54 links, 53 joints
Links:
- link gripper: geometry visual mesh filename=meshes/right_hand_palm_link.STL
- link right_hand_index_0_link: geometry visual mesh filename=meshes/right_hand_index_0_link.STL
- link right_hand_index_1_link: geometry visual mesh filename=meshes/right_hand_index_1_link.STL
- link right_hand_middle_0_link: geometry visual mesh filename=meshes/right_hand_middle_0_link.STL
- link right_hand_middle_1_link: geometry visual mesh filename=meshes/right_hand_middle_1_link.STL
- link right_hand_thumb_0_link: geometry visual mesh filename=meshes/right_hand_thumb_0_link.STL
- link right_hand_thumb_1_link: geometry visual mesh filename=meshes/right_hand_thumb_1_link.STL
- link right_hand_thumb_2_link: geometry visual mesh filename=meshes/right_hand_thumb_2_link.STL
Joints:
- joint left_ankle_pitch_joint: type revolute -> fixed
- joint left_ankle_roll_joint: type revolute -> fixed
- joint left_elbow_joint: type revolute -> fixed
- joint left_hand_index_0_joint: type revolute -> fixed
- joint left_hand_index_1_joint: type revolute -> fixed
- joint left_hand_middle_0_joint: type revolute -> fixed
- joint left_hand_middle_1_joint: type revolute -> fixed
- joint left_hand_thumb_0_joint: type revolute -> fixed
- joint left_hand_thumb_1_joint: type revolute -> fixed
- joint left_hand_thumb_2_joint: type revolute -> fixed
- joint left_hip_pitch_joint: type revolute -> fixed
- joint left_hip_roll_joint: type revolute -> fixed
- joint left_hip_yaw_joint: type revolute -> fixed
- joint left_knee_joint: type revolute -> fixed
- joint left_shoulder_pitch_joint: type revolute -> fixed
- joint left_shoulder_roll_joint: type revolute -> fixed
- joint left_shoulder_yaw_joint: type revolute -> fixed
- joint left_wrist_pitch_joint: type revolute -> fixed
- joint left_wrist_roll_joint: type revolute -> fixed
- joint left_wrist_yaw_joint: type revolute -> fixed
- joint right_ankle_pitch_joint: type revolute -> fixed
- joint right_ankle_roll_joint: type revolute -> fixed
- joint right_hand_index_1_joint: type revolute -> fixed
- joint right_hand_middle_1_joint: type revolute -> fixed
- joint right_hand_thumb_0_joint: type revolute -> fixed
- joint right_hand_thumb_2_joint: type revolute -> fixed
- joint right_hip_pitch_joint: type revolute -> fixed
- joint right_hip_roll_joint: type revolute -> fixed
- joint right_hip_yaw_joint: type revolute -> fixed
- joint right_knee_joint: type revolute -> fixed

Commit message: robot origin update - new endeffector for leachy and reachy

File: myGym/envs/robots/nico/nico_grasper.urdf (robot description, URDF)
Before this commit: robot nico_upper_rh6d, 29 links, 28 joints
Joints:
- joint endeffector_joint: origin xyz=0.03 0.0 -0.05 rpy=1.57 0 1.57  -> xyz=0.03 0.0 -0.05 rpy=3.14 1.57 0

File: myGym/envs/robots/pollen/reachy/urdf/leachy.urdf (robot description, URDF)
Before this commit: robot Leachy_w_hand, 10 links, 9 joints
Links:
- added link l_wrist, mass 0.115; collision mesh filename=package://reachy/meshes/wrist-respondable.stl; visual mesh filename=package://reachy/meshes/wrist-visual.stl
- link base: geometry visual mesh filename=package://reachy/meshes/trunk-visual.stl
- link endeffector: mass 0.009 -> 0.0000332; geometry visual cylinder length=0.05 radius=0.002
- link gripper: mass 0.115 -> 0.009; geometry collision mesh filename=package://reachy/meshes/open_bionics_hand_left-respondable.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; visual mesh filename=package://reachy/meshes/open_bionics_hand_left-visual.stl
Joints:
- added joint endeffector_joint: type fixed, parent gripper, child endeffector, origin xyz=0.0 -0.05 -0.12 rpy=-1.57 0 0
- joint l_forearm_yaw_rjoint: child gripper -> l_wrist
- joint l_wrist_pitch_rjoint: child endeffector -> gripper; parent gripper -> l_wrist

File: myGym/envs/robots/pollen/reachy/urdf/reachy.urdf (robot description, URDF)
Before this commit: robot Reachy, 12 links, 11 joints
Links:
- removed link ball
- added link wrist_hand, mass 0.009; collision mesh filename=package://reachy/meshes/wrist-hand-respondable.stl; visual mesh filename=package://reachy/meshes/wrist-hand-visual.stl
- link base: geometry visual mesh filename=package://reachy/meshes/trunk-visual.stl
- link endeffector: mass None -> 0.0000332; geometry visual cylinder length=0.05 radius=0.002
- link gripper: mass 0.009 -> 0.090; geometry collision mesh filename=package://reachy/meshes/ball-tip-respondable.stl; visual mesh filename=package://reachy/meshes/ball-tip-visual.stl
Joints:
- joint endeffector_joint: origin xyz=0 0.0 -0.13 rpy=0 0 0 -> xyz=0.0 0.0 -0.12 rpy=0 0 -1.57
- joint head_yaw: origin xyz=0 0 0.13775 rpy=0 0 0 -> xyz=0 0 0.43775 rpy=0 0 0
- joint shoulder_pitch_rjoint: origin xyz=0 -0.14 0 rpy=0 -1.5 0 -> xyz=0 -0.14 0.3 rpy=0 -1.5 0
- joint wrist_pitch_rjoint: child gripper -> wrist_hand
- joint wrist_roll_rjoint: child ball -> gripper; parent gripper -> wrist_hand
