Commit message: train G1 scripts

File: myGym/envs/robots/unitree/g1_mygym.urdf (robot description, URDF)
Before this commit: robot g1_29dof_with_hand_rev_1_0, 54 links, 53 joints
Joints:
- removed joint right_elbow_joint
- removed joint right_hand_index_0_joint
- removed joint right_hand_middle_0_joint
- removed joint right_hand_thumb_1_joint
- removed joint right_shoulder_pitch_joint
- removed joint right_shoulder_roll_joint
- removed joint right_shoulder_yaw_joint
- removed joint right_wrist_pitch_joint
- removed joint right_wrist_roll_joint
- removed joint right_wrist_yaw_joint
- removed joint waist_pitch_joint
- removed joint waist_roll_joint
- removed joint waist_yaw_joint
- added joint right_elbow_rjoint: type revolute, parent right_shoulder_yaw_link, child right_elbow_link, origin xyz=0.015783 0 -0.080518 rpy=0 0 0, axis 0 1 0, limit lower=-1.0472 upper=2.0944 effort=25 velocity=37
- added joint right_hand_index_0_gjoint: type revolute, parent right_hand_palm_link, child right_hand_index_0_link, origin xyz=0.0777 -0.0016 0.0285 rpy=0 0 0, axis 0 0 1, limit lower=0 upper=1.57079632 effort=1.4 velocity=12
- added joint right_hand_middle_0_gjoint: type revolute, parent right_hand_palm_link, child right_hand_middle_0_link, origin xyz=0.0777 -0.0016 -0.0285 rpy=0 0 0, axis 0 0 1, limit lower=0 upper=1.57079632 effort=1.4 velocity=12
- added joint right_hand_thumb_1_gjoint: type revolute, parent right_hand_thumb_0_link, child right_hand_thumb_1_link, origin xyz=-0.0025 0.0193 0 rpy=0 0 0, axis 0 0 1, limit lower=-1.04719755 upper=0.72431163 effort=1.4 velocity=12
- added joint right_shoulder_pitch_rjoint: type revolute, parent torso_link, child right_shoulder_pitch_link, origin xyz=0.0039563 -0.10021 0.24778 rpy=-0.27931 5.4949E-05 0.00019159, axis 0 1 0, limit lower=-3.0892 upper=2.6704 effort=25 velocity=37
- added joint right_shoulder_roll_rjoint: type revolute, parent right_shoulder_pitch_link, child right_shoulder_roll_link, origin xyz=0 -0.038 -0.013831 rpy=0.27925 0 0, axis 1 0 0, limit lower=-2.2515 upper=1.5882 effort=25 velocity=37
- added joint right_shoulder_yaw_rjoint: type revolute, parent right_shoulder_roll_link, child right_shoulder_yaw_link, origin xyz=0 -0.00624 -0.1032 rpy=0 0 0, axis 0 0 1, limit lower=-2.618 upper=2.618 effort=25 velocity=37
- added joint right_wrist_pitch_rjoint: type revolute, parent right_wrist_roll_link, child right_wrist_pitch_link, origin xyz=0.038 0 0 rpy=0 0 0, axis 0 1 0, limit lower=-1.614429558 upper=1.614429558 effort=5 velocity=22
- added joint right_wrist_roll_rjoint: type revolute, parent right_elbow_link, child right_wrist_roll_link, origin xyz=0.100 -0.00188791 -0.010 rpy=0 0 0, axis 1 0 0, limit lower=-1.972222054 upper=1.972222054 effort=25 velocity=37
- added joint right_wrist_yaw_rjoint: type revolute, parent right_wrist_pitch_link, child right_wrist_yaw_link, origin xyz=0.046 0 0 rpy=0 0 0, axis 0 0 1, limit lower=-1.614429558 upper=1.614429558 effort=5 velocity=22
- added joint waist_pitch_rjoint: type revolute, parent waist_roll_link, child torso_link, origin xyz=0 0 0 rpy=0 0 0, axis 0 1 0, limit lower=-0.52 upper=0.52 effort=50 velocity=37
- added joint waist_roll_rjoint: type revolute, parent waist_yaw_link, child waist_roll_link, origin xyz=-0.0039635 0 0.044 rpy=0 0 0, axis 1 0 0, limit lower=-0.52 upper=0.52 effort=50 velocity=37
- added joint waist_yaw_rjoint: type revolute, parent pelvis, child waist_yaw_link, origin xyz=0 0 0 rpy=0 0 0, axis 0 0 1, limit lower=-2.618 upper=2.618 effort=88 velocity=32

Commit message: config update

File: myGym/envs/robots/unitree/g1_mygym.urdf (robot description, URDF)
Before this commit: robot g1_29dof_with_hand_rev_1_0, 54 links, 53 joints
Links:
- removed link right_hand_palm_link
- added link gripper, mass 0.37283854; collision mesh filename=meshes/right_hand_palm_link.STL; visual mesh filename=meshes/right_hand_palm_link.STL
Joints:
- joint endeffector_joint: parent right_hand_palm_link -> gripper
- joint right_hand_index_0_gjoint: parent right_hand_palm_link -> gripper
- joint right_hand_middle_0_gjoint: parent right_hand_palm_link -> gripper
- joint right_hand_palm_joint: child right_hand_palm_link -> gripper
- joint right_hand_thumb_0_joint: parent right_hand_palm_link -> gripper
