Commit message: robt.py update, g1 urdf update

File: myGym/envs/robots/unitree/g1_mygym_full.urdf (robot description, URDF)
Before this commit: robot g1_29dof_with_hand_rev_1_0, 56 links, 55 joints
Links:
- link gripper: geometry visual mesh filename=meshes/right_hand_palm_link.STL
- link right_hand_index_0_link: geometry visual mesh filename=meshes/right_hand_index_0_link.STL
- link right_hand_index_1_link: geometry visual mesh filename=meshes/right_hand_index_1_link.STL
- link right_hand_middle_0_link: geometry visual mesh filename=meshes/right_hand_middle_0_link.STL
- link right_hand_middle_1_link: geometry visual mesh filename=meshes/right_hand_middle_1_link.STL
- link right_hand_thumb_0_link: geometry visual mesh filename=meshes/right_hand_thumb_0_link.STL
- link right_hand_thumb_1_link: geometry visual mesh filename=meshes/right_hand_thumb_1_link.STL
- link right_hand_thumb_2_link: geometry visual mesh filename=meshes/right_hand_thumb_2_link.STL
Joints:
- removed joint left_hip_pitch_joint
- removed joint left_hip_roll_joint
- removed joint left_hip_yaw_joint
- removed joint right_ankle_pitch_joint
- removed joint right_ankle_roll_joint
- removed joint right_knee_joint
- added joint left_hip_pitch_rjoint: type revolute, parent pelvis, child left_hip_pitch_link, origin xyz=0 0.064452 -0.1027 rpy=0 0 0, axis 0 1 0, limit lower=-2.5307 upper=2.8798 effort=88 velocity=32
- added joint left_hip_roll_rjoint: type fixed, parent left_hip_pitch_link, child left_hip_roll_link, origin xyz=0 0.052 -0.030465 rpy=0 -0.1749 0, axis 1 0 0, limit lower=-0.5236 upper=2.9671 effort=139 velocity=20
- added joint left_hip_yaw_rjoint: type revolute, parent left_hip_roll_link, child left_hip_yaw_link, origin xyz=0.025001 0 -0.12412 rpy=0 0 0, axis 0 0 1, limit lower=-2.7576 upper=2.7576 effort=88 velocity=32
- added joint right_ankle_pitch_rjoint: type revolute, parent right_knee_link, child right_ankle_pitch_link, origin xyz=0 9.4445E-05 -0.30001 rpy=0 0 0, axis 0 1 0, limit lower=-0.87267 upper=0.5236 effort=50 velocity=37
- added joint right_ankle_roll_rjoint: type fixed, parent right_ankle_pitch_link, child right_ankle_roll_link, origin xyz=0 0 -0.017558 rpy=0 0 0, axis 1 0 0, limit lower=-0.2618 upper=0.2618 effort=50 velocity=37
- added joint right_knee_rjoint: type fixed, parent right_hip_yaw_link, child right_knee_link, origin xyz=-0.078273 -0.0021489 -0.17734 rpy=0 0.1749 0, axis 0 1 0, limit lower=-0.087267 upper=2.8798 effort=139 velocity=20
- joint left_ankle_pitch_rjoint: type fixed -> revolute
- joint right_hip_pitch_rjoint: type fixed -> revolute
- joint right_hip_yaw_rjoint: type fixed -> revolute
- joint waist_pitch_rjoint: type fixed -> revolute
- joint waist_roll_rjoint: type fixed -> revolute
- joint waist_yaw_rjoint: type fixed -> revolute
