Commit message: g1 6DOF gripper update

File: myGym/envs/robots/unitree/g1_mygym6DOFG.urdf (robot description, URDF)
Before this commit: robot g1_29dof_with_hand_rev_1_0, 57 links, 56 joints
Joints:
- removed joint right_hand_index_1_joint
- removed joint right_hand_middle_1_joint
- removed joint right_hand_thumb_2_joint
- added joint right_hand_index_1_gjoint: type revolute, parent right_hand_index_0_link, child right_hand_index_1_link, origin xyz=0.0458 0 0 rpy=0 0 0, axis 0 0 1, limit lower=0 upper=1.74532925 effort=1.4 velocity=12
- added joint right_hand_middle_1_gjoint: type revolute, parent right_hand_middle_0_link, child right_hand_middle_1_link, origin xyz=0.0458 0 0 rpy=0 0 0, axis 0 0 1, limit lower=0 upper=1.74532925 effort=1.4 velocity=12
- added joint right_hand_thumb_2_gjoint: type revolute, parent right_hand_thumb_1_link, child right_hand_thumb_2_link, origin xyz=0 0.0458 0 rpy=0 0 0, axis 0 0 1, limit lower=-1.74532925 upper=0 effort=1.4 velocity=12
