Commit message: panda oraculum WIP

File: myGym/envs/robots/franka_emika/panda_bullet/panda.urdf (robot description, URDF)
Before this commit: robot panda, 13 links, 12 joints
Links:
- link panda_leftfinger: geometry visual mesh filename=package://meshes/visual/finger.obj
- link panda_rightfinger: geometry visual mesh filename=package://meshes/visual/finger.obj
