Commit message: visualize_robot_ik WORKING - yumi urdf end efector update

File: myGym/envs/robots/abb/yumi/urdf/yumi.urdf (robot description, URDF)
Before this commit: robot yumi, 23 links, 22 joints
Links:
- added link gripper_l_finger_l, mass 0.01; collision mesh filename=package://yumi/meshes/gripper/coarse/finger.stl; visual mesh filename=package://yumi/meshes/gripper/finger.stl
- link endeffector: mass 0.01 -> 0.0000332; geometry visual cylinder length=0.05 radius=0.002
Joints:
- added joint endeffector_joint: type fixed, parent gripper_r_base, child endeffector, origin xyz=0.0 0.0 0.1 rpy=3.14 0 0
- joint gripper_l_gjoint_m: child endeffector -> gripper_l_finger_l

Commit message: urdf update od yumi,panda,kuka,nico and pepper urdf - top grasp end effector orientation aligned for all robots - ready for oraculum

File: myGym/envs/robots/abb/yumi/urdf/yumi.urdf (robot description, URDF)
Before this commit: robot yumi, 24 links, 23 joints
Links:
- removed link world
Joints:
- removed joint world_joint
- joint endeffector_joint: origin xyz=0.0 0.0 0.1 rpy=3.14 0 0 -> xyz=0.0 0.0 0.12 rpy=3.14 0 0
- joint gripper_l_gjoint: type prismatic -> fixed
- joint gripper_l_gjoint_m: type prismatic -> fixed

File: myGym/envs/robots/nico/nico_grasper.urdf (robot description, URDF)
Before this commit: robot nico_upper_rh6d, 29 links, 28 joints
Joints:
- removed joint r_arm_x
- removed joint r_elbow_y
- removed joint r_indexfinger_x
- removed joint r_litlefinger_x
- removed joint r_middlefingers_x
- removed joint r_shoulder_y
- removed joint r_shoulder_z
- removed joint r_thumb_z
- removed joint r_wrist_x
- removed joint r_wrist_z
- added joint gjoint_r_indexfinger_x: type revolute, parent right_palm, child r_indexfinger, origin xyz=0.00 -0.02 -0.06 rpy=0 0 0, axis 0 1 0, limit lower=-2.57 upper=0 effort=30 velocity=1
- added joint gjoint_r_littlefinger_x: type revolute, parent right_palm, child r_littlefinger, origin xyz=0.00 0.02 -0.06 rpy=0 0 0, axis 0 1 0, limit lower=-2.57 upper=0 effort=30 velocity=1
- added joint gjoint_r_middlefingers_x: type revolute, parent right_palm, child r_middlefinger, origin xyz=0 0 -0.06 rpy=0 0 0, axis 0 1 0, limit lower=-2.57 upper=0 effort=30 velocity=1
- added joint gjoint_r_thumb_z: type revolute, parent thumb_intermediate_link, child right_thumb, origin xyz=0 0 0 rpy=0 0 0, axis 0 1 0, limit lower=-2.57 upper=0 effort=30 velocity=1
- added joint rjoint_r_arm_x: type revolute, parent right_collarbone, child right_upper_arm, origin xyz=0.00 -0.073 -0.023 rpy=0 0 0, axis -1 0 0, limit lower=0 upper=1.2217 effort=30 velocity=1
- added joint rjoint_r_elbow_y: type revolute, parent right_upper_arm, child right_lower_arm, origin xyz=0.0 0 -0.17 rpy=0 3.14 0, axis 0 1 0, limit lower=0.8726 upper=3.1416 effort=30 velocity=1
- added joint rjoint_r_shoulder_y: type revolute, parent right_shoulder, child right_collarbone, origin xyz=-0.021 -0.023 0.033 rpy=0 0 0, axis 0 -1 0, limit lower=-1.5707 upper=3.1416 effort=30 velocity=1
- added joint rjoint_r_shoulder_z: type revolute, parent torso, child right_shoulder, origin xyz=0.000 -0.040 0.23 rpy=0 0 0, axis 0 0 1, limit lower=-0.4363 upper=1.3963 effort=30 velocity=1
- added joint rjoint_r_wrist_x: type revolute, parent right_wrist, child right_palm, origin xyz=0 0 -0.10 rpy=0 0 0, axis 0 -1 0, limit lower=-0.785398163 upper=0.785398163 effort=30 velocity=1
- added joint rjoint_r_wrist_z: type revolute, parent right_lower_arm, child right_wrist, origin xyz=0 0 -0.105 rpy=0 0 1.5707, axis 0 0 1, limit lower=-1.5707 upper=1.5707 effort=30 velocity=1

Commit message: cheerypick from PRAG brabch - urdf endeffector update for various robots

File: myGym/envs/robots/abb/yumi/urdf/yumi.urdf (robot description, URDF)
Before this commit: robot yumi, 23 links, 22 joints
Links:
- removed link world
- added link gripper_l_finger_l, mass 0.01; collision mesh filename=package://yumi/meshes/gripper/coarse/finger.stl; visual mesh filename=package://yumi/meshes/gripper/finger.stl
- link endeffector: mass 0.01 -> 0.0000332; geometry visual cylinder length=0.05 radius=0.002
Joints:
- removed joint world_joint
- added joint endeffector_joint: type fixed, parent gripper_r_base, child endeffector, origin xyz=0.0 0.0 0.12 rpy=3.14 0 0
- joint gripper_l_gjoint: type prismatic -> fixed
- joint gripper_l_gjoint_m: child endeffector -> gripper_l_finger_l; type prismatic -> fixed

File: myGym/envs/robots/franka_emika/panda/urdf/panda1.urdf (robot description, URDF)
Before this commit: robot panda, 14 links, 13 joints
Links:
- link endeffector: mass None -> 0.0000332; geometry visual cylinder length=0.05 radius=0.002
Joints:
- joint endeffector_joint: origin xyz=0 0.0 0.1 rpy=0 0 0 -> xyz=0.0 0.0 0.12 rpy=3.14 0 0

File: myGym/envs/robots/franka_emika/panda/urdf/panda_cgripper.urdf (robot description, URDF)
Before this commit: robot panda, 22 links, 21 joints
Links:
- link endeffector: mass None -> 0.0000332; geometry visual cylinder length=0.05 radius=0.002
Joints:
- joint endeffector_joint: origin xyz=0 0.0 0.152 rpy=0 0 0 -> xyz=0.0 0.0 0.12 rpy=3.14 0 0

File: myGym/envs/robots/franka_emika/panda_bullet/panda.urdf (robot description, URDF)
Before this commit: robot panda, 13 links, 12 joints
Links:
- link endeffector: mass None -> 0.0000332; geometry visual cylinder length=0.05 radius=0.002
Joints:
- joint endeffector_joint: origin xyz=0 0.0 0.1 rpy=0 0 0 -> xyz=0.0 0.0 0.12 rpy=3.14 0 0

File: myGym/envs/robots/franka_emika/panda_moveit/urdf/panda2.urdf (robot description, URDF)
Before this commit: robot panda, 13 links, 12 joints
Links:
- link endeffector: mass None -> 0.0000332; geometry visual cylinder length=0.05 radius=0.002
Joints:
- joint endeffector_joint: origin xyz=0 0.0 0.1 rpy=0 0 0 -> xyz=0.0 0.0 0.12 rpy=3.14 0 0

File: myGym/envs/robots/kuka_gripper/kuka_gripper.urdf (robot description, URDF)
Before this commit: robot kuka_gripper, 18 links, 17 joints
Links:
- link endeffector: mass None -> 0.0000332; geometry visual cylinder length=0.05 radius=0.002
Joints:
- joint endeffector_joint: origin xyz=0 0.0 0.1 rpy=0 0 0 -> xyz=0.0 0.0 0.12 rpy=3.14 0 0

File: myGym/envs/robots/pepper/pepper.urdf (robot description, URDF)
Before this commit: robot JulietteY20MP, 99 links, 98 joints
Links:
- removed link r_gripper
- removed link r_hand
- added link RFinger23_link , mass 2e-03; collision mesh filename=meshes/pepper/PhalaxEnd.obj scale=1 1 1; visual mesh filename=meshes/pepper/PhalaxEnd.obj scale=1 1 1
- link endeffector: mass 2e-03 -> 0.0000332; geometry visual cylinder length=0.05 radius=0.002
Joints:
- removed joint LGripper_gjoint
- removed joint RFinger11
- removed joint RFinger21_rjoint
- removed joint RFinger22_rjoint
- removed joint RFinger31
- removed joint RFinger41
- removed joint RGripper_gjoint
- removed joint RHand
- added joint LGripper_joint: type fixed, parent l_wrist, child gripper, origin xyz=0.07 0.0 -0.01802319018 rpy=-3.14 0.0 -1.57, axis 0 0 0
- added joint RFinger11_gjoint: type revolute, parent r_wrist, child RFinger11_link, origin xyz=0.0821 0.0268 0.004 rpy=1.39757 1.04064 0.0334335, axis 0 0 1.0, limit lower=0.0 upper=0.872665 effort=0.144 velocity=12.56, mimic joint=RHand multiplier=0.872665 offset=0
- added joint RFinger21_gjoint: type revolute, parent r_wrist, child RFinger21_link, origin xyz=0.0873 0.0073 0.006 rpy=1.5708 1.0472 0.061086, axis 0 0 1.0, limit lower=0.0 upper=0.872665 effort=0.144 velocity=12.56, mimic joint=RHand multiplier=0.872665 offset=0
- added joint RFinger22_joint: type fixed, parent RFinger21_link, child RFinger22_link, origin xyz=0.018 0 0 rpy=0 0 -1.0472, axis 0 0 1.0, limit lower=0.0 upper=0.872665 effort=0.144 velocity=12.56, mimic joint=RHand multiplier=0.872665 offset=0
- added joint RFinger23_link_joint: type fixed, parent RFinger22_link, child RFinger23_link , origin xyz=0.018 0 0 rpy=0 0 -1.0472, axis 0 0 1.0, limit lower=0.0 upper=0.872665 effort=0.144 velocity=12.56, mimic joint=RHand multiplier=0.872665 offset=0
- added joint RFinger31_gjoint: type revolute, parent r_wrist, child RFinger31_link, origin xyz=0.0833 -0.0123 0.004 rpy=1.67523 1.04483 0.029316, axis 0 0 1.0, limit lower=0.0 upper=0.872665 effort=0.144 velocity=12.56, mimic joint=RHand multiplier=0.872665 offset=0
- added joint RFinger41_gjoint: type revolute, parent r_wrist, child RFinger41_link, origin xyz=0.074 -0.0309 0 rpy=1.74402 1.04064 -0.0683394, axis 0 0 1.0, limit lower=0.0 upper=0.872665 effort=0.144 velocity=12.56, mimic joint=RHand multiplier=0.872665 offset=0
- joint endeffector_joint: axis 0 0 1.0 -> (none); limit lower=0.0 upper=0.872665 effort=0.144 velocity=12.56 -> (none); mimic joint=RHand multiplier=0.872665 offset=0 -> (none); origin xyz=0.018 0 0 rpy=0 0 -1.0472 -> xyz=0.07 0.0 -0.04 rpy=0 0 0; parent RFinger22_link -> r_wrist

Commit message: ALL ROBOTSPOSITIO

File: myGym/envs/robots/abb/yumi/urdf/yumi.urdf (robot description, URDF)
Before this commit: robot yumi, 23 links, 22 joints
Links:
- added link ee_x_axis; visual cylinder length=0.06 radius=0.002
- added link ee_y_axis; visual cylinder length=0.06 radius=0.002
- added link ee_z_axis; visual cylinder length=0.06 radius=0.002
- link endeffector: mass 0.0000332 -> None; geometry visual sphere radius=0.005
Joints:
- added joint ee_x_axis_joint: type fixed, parent gripper, child ee_x_axis, origin xyz=0.0 0.0 0.12 rpy=3.14 0 0
- added joint ee_y_axis_joint: type fixed, parent gripper, child ee_y_axis, origin xyz=0.0 0.0 0.12 rpy=3.14 0 0
- added joint ee_z_axis_joint: type fixed, parent gripper, child ee_z_axis, origin xyz=0.0 0.0 0.12 rpy=3.14 0 0
- joint endeffector_joint: parent gripper_r_base -> gripper
- joint gripper_l_gjoint: type fixed -> prismatic
- joint gripper_l_gjoint_m: type fixed -> prismatic

File: myGym/envs/robots/hsr/hsrb4s.urdf (robot description, URDF)
Before this commit: robot hsrb, 45 links, 44 joints
Joints:
- removed joint head_center_camera_frame_rjoint
- removed joint head_l_stereo_camera_gazebo_frame_rjoint
- removed joint head_r_stereo_camera_gazebo_frame_rjoint
- added joint head_center_camera_frame_joint: type fixed, parent head_tilt_link, child head_center_camera_frame, origin xyz=0.0195 0.0 0.061 rpy=-1.5707963268 0.0 -1.5707963268
- added joint head_l_stereo_camera_gazebo_frame_joint: type fixed, parent head_l_stereo_camera_link, child head_l_stereo_camera_gazebo_frame, origin xyz=0 0 0 rpy=1.5707963268 -1.5707963268 0.0
- added joint head_r_stereo_camera_gazebo_frame_joint: type fixed, parent head_r_stereo_camera_link, child head_r_stereo_camera_gazebo_frame, origin xyz=0 0 0 rpy=1.5707963268 -1.5707963268 0.0
- joint base_l_drive_wheel_rjoint: type continuous -> fixed
- joint base_l_passive_wheel_x_frame_rjoint: type continuous -> fixed
- joint base_l_passive_wheel_y_frame_rjoint: type continuous -> fixed
- joint base_l_passive_wheel_z_rjoint: type continuous -> fixed
- joint base_r_drive_wheel_rjoint: type continuous -> fixed
- joint base_r_passive_wheel_x_frame_rjoint: type continuous -> fixed
- joint base_r_passive_wheel_y_frame_rjoint: type continuous -> fixed
- joint base_r_passive_wheel_z_rjoint: type continuous -> fixed
- joint base_roll_rjoint: type continuous -> fixed

File: myGym/envs/robots/tiago/tiago_dual_mygym.urdf (robot description, URDF)
Before this commit: robot tiago_dual_mygym, 37 links, 36 joints
Links:
- added link ee_x_axis; visual cylinder length=0.06 radius=0.002
- added link ee_y_axis; visual cylinder length=0.06 radius=0.002
- added link ee_z_axis; visual cylinder length=0.06 radius=0.002
- link endeffector: mass 0.0000332 -> None; geometry visual sphere radius=0.005
Joints:
- added joint ee_x_axis_joint: type fixed, parent gripper, child ee_x_axis, origin xyz=0.0 0.0 -0.2 rpy=3.14 0 0
- added joint ee_y_axis_joint: type fixed, parent gripper, child ee_y_axis, origin xyz=0.0 0.0 -0.2 rpy=3.14 0 0
- added joint ee_z_axis_joint: type fixed, parent gripper, child ee_z_axis, origin xyz=0.0 0.0 -0.2 rpy=3.14 0 0
- joint endeffector_joint: origin xyz=0.0 0.0 -0.20 rpy=0 0 -3.1415 -> xyz=0.0 0.0 -0.2 rpy=0 0 0

File: myGym/envs/robots/tiago/tiago_dual_mygym_fix.urdf (robot description, URDF)
Before this commit: robot tiago_dual_mygym, 37 links, 36 joints
Links:
- added link ee_x_axis; visual cylinder length=0.06 radius=0.002
- added link ee_y_axis; visual cylinder length=0.06 radius=0.002
- added link ee_z_axis; visual cylinder length=0.06 radius=0.002
- link endeffector: mass 0.0000332 -> None; geometry visual sphere radius=0.005
Joints:
- added joint ee_x_axis_joint: type fixed, parent gripper, child ee_x_axis, origin xyz=0.0 0.0 -0.2 rpy=3.14 0 0
- added joint ee_y_axis_joint: type fixed, parent gripper, child ee_y_axis, origin xyz=0.0 0.0 -0.2 rpy=3.14 0 0
- added joint ee_z_axis_joint: type fixed, parent gripper, child ee_z_axis, origin xyz=0.0 0.0 -0.2 rpy=3.14 0 0
- joint endeffector_joint: origin xyz=0.0 0.0 -0.20 rpy=0 0 -3.1415 -> xyz=0.0 0.0 -0.2 rpy=0 0 0

File: myGym/envs/robots/tiago/tiago_dual_mygym_rot.urdf (robot description, URDF)
Before this commit: robot tiago_dual_mygym, 37 links, 36 joints
Links:
- added link ee_x_axis; visual cylinder length=0.06 radius=0.002
- added link ee_y_axis; visual cylinder length=0.06 radius=0.002
- added link ee_z_axis; visual cylinder length=0.06 radius=0.002
- link endeffector: mass 0.0000332 -> None; geometry visual sphere radius=0.005
Joints:
- added joint ee_x_axis_joint: type fixed, parent gripper, child ee_x_axis, origin xyz=0.0 0.0 -0.2 rpy=3.14 0 0
- added joint ee_y_axis_joint: type fixed, parent gripper, child ee_y_axis, origin xyz=0.0 0.0 -0.2 rpy=3.14 0 0
- added joint ee_z_axis_joint: type fixed, parent gripper, child ee_z_axis, origin xyz=0.0 0.0 -0.2 rpy=3.14 0 0
- joint endeffector_joint: origin xyz=0.0 0.0 -0.20 rpy=0 0 -3.1415 -> xyz=0.0 0.0 -0.2 rpy=0 0 0

File: myGym/envs/robots/tiago/tiago_dual_mygym_rotslide.urdf (robot description, URDF)
Before this commit: robot tiago_dual_mygym, 37 links, 36 joints
Links:
- added link ee_x_axis; visual cylinder length=0.06 radius=0.002
- added link ee_y_axis; visual cylinder length=0.06 radius=0.002
- added link ee_z_axis; visual cylinder length=0.06 radius=0.002
- link endeffector: mass 0.0000332 -> None; geometry visual sphere radius=0.005
Joints:
- added joint ee_x_axis_joint: type fixed, parent gripper, child ee_x_axis, origin xyz=0.0 0.0 -0.2 rpy=3.14 0 0
- added joint ee_y_axis_joint: type fixed, parent gripper, child ee_y_axis, origin xyz=0.0 0.0 -0.2 rpy=3.14 0 0
- added joint ee_z_axis_joint: type fixed, parent gripper, child ee_z_axis, origin xyz=0.0 0.0 -0.2 rpy=3.14 0 0
- joint endeffector_joint: origin xyz=0.0 0.0 -0.20 rpy=0 0 -3.1415 -> xyz=0.0 0.0 -0.2 rpy=0 0 0

File: myGym/envs/robots/tiago/tiago_dual_mygym_rotslide2.urdf (robot description, URDF)
Before this commit: robot tiago_dual_mygym, 38 links, 37 joints
Links:
- added link ee_x_axis; visual cylinder length=0.06 radius=0.002
- added link ee_y_axis; visual cylinder length=0.06 radius=0.002
- added link ee_z_axis; visual cylinder length=0.06 radius=0.002
- link endeffector: mass 0.0000332 -> None; geometry visual sphere radius=0.005
Joints:
- added joint ee_x_axis_joint: type fixed, parent gripper, child ee_x_axis, origin xyz=0.0 0.0 -0.2 rpy=3.14 0 0
- added joint ee_y_axis_joint: type fixed, parent gripper, child ee_y_axis, origin xyz=0.0 0.0 -0.2 rpy=3.14 0 0
- added joint ee_z_axis_joint: type fixed, parent gripper, child ee_z_axis, origin xyz=0.0 0.0 -0.2 rpy=3.14 0 0
- joint baseslide_rjoint2: limit lower=-0.5 upper=0.5 effort=16 velocity=0.05 -> lower=-1.0 upper=0.0 effort=16 velocity=0.05
- joint endeffector_joint: origin xyz=0.0 0.0 -0.20 rpy=0 0 -3.1415 -> xyz=0.0 0.0 -0.2 rpy=0 0 0

File: myGym/envs/robots/tiago/tiago_pal_gripper.urdf (robot description, URDF)
Before this commit: robot tiago, 48 links, 47 joints
Links:
- added link ee_x_axis; visual cylinder length=0.06 radius=0.002
- added link ee_y_axis; visual cylinder length=0.06 radius=0.002
- added link ee_z_axis; visual cylinder length=0.06 radius=0.002
- link endeffector: geometry visual sphere radius=0.005
Joints:
- removed joint endeffector_gjoint
- removed joint torso_lift_joint
- added joint ee_x_axis_joint: type fixed, parent gripper, child ee_x_axis, origin xyz=0.05 0.0 0.0 rpy=0 1.57 0
- added joint ee_y_axis_joint: type fixed, parent gripper, child ee_y_axis, origin xyz=0.05 0.0 0.0 rpy=0 1.57 0
- added joint ee_z_axis_joint: type fixed, parent gripper, child ee_z_axis, origin xyz=0.05 0.0 0.0 rpy=0 1.57 0
- added joint endeffector_joint: type fixed, parent gripper, child endeffector, origin xyz=0.05 0.0 0.0 rpy=0 -1.57 0
- added joint torso_lift_rjoint: type prismatic, parent torso_fixed_link, child torso_lift_link, origin xyz=0.0 0.0 0.597 rpy=0.0 0.0 0.0, axis 0 0 1, limit lower=0 upper=0.35 effort=2000 velocity=0.07

File: myGym/envs/robots/unitree/g1_mygym.urdf (robot description, URDF)
Before this commit: robot g1_29dof_with_hand_rev_1_0, 54 links, 53 joints
Links:
- added link ee_x_axis; visual cylinder length=0.06 radius=0.002
- added link ee_y_axis; visual cylinder length=0.06 radius=0.002
- added link ee_z_axis; visual cylinder length=0.06 radius=0.002
- link endeffector: mass 0.0000332 -> None; geometry visual sphere radius=0.005
Joints:
- added joint ee_x_axis_joint: type fixed, parent gripper, child ee_x_axis, origin xyz=0.07 0.07 0.0 rpy=-1.57 -1.57 0
- added joint ee_y_axis_joint: type fixed, parent gripper, child ee_y_axis, origin xyz=0.07 0.07 0.0 rpy=-1.57 -1.57 0
- added joint ee_z_axis_joint: type fixed, parent gripper, child ee_z_axis, origin xyz=0.07 0.07 0.0 rpy=-1.57 -1.57 0

File: myGym/envs/robots/unitree/g1_mygym_dual.urdf (robot description, URDF)
Before this commit: robot g1_29dof_with_hand_rev_1_0, 54 links, 53 joints
Links:
- removed link right_hand_palm_link
- added link ee_x_axis; visual cylinder length=0.06 radius=0.002
- added link ee_y_axis; visual cylinder length=0.06 radius=0.002
- added link ee_z_axis; visual cylinder length=0.06 radius=0.002
- added link gripper, mass 0.37283854; collision mesh filename=meshes/right_hand_palm_link.STL; visual mesh filename=meshes/right_hand_palm_link.STL
- link endeffector: mass 0.0000332 -> None; geometry visual sphere radius=0.005
Joints:
- added joint ee_x_axis_joint: type fixed, parent gripper, child ee_x_axis, origin xyz=0.07 0.07 0.0 rpy=-1.57 -1.57 0
- added joint ee_y_axis_joint: type fixed, parent gripper, child ee_y_axis, origin xyz=0.07 0.07 0.0 rpy=-1.57 -1.57 0
- added joint ee_z_axis_joint: type fixed, parent gripper, child ee_z_axis, origin xyz=0.07 0.07 0.0 rpy=-1.57 -1.57 0
- joint endeffector_joint: parent right_hand_palm_link -> gripper
- joint right_hand_index_0_gjoint: parent right_hand_palm_link -> gripper
- joint right_hand_middle_0_gjoint: parent right_hand_palm_link -> gripper
- joint right_hand_palm_joint: child right_hand_palm_link -> gripper
- joint right_hand_thumb_0_joint: parent right_hand_palm_link -> gripper

File: myGym/envs/robots/universal_robots/urdf/ur10.urdf (robot description, URDF)
Before this commit: robot ur10, 13 links, 12 joints
Links:
- added link ee_x_axis; visual cylinder length=0.06 radius=0.002
- added link ee_y_axis; visual cylinder length=0.06 radius=0.002
- added link ee_z_axis; visual cylinder length=0.06 radius=0.002
- link endeffector: geometry visual sphere radius=0.005
Joints:
- added joint ee_x_axis_joint: type fixed, parent gripper, child ee_x_axis, origin xyz=0.05 0.0 0.0 rpy=0 1.57 0
- added joint ee_y_axis_joint: type fixed, parent gripper, child ee_y_axis, origin xyz=0.05 0.0 0.0 rpy=0 1.57 0
- added joint ee_z_axis_joint: type fixed, parent gripper, child ee_z_axis, origin xyz=0.05 0.0 0.0 rpy=0 1.57 0
- joint endeffector_joint: origin xyz=0.05 0.0 0.0 rpy=0 0 0 -> xyz=0.05 0.0 0.0 rpy=0 -1.57 0

File: myGym/envs/robots/universal_robots/urdf/ur3.urdf (robot description, URDF)
Before this commit: robot ur3, 13 links, 12 joints
Links:
- added link ee_x_axis; visual cylinder length=0.06 radius=0.002
- added link ee_y_axis; visual cylinder length=0.06 radius=0.002
- added link ee_z_axis; visual cylinder length=0.06 radius=0.002
- link endeffector: geometry visual sphere radius=0.005
Joints:
- added joint ee_x_axis_joint: type fixed, parent gripper, child ee_x_axis, origin xyz=0.05 0.0 0.0 rpy=0 1.57 0
- added joint ee_y_axis_joint: type fixed, parent gripper, child ee_y_axis, origin xyz=0.05 0.0 0.0 rpy=0 1.57 0
- added joint ee_z_axis_joint: type fixed, parent gripper, child ee_z_axis, origin xyz=0.05 0.0 0.0 rpy=0 1.57 0
- joint endeffector_joint: origin xyz=0.05 0.0 0.0 rpy=0 0 0 -> xyz=0.05 0.0 0.0 rpy=0 -1.57 0

File: myGym/envs/robots/universal_robots/urdf/ur5.urdf (robot description, URDF)
Before this commit: robot ur5, 13 links, 12 joints
Links:
- added link ee_x_axis; visual cylinder length=0.06 radius=0.002
- added link ee_y_axis; visual cylinder length=0.06 radius=0.002
- added link ee_z_axis; visual cylinder length=0.06 radius=0.002
- link endeffector: geometry visual sphere radius=0.005
Joints:
- added joint ee_x_axis_joint: type fixed, parent gripper, child ee_x_axis, origin xyz=0.05 0.0 0.0 rpy=0 1.57 0
- added joint ee_y_axis_joint: type fixed, parent gripper, child ee_y_axis, origin xyz=0.05 0.0 0.0 rpy=0 1.57 0
- added joint ee_z_axis_joint: type fixed, parent gripper, child ee_z_axis, origin xyz=0.05 0.0 0.0 rpy=0 1.57 0
- joint endeffector_joint: origin xyz=0.05 0.0 0.0 rpy=0 0 0 -> xyz=0.05 0.0 0.0 rpy=0 -1.57 0
