Commit message: unused robot urdf and meshes cleaned - unittest for unused files - robot repositioning bugfixes

File: myGym/envs/robots/abb/yumi/urdf/yumi.urdf (robot description, URDF)
Before this commit: robot yumi, 26 links, 25 joints
Joints:
- joint ee_x_axis_joint: origin xyz=0.0 0.0 0.12 rpy=3.14 0 0 -> xyz=0.0 0.0 0.12 rpy=0 0 0
- joint ee_y_axis_joint: origin xyz=0.0 0.0 0.12 rpy=3.14 0 0 -> xyz=0.0 0.0 0.12 rpy=0 0 0
- joint ee_z_axis_joint: origin xyz=0.0 0.0 0.12 rpy=3.14 0 0 -> xyz=0.0 0.0 0.12 rpy=0 0 0

File: myGym/envs/robots/pepper/pepper.urdf (robot description, URDF)
Before this commit: robot JulietteY20MP, 98 links, 97 joints
Links:
- removed link r_wrist
- added link ee_x_axis; visual cylinder length=0.06 radius=0.002
- added link ee_y_axis; visual cylinder length=0.06 radius=0.002
- added link ee_z_axis; visual cylinder length=0.06 radius=0.002
- added link lgrip, mass 2e-03
- link endeffector: mass 0.0000332 -> None; geometry visual sphere radius=0.005
- link gripper: mass 2e-03 -> 0.27555; geometry collision mesh filename=meshes/pepper/RWristYaw_vhacd.obj scale=1 1 1; visual mesh filename=meshes/pepper/RWristYaw.obj scale=1 1 1
Joints:
- added joint ee_x_axis_joint: type fixed, parent gripper, child ee_x_axis, origin xyz=0.07 0.0 -0.04 rpy=-3.14 0 1.57
- added joint ee_y_axis_joint: type fixed, parent gripper, child ee_y_axis, origin xyz=0.07 0.0 -0.04 rpy=-3.14 0 1.57
- added joint ee_z_axis_joint: type fixed, parent gripper, child ee_z_axis, origin xyz=0.07 0.0 -0.04 rpy=-3.14 0 1.57
- joint LGripper_joint: child gripper -> lgrip
- joint RFinger11_gjoint: limit lower=0.0 upper=0.872665 effort=0.144 velocity=12.56 -> lower=0.0 upper=1.57 effort=0.144 velocity=12.56; parent r_wrist -> gripper
- joint RFinger21_gjoint: limit lower=0.0 upper=0.872665 effort=0.144 velocity=12.56 -> lower=0.0 upper=1.57 effort=0.144 velocity=12.56; parent r_wrist -> gripper
- joint RFinger31_gjoint: limit lower=0.0 upper=0.872665 effort=0.144 velocity=12.56 -> lower=0.0 upper=1.57 effort=0.144 velocity=12.56; parent r_wrist -> gripper
- joint RFinger41_gjoint: limit lower=0.0 upper=0.872665 effort=0.144 velocity=12.56 -> lower=0.0 upper=1.57 effort=0.144 velocity=12.56; parent r_wrist -> gripper
- joint RHand/Touch/Back_sensor_fixedjoint: parent r_wrist -> gripper
- joint RThumb1: parent r_wrist -> gripper
- joint RWristYaw_rjoint: child r_wrist -> gripper
- joint endeffector_joint: parent r_wrist -> gripper
