Commit message: Add a human module

File: myGym/envs/robots/real_hands/humanoid_with_hands.urdf (robot description, URDF)
Before this commit: robot , 115 links, 114 joints
Links:
- removed link link0_15
- removed link link0_17
- removed link link0_19
- removed link link0_21
- removed link link0_32
- removed link link0_34
- removed link link0_36
- removed link link0_38
- removed link link0_40
- removed link link0_42
- removed link link0_44
- removed link link0_46
- removed link link0_48
- removed link link0_50
- removed link link0_52
- removed link r_index3
- removed link r_middle0
- removed link r_middle1
- removed link r_middle2
- removed link r_middle3
- removed link r_pinky0
- removed link r_pinky1
- removed link r_pinky2
- removed link r_pinky3
- removed link r_ring0
- removed link r_ring1
- removed link r_ring2
- removed link r_ring3
- removed link r_thumb0
- removed link r_thumb1
- removed link r_thumb2
- removed link r_thumb3
- added link direction_cone, mass 0.00000; visual mesh filename=mesh/cone.stl scale=0.002 0.002 0.01
- added link r_index3_endeffector, mass 0.00274; collision mesh filename=mesh/right/index3.stl scale=1.00000 1.00000 1.00000
Joints:
- removed joint jointfix_0_21
- removed joint jointfix_10_32
- removed joint jointfix_11_13
- removed joint jointfix_12_44
- removed joint jointfix_13_42
- removed joint jointfix_14_40
- removed joint jointfix_15_38
- removed joint jointfix_16_52
- removed joint jointfix_17_50
- removed joint jointfix_18_48
- removed joint jointfix_19_46
- removed joint jointfix_1_19
- removed joint jointfix_2_17
- removed joint jointfix_3_15
- removed joint jointfix_8_36
- removed joint jointfix_9_34
- removed joint r_middle_DIP
- removed joint r_middle_MCP
- removed joint r_middle_PIP
- removed joint r_pinky_ABD
- removed joint r_pinky_DIP
- removed joint r_pinky_MCP
- removed joint r_pinky_PIP
- removed joint r_ring_ABD
- removed joint r_ring_DIP
- removed joint r_ring_MCP
- removed joint r_ring_PIP
- removed joint r_thumb_ABD
- removed joint r_thumb_DIP
- removed joint r_thumb_MCP
- removed joint r_thumb_PIP
- added joint joint_direction_cone: type fixed, parent r_index3_endeffector, child direction_cone, origin xyz=0.00000 0.00000 0.00000 rpy=0.00000 -0.00000 0.00000, axis 0.00000 0.00000 0.00000
- joint jointfix_4_29: child r_index3 -> r_index3_endeffector
- joint r_index_ABD: type continuous -> fixed
- joint r_index_DIP: type continuous -> fixed
- joint r_index_MCP: type continuous -> fixed
- joint r_index_PIP: type continuous -> fixed
- joint r_wrist_PRO: type continuous -> fixed
- joint r_wrist_UDEV: type continuous -> fixed

Commit message: human urdf update

File: myGym/envs/robots/real_hands/humanoid_with_hands.urdf (robot description, URDF)
Before this commit: robot , 85 links, 84 joints
Links:
- removed link r_index3_endeffector
- added link ee_x_axis; visual cylinder length=0.06 radius=0.002
- added link ee_y_axis; visual cylinder length=0.06 radius=0.002
- added link ee_z_axis; visual cylinder length=0.06 radius=0.002
- added link endeffector; visual sphere radius=0.005
- added link gripper, mass 0.00274; collision mesh filename=mesh/right/index3.stl scale=1.00000 1.00000 1.00000
Joints:
- added joint ee_x_axis_joint: type fixed, parent gripper, child ee_x_axis, origin xyz=0.0 0.0 0.1 rpy=0 0 0
- added joint ee_y_axis_joint: type fixed, parent gripper, child ee_y_axis, origin xyz=0.0 0.0 0.1 rpy=0 0 0
- added joint ee_z_axis_joint: type fixed, parent gripper, child ee_z_axis, origin xyz=0.0 0.0 0.1 rpy=0 0 0
- added joint endeffector_joint: type fixed, parent gripper, child endeffector, origin xyz=0.0 0.0 0.1 rpy=0 3.14 0
- joint joint_direction_cone: parent r_index3_endeffector -> gripper
- joint jointfix_4_29: child r_index3_endeffector -> gripper
