Commit message: change urdf files to make robots work

File: myGym/envs/robots/gummi_arm/urdf/gummi.urdf (robot description, URDF)
Before this commit: robot gummi, 22 links, 21 joints
Links:
- removed link end_effector
- added link endeffector, mass 0.00478605585780196; collision mesh filename=package://gummi_arm/meshes/i2.stl; visual mesh filename=package://gummi_arm/meshes/i2.stl
Joints:
- joint i2f: child end_effector -> endeffector

File: myGym/envs/robots/pollen/reachy/urdf/leachy.urdf (robot description, URDF)
Before this commit: robot Leachy_w_hand, 10 links, 9 joints
Links:
- removed link end_effector
- added link endeffector, mass 0.009; collision mesh filename=package://reachy/meshes/open_bionics_hand_left-respondable.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; visual mesh filename=package://reachy/meshes/open_bionics_hand_left-visual.stl
Joints:
- joint l_wrist_pitch: child end_effector -> endeffector

File: myGym/envs/robots/pollen/reachy/urdf/reachy_and_leachy.urdf (robot description, URDF)
Before this commit: robot Leachy_w_hand, 17 links, 16 joints
Links:
- removed link end_effector
- added link endeffector, mass 0.090; collision mesh filename=package://reachy/meshes/ball-tip-respondable.stl; visual mesh filename=package://reachy/meshes/ball-tip-visual.stl
Joints:
- joint wrist_roll: child end_effector -> endeffector

Commit message: add _rjoint to urdf file joints to make gummi and leachy move

File: myGym/envs/robots/gummi_arm/urdf/gummi.urdf (robot description, URDF)
Before this commit: robot gummi, 22 links, 21 joints
Joints:
- removed joint elbow
- removed joint gripper
- removed joint i1f
- removed joint i2f
- removed joint i3f
- removed joint i4f
- removed joint i5f
- removed joint shoulder_pitch
- removed joint shoulder_roll
- removed joint shoulder_yaw
- removed joint upperarm_roll
- removed joint wrist_pitch
- added joint elbow_rjoint: type revolute, parent upperarm, child lowerarm_preroll_u, origin xyz=-0.006 0.0184 -0.23533 rpy=0 1 0, axis 0 -1 0, limit lower=-0.75 upper=0.35 effort=0 velocity=0
- added joint gripper_rjoint: type revolute, parent wrist, child gripper, origin xyz=0 0 0 rpy=0 0 0, axis 0 1 0, limit lower=0 upper=2 effort=0 velocity=0
- added joint i1f_rjoint: type revolute, parent wrist, child i1, origin xyz=0.059922 -0.031986 0.0029515 rpy=-0.79367 0.12795 -0.91441, axis 0 -1 0, limit lower=0 upper=0.8 effort=0 velocity=0, mimic joint=gripper
- added joint i2f_rjoint: type revolute, parent wrist, child endeffector, origin xyz=0.12886 -0.0060786 -0.0024749 rpy=-6.9389E-16 -8.4436E-17 -0.12109, axis 0 -1 0, limit lower=0 upper=0.8 effort=0 velocity=0, mimic joint=gripper
- added joint i3f_rjoint: type revolute, parent wrist, child i3, origin xyz=0.13223 0.0086295 -0.0025 rpy=-1.0408E-15 -5.7778E-30 -5.5511E-15, axis 0 -1 0, limit lower=0 upper=0.8 effort=0 velocity=0, mimic joint=gripper
- added joint i4f_rjoint: type revolute, parent wrist, child i4, origin xyz=0.13046 0.023543 -0.0025 rpy=-1.0408E-15 1.4051E-16 0.13418, axis 0 -1 0, limit lower=0 upper=0.8 effort=0 velocity=0, mimic joint=gripper
- added joint i5f_rjoint: type revolute, parent wrist, child i5, origin xyz=0.12703 0.037692 -0.0025 rpy=1.9429E-14 -3.8109E-15 0.19369, axis 0 -1 0, limit lower=0 upper=0.8 effort=0 velocity=0, mimic joint=gripper
- added joint shoulder_pitch_rjoint: type revolute, parent shoulder, child upperarm_preroll, origin xyz=-0.024 -0.17679 8.6827E-05 rpy=0.15 0 0, axis -1 0 0, limit lower=-0.15 upper=1.1 effort=0 velocity=0
- added joint shoulder_roll_rjoint: type revolute, parent shoulder_preroll, child shoulder, origin xyz=-2.6378E-05 0.057605 0.1302 rpy=0 -2 0, axis 0 -1 0, limit lower=-0.95 upper=2.3 effort=0 velocity=0
- added joint shoulder_yaw_rjoint: type revolute, parent base_link, child shoulder_preroll, origin xyz=-0.00027025 -0.10997 0.008 rpy=0 0 0, axis 0 0 1, limit lower=-0.75 upper=1 effort=0 velocity=0
- added joint upperarm_roll_rjoint: type revolute, parent upperarm_preroll, child upperarm, origin xyz=0.056992 -0.010088 -0.035587 rpy=0 0 0, axis 0 0 -1, limit lower=-1.56 upper=1.56 effort=0 velocity=0
- added joint wrist_pitch_rjoint: type revolute, parent lowerarm, child wrist, origin xyz=0.1511 -0.01935 0.0048471 rpy=0 0 0, axis 0 1 0, limit lower=-1 upper=1 effort=0 velocity=0

File: myGym/envs/robots/pollen/reachy/urdf/leachy.urdf (robot description, URDF)
Before this commit: robot Leachy_w_hand, 10 links, 9 joints
Joints:
- removed joint l_arm_yaw
- removed joint l_elbow_pitch
- removed joint l_forearm_yaw
- removed joint l_shoulder_pitch
- removed joint l_shoulder_roll
- removed joint l_wrist_pitch
- added joint l_arm_yaw_rjoint: type revolute, parent l_shoulder_to_arm, child l_upper_arm, origin xyz=0 0 0 rpy=0 0 0, axis 0 0 1, limit lower=-1.5708 upper=1.5708 effort=30 velocity=1
- added joint l_elbow_pitch_rjoint: type revolute, parent l_upper_arm, child l_forearm, origin xyz=0 0 -0.30745 rpy=0 0 0, axis 0 1 0, limit lower=-2.18166 upper=0 effort=30 velocity=1
- added joint l_forearm_yaw_rjoint: type revolute, parent l_forearm, child gripper, origin xyz=0 0 0 rpy=0 0 0, axis 0 0 1, limit lower=-2.61799 upper=2.61799 effort=30 velocity=1
- added joint l_shoulder_pitch_rjoint: type revolute, parent base, child l_shoulder, origin xyz=0 0.14 0 rpy=0 -1.5 0, axis 0 1 0, limit lower=-1.5708 upper=3.14159 effort=30 velocity=1
- added joint l_shoulder_roll_rjoint: type revolute, parent l_shoulder, child l_shoulder_to_arm, origin xyz=0 0 0 rpy=0 0 0, axis 1 0 0, limit lower=-0.174533 upper=3.14159 effort=30 velocity=1
- added joint l_wrist_pitch_rjoint: type revolute, parent gripper, child endeffector, origin xyz=0 0 -0.22415 rpy=0 0 0, axis 0 1 0, limit lower=-1.22173 upper=1.22173 effort=30 velocity=1

File: myGym/envs/robots/pollen/reachy/urdf/reachy_and_leachy.urdf (robot description, URDF)
Before this commit: robot Leachy_w_hand, 17 links, 16 joints
Joints:
- removed joint arm_yaw
- removed joint elbow_pitch
- removed joint forearm_yaw
- removed joint l_arm_yaw
- removed joint l_elbow_pitch
- removed joint l_forearm_yaw
- removed joint l_shoulder_pitch
- removed joint l_shoulder_roll
- removed joint l_wrist_pitch
- removed joint shoulder_pitch
- removed joint shoulder_roll
- removed joint wrist_pitch
- removed joint wrist_roll
- added joint arm_yaw_rjoint: type revolute, parent shoulder_to_arm, child upper_arm, origin xyz=0 0 0 rpy=0 0 0, axis 0 0 1, limit lower=-1.5708 upper=1.5708 effort=30 velocity=1
- added joint elbow_pitch_rjoint: type revolute, parent upper_arm, child forearm, origin xyz=0 0 -0.30745 rpy=0 0 0, axis 0 1 0, limit lower=-2.18166 upper=0 effort=30 velocity=1
- added joint forearm_yaw_rjoint: type revolute, parent forearm, child wrist, origin xyz=0 0 0 rpy=0 0 0, axis 0 0 1, limit lower=-2.61799 upper=2.61799 effort=30 velocity=1
- added joint l_arm_yaw_rjoint: type revolute, parent l_shoulder_to_arm, child l_upper_arm, origin xyz=0 0 0 rpy=0 0 0, axis 0 0 1, limit lower=-1.5708 upper=1.5708 effort=30 velocity=1
- added joint l_elbow_pitch_rjoint: type revolute, parent l_upper_arm, child l_forearm, origin xyz=0 0 -0.30745 rpy=0 0 0, axis 0 1 0, limit lower=-2.18166 upper=0 effort=30 velocity=1
- added joint l_forearm_yaw_rjoint: type revolute, parent l_forearm, child l_wrist, origin xyz=0 0 0 rpy=0 0 0, axis 0 0 1, limit lower=-2.61799 upper=2.61799 effort=30 velocity=1
- added joint l_shoulder_pitch_rjoint: type revolute, parent base, child l_shoulder, origin xyz=0 0.14 0 rpy=0 -1.5 0, axis 0 1 0, limit lower=-1.5708 upper=3.14159 effort=30 velocity=1
- added joint l_shoulder_roll_rjoint: type revolute, parent l_shoulder, child l_shoulder_to_arm, origin xyz=0 0 0 rpy=0 0 0, axis 1 0 0, limit lower=-0.174533 upper=3.14159 effort=30 velocity=1
- added joint l_wrist_pitch_rjoint: type revolute, parent l_wrist, child l_gripper, origin xyz=0 0 -0.22415 rpy=0 0 0, axis 0 1 0, limit lower=-1.22173 upper=1.22173 effort=30 velocity=1
- added joint shoulder_pitch_rjoint: type revolute, parent base, child shoulder, origin xyz=0 -0.14 0 rpy=0 -1.5 0, axis 0 1 0, limit lower=-1.5708 upper=3.14159 effort=30 velocity=1
- added joint shoulder_roll_rjoint: type revolute, parent shoulder, child shoulder_to_arm, origin xyz=0 0 0 rpy=0 0 0, axis 1 0 0, limit lower=-3.14159 upper=0.174533 effort=30 velocity=1
- added joint wrist_pitch_rjoint: type revolute, parent wrist, child gripper, origin xyz=0 0 -0.22425 rpy=0 0 0, axis 0 1 0, limit lower=-1.22173 upper=1.22173 effort=30 velocity=1
- added joint wrist_roll_rjoint: type revolute, parent gripper, child endeffector, origin xyz=0 0 -0.03243 rpy=0 0 0, axis 1 0 0, limit lower=-1.0472 upper=1.0472 effort=30 velocity=1

Commit message: robot endeffctor update and repositioning

File: myGym/envs/robots/gummi_arm/urdf/gummi.urdf (robot description, URDF)
Before this commit: robot gummi, 22 links, 21 joints
Links:
- removed link wrist
- added link ee_x_axis; visual cylinder length=0.06 radius=0.002
- added link ee_y_axis; visual cylinder length=0.06 radius=0.002
- added link ee_z_axis; visual cylinder length=0.06 radius=0.002
- added link i2, mass 0.00478605585780196; collision mesh filename=package://gummi_arm/meshes/i2.stl; visual mesh filename=package://gummi_arm/meshes/i2.stl
- link endeffector: mass 0.00478605585780196 -> None; geometry visual sphere radius=0.005
- link gripper: mass 0.001 -> 0.0644774651698934; geometry collision mesh filename=package://gummi_arm/meshes/wrist.stl; visual mesh filename=package://gummi_arm/meshes/wrist.stl
Joints:
- removed joint gripper_rjoint
- added joint ee_x_axis_joint: type fixed, parent gripper, child ee_x_axis, origin xyz=0.1 -0.0 0.03 rpy=0 0 -1.57
- added joint ee_y_axis_joint: type fixed, parent gripper, child ee_y_axis, origin xyz=0.1 -0.0 0.03 rpy=0 0 -1.57
- added joint ee_z_axis_joint: type fixed, parent gripper, child ee_z_axis, origin xyz=0.1 -0.0 0.03 rpy=0 0 -1.57
- added joint endeffector_joint: type fixed, parent gripper, child endeffector, origin xyz=0.1 -0.0 0.03 rpy=-3.14 0 0
- joint forearm_roll: limit effort=0 velocity=1 -> lower=-3.14 upper=3.14 effort=0 velocity=1; type continuous -> revolute
- joint i1f_rjoint: parent wrist -> gripper
- joint i2f_rjoint: child endeffector -> i2; parent wrist -> gripper
- joint i3f_rjoint: parent wrist -> gripper
- joint i4f_rjoint: parent wrist -> gripper
- joint i5f_rjoint: parent wrist -> gripper
- joint wrist_pitch_rjoint: child wrist -> gripper

File: myGym/envs/robots/jaco_arm/jaco/urdf/jaco_robotiq_fixed.urdf (robot description, URDF)
Before this commit: robot j2s7s300, 20 links, 19 joints
Links:
- added link ee_x_axis; visual cylinder length=0.06 radius=0.002
- added link ee_y_axis; visual cylinder length=0.06 radius=0.002
- added link ee_z_axis; visual cylinder length=0.06 radius=0.002
- link endeffector: mass 0.0000332 -> None; geometry visual sphere radius=0.005
Joints:
- added joint ee_x_axis_joint: type fixed, parent gripper, child ee_x_axis, origin xyz=0.0 0.0 -0.23 rpy=0 3.14 1.57
- added joint ee_y_axis_joint: type fixed, parent gripper, child ee_y_axis, origin xyz=0.0 0.0 -0.23 rpy=0 3.14 1.57
- added joint ee_z_axis_joint: type fixed, parent gripper, child ee_z_axis, origin xyz=0.0 0.0 -0.23 rpy=0 3.14 1.57

File: myGym/envs/robots/pollen/reachy/urdf/reachy.urdf (robot description, URDF)
Before this commit: robot Reachy, 12 links, 11 joints
Links:
- added link ee_x_axis; visual cylinder length=0.06 radius=0.002
- added link ee_y_axis; visual cylinder length=0.06 radius=0.002
- added link ee_z_axis; visual cylinder length=0.06 radius=0.002
- link endeffector: mass 0.0000332 -> None; geometry visual sphere radius=0.005
Joints:
- added joint ee_x_axis_joint: type fixed, parent gripper, child ee_x_axis, origin xyz=0.0 -0.0 -0.12 rpy=3.14 0 0
- added joint ee_y_axis_joint: type fixed, parent gripper, child ee_y_axis, origin xyz=0.0 -0.0 -0.12 rpy=3.14 0 0
- added joint ee_z_axis_joint: type fixed, parent gripper, child ee_z_axis, origin xyz=0.0 -0.0 -0.12 rpy=3.14 0 0

Commit message: robot updates - gripper open and close position added

File: myGym/envs/robots/gummi_arm/urdf/gummi.urdf (robot description, URDF)
Before this commit: robot gummi, 25 links, 24 joints
Joints:
- removed joint i1f_rjoint
- removed joint i2f_rjoint
- removed joint i3f_rjoint
- removed joint i4f_rjoint
- removed joint i5f_rjoint
- added joint i1f_gjoint: type revolute, parent gripper, child i1, origin xyz=0.059922 -0.031986 0.0029515 rpy=-0.79367 0.12795 -0.91441, axis 0 -1 0, limit lower=0 upper=0.8 effort=0 velocity=0, mimic joint=gripper
- added joint i2f_gjoint: type revolute, parent gripper, child i2, origin xyz=0.12886 -0.0060786 -0.0024749 rpy=-6.9389E-16 -8.4436E-17 -0.12109, axis 0 -1 0, limit lower=0 upper=0.8 effort=0 velocity=0, mimic joint=gripper
- added joint i3f_gjoint: type revolute, parent gripper, child i3, origin xyz=0.13223 0.0086295 -0.0025 rpy=-1.0408E-15 -5.7778E-30 -5.5511E-15, axis 0 -1 0, limit lower=0 upper=0.8 effort=0 velocity=0, mimic joint=gripper
- added joint i4f_gjoint: type revolute, parent gripper, child i4, origin xyz=0.13046 0.023543 -0.0025 rpy=-1.0408E-15 1.4051E-16 0.13418, axis 0 -1 0, limit lower=0 upper=0.8 effort=0 velocity=0, mimic joint=gripper
- added joint i5f_gjoint: type revolute, parent gripper, child i5, origin xyz=0.12703 0.037692 -0.0025 rpy=1.9429E-14 -3.8109E-15 0.19369, axis 0 -1 0, limit lower=0 upper=0.8 effort=0 velocity=0, mimic joint=gripper

File: myGym/envs/robots/jaco_arm/jaco/urdf/jaco_robotiq_fixed.urdf (robot description, URDF)
Before this commit: robot j2s7s300, 23 links, 22 joints
Joints:
- removed joint robotiq_85_left_finger_gjoint
- removed joint robotiq_85_left_finger_tip_joint
- removed joint robotiq_85_right_finger_gjoint
- removed joint robotiq_85_right_finger_tip_joint
- added joint robotiq_85_left_finger_joint: type fixed, parent robotiq_85_left_knuckle_link, child robotiq_85_left_finger_link, origin xyz=-0.00408552455 -0.03148604435 0.0 rpy=0 0 0, limit lower=-3.14 upper=3.14 velocity=1.0
- added joint robotiq_85_left_finger_tip_gjoint: type revolute, parent robotiq_85_left_inner_knuckle_link, child robotiq_85_left_finger_tip_link, origin xyz=0.04303959807 -0.03759940821 0.0 rpy=0.0 0.0 0.0, axis 0 0 1, limit lower=-0.8757 upper=0.0 velocity=1.0
- added joint robotiq_85_right_finger_joint: type fixed, parent robotiq_85_right_knuckle_link, child robotiq_85_right_finger_link, origin xyz=-0.00408552455 -0.03148604435 0.0 rpy=0 0 0, limit lower=-3.14 upper=3.14 velocity=1.0
- added joint robotiq_85_right_finger_tip_gjoint: type revolute, parent robotiq_85_right_inner_knuckle_link, child robotiq_85_right_finger_tip_link, origin xyz=0.04303959807 -0.03759940821  0.0 rpy=0.0 0.0 0.0, axis 0 0 1, limit lower=-0.8757 upper=0.0 velocity=1.0

File: myGym/envs/robots/nico/nico_grasper.urdf (robot description, URDF)
Before this commit: robot nico_upper_rh6d, 32 links, 31 joints
Joints:
- joint r_thumb_z_gjoint: type fixed -> revolute

Commit message: gripper status working - tested

File: myGym/envs/robots/gummi_arm/urdf/gummi.urdf (robot description, URDF)
Before this commit: robot gummi, 25 links, 24 joints
Joints:
- removed joint forearm_roll
- added joint forearm_roll_rjoint: type revolute, parent lowerarm_preroll_d, child lowerarm, origin xyz=0.043506 -0.00023376 -0.019876 rpy=0 0 0, axis -1 0 0, limit lower=-3.14 upper=3.14 effort=0 velocity=1
