Commit message: Fix MuJoCo integration issues: inertia, fixed joints, mesh paths, ground plane, reward obs
Agent-Logs-Url: https://github.com/incognite-lab/myGym/sessions/e4c77b20-63e1-46f8-85a6-a39b352de51b

Co-authored-by: michalvavrecka <16919032+michalvavrecka@users.noreply.github.com>

File: myGym/envs/rooms/collision/table_complex.urdf (robot description, URDF)
Before this commit: robot table_universal, 1 links, 0 joints
Links:
- link table_universal: geometry collision box size=0.01 0.2 0.1; collision box size=0.02 0.39 .77
