Commit message: walker urdf update - -working

File: myGym/envs/robots/ubtech/tiangong2pro_urdf/urdf/tiangong2.0_pro_with_hands.urdf (robot description, URDF)
Before this commit: robot tiangong2pro_urdf_with_hands, 63 links, 62 joints
Links:
- added link ee_x_axis, mass 0.0001; visual cylinder length=0.06 radius=0.002
- added link ee_y_axis, mass 0.0001; visual cylinder length=0.06 radius=0.002
- added link ee_z_axis, mass 0.0001; visual cylinder length=0.06 radius=0.002
- added link endeffector, mass 0.0001; visual sphere radius=0.005
- added link gripper, mass 0.0001; visual sphere radius=0.005
Joints:
- removed joint body_yaw_joint
- removed joint elbow_pitch_r_joint
- removed joint elbow_yaw_r_joint
- removed joint right_index_1_joint
- removed joint right_little_1_joint
- removed joint right_middle_1_joint
- removed joint right_ring_1_joint
- removed joint right_thumb_1_joint
- removed joint shoulder_pitch_r_joint
- removed joint shoulder_roll_r_joint
- removed joint shoulder_yaw_r_joint
- removed joint wrist_pitch_r_joint
- removed joint wrist_roll_r_joint
- added joint body_yaw_rjoint: type revolute, parent pelvis, child waist_yaw_link, origin xyz=0 0 0 rpy=0 0 0, axis 0 0 1, limit lower=-2.9670597283903604 upper=3.141592653589793 effort=91.0 velocity=9.215338450530059
- added joint ee_x_axis_joint: type fixed, parent gripper, child ee_x_axis, origin xyz=0.03 0.0 0.10 rpy=0 0 1.57
- added joint ee_y_axis_joint: type fixed, parent gripper, child ee_y_axis, origin xyz=0.03 0.0 0.10 rpy=1.57 0 0
- added joint ee_z_axis_joint: type fixed, parent gripper, child ee_z_axis, origin xyz=0.03 0.0 0.10 rpy=0 1.57 0
- added joint elbow_pitch_r_rjoint: type revolute, parent shoulder_yaw_r_link, child elbow_pitch_r_link, origin xyz=0.02 0 -0.1975 rpy=0 0 0, axis 0 1 0, limit lower=-2.6179938779914944 upper=0.2617993877991494 effort=35.0 velocity=5.235987755982989
- added joint elbow_yaw_r_rjoint: type revolute, parent elbow_pitch_r_link, child elbow_yaw_r_link, origin xyz=-0.02 0 -0.0543 rpy=0 0 0, axis 0 0 1, limit lower=-2.9670597283903604 upper=2.9670597283903604 effort=24.0 velocity=10.471975511965978
- added joint endeffector_joint: type fixed, parent gripper, child endeffector, origin xyz=0.03 0.0 0.10 rpy=0 -1.57 0
- added joint gripper_joint: type fixed, parent R_base_link, child gripper, origin xyz=-0.00 -0.00 0.0 rpy=0 0 0
- added joint right_index_1_gjoint: type revolute, parent R_base_link, child right_index_1, origin xyz=-0.000285 0.020275 0.136946 rpy=1.5359 0 0, axis 0 -0.069756  -0.997564, limit lower=0 upper=1.333 effort=50 velocity=1
- added joint right_little_1_gjoint: type revolute, parent R_base_link, child right_little_1, origin xyz=-0.000285 -0.037422 0.13446 rpy=1.6755 0 0, axis 0 0 -1, limit lower=0 upper=1.333 effort=50 velocity=1
- added joint right_middle_1_gjoint: type revolute, parent R_base_link, child right_middle_1, origin xyz=-0.000285 0.00295 0.1371 rpy=1.5708 0 0, axis 0 0 -1, limit lower=0 upper=1.333 effort=50 velocity=1
- added joint right_ring_1_gjoint: type revolute, parent R_base_link, child right_ring_1, origin xyz=-0.000285 -0.018271 0.136282 rpy=1.6232 0 0, axis 0 0 -1, limit lower=0 upper=1.333 effort=50 velocity=1
- added joint right_thumb_1_gjoint: type revolute, parent R_base_link, child right_thumb_1, origin xyz=0.01696 0.02045 0.06635 rpy=0 0 0, axis 0 0 -1, limit lower=0 upper=1.246165 effort=50 velocity=1
- added joint shoulder_pitch_r_rjoint: type revolute, parent waist_yaw_link, child shoulder_pitch_r_link, origin xyz=0 -0.1444 0.37712 rpy=-0.087266 0 0, axis 0 1 0, limit lower=-2.9670597283903604 upper=2.9670597283903604 effort=91.0 velocity=9.215338450530059
- added joint shoulder_roll_r_rjoint: type revolute, parent shoulder_pitch_r_link, child shoulder_roll_r_link, origin xyz=0 -0.068 0 rpy=0 0 0, axis 1 0 0, limit lower=-2.6179938779914944 upper=0.2617993877991494 effort=95.0 velocity=3.979350694547071
- added joint shoulder_yaw_r_rjoint: type revolute, parent shoulder_roll_r_link, child shoulder_yaw_r_link, origin xyz=0 0 -0.1025 rpy=0 0 0, axis 0 0 1, limit lower=-2.9670597283903604 upper=2.9670597283903604 effort=35.0 velocity=5.235987755982989
- added joint wrist_pitch_r_rjoint: type revolute, parent elbow_yaw_r_link, child wrist_pitch_r_link, origin xyz=0 0 -0.1887 rpy=0 0 0, axis 0 1 0, limit lower=-0.7853981633974483 upper=1.0471975511965976 effort=6.3 velocity=7.5398223686155035
- added joint wrist_roll_r_rjoint: type revolute, parent wrist_pitch_r_link, child wrist_roll_r_link, origin xyz=0 0 -0.02 rpy=0 0 0, axis 1 0 0, limit lower=-1.3089969389957472 upper=1.6580627893946132 effort=6.3 velocity=7.5398223686155035
