Commit message: icub and walker update

File: myGym/envs/robots/iCub/icub.urdf (robot description, URDF)
Before this commit: robot iCub, 59 links, 58 joints
Joints:
- joint endeffector_joint: origin xyz=-0.07 -0.03 0.0 rpy=-1.57 -1.57 -1.57 -> xyz=-0.07 -0.03 0.0 rpy=1.57 0 3.14

File: myGym/envs/robots/iCub/icubfull.urdf (robot description, URDF)
Before this commit: robot iCub, 103 links, 102 joints
Links:
- removed link r_hand_dh_frame
- added link ee_x_axis, mass 0.0001; visual cylinder length=0.06 radius=0.002
- added link ee_y_axis, mass 0.0001; visual cylinder length=0.06 radius=0.002
- added link ee_z_axis, mass 0.0001; visual cylinder length=0.06 radius=0.002
- added link endeffector, mass 0.0001; visual sphere radius=0.005
- added link gripper, mass 0
Joints:
- removed joint r_elbow
- removed joint r_hand_index_0_joint
- removed joint r_hand_little_0_joint
- removed joint r_hand_middle_0_joint
- removed joint r_hand_ring_0_joint
- removed joint r_hand_thumb_0_joint
- removed joint r_shoulder_pitch
- removed joint r_shoulder_roll
- removed joint r_shoulder_yaw
- removed joint r_wrist_pitch
- removed joint r_wrist_prosup
- removed joint r_wrist_yaw
- added joint ee_x_axis_joint: type fixed, parent gripper, child ee_x_axis, origin xyz=-0.07 -0.03 0.0 rpy=-1.57 -1.57 0
- added joint ee_y_axis_joint: type fixed, parent gripper, child ee_y_axis, origin xyz=-0.07 -0.03 0.0 rpy=1.57 -1.57 0
- added joint ee_z_axis_joint: type fixed, parent gripper, child ee_z_axis, origin xyz=-0.07 -0.03 0.0 rpy=1.57 -1.57 0
- added joint endeffector_joint: type fixed, parent gripper, child endeffector, origin xyz=-0.07 -0.03 0.0 rpy=1.57 0 3.14
- added joint r_elbow_rjoint: type revolute, parent r_upper_arm, child r_elbow_1, origin xyz=0 -0.0224999 0.07926 rpy=0 1.30899700697 0, axis 2.22044604925e-16 1.0 0.0, limit lower=0.261799387799 upper=1.85004900711 effort=50000 velocity=50000
- added joint r_hand_index_0_gjoint: type revolute, parent r_hand, child r_hand_index_0, origin xyz=-0.0525584344285222 0.00514320000012944 0.039473341148855 rpy=1.48159614751736 -2.80851293007006 0.00659385709493776, axis 0.0 0.0 1.0, limit lower=-0.3490658503988659 upper=0.0 effort=50000 velocity=50000
- added joint r_hand_little_0_gjoint: type revolute, parent r_hand, child r_hand_little_0, origin xyz=-0.0636290045193172 0.00444319999987861 -0.0101109273025847 rpy=-1.54796540941373 -0.154343069643928 3.05377499029501, axis 0.0 0.0 1.0, limit lower=0.0 upper=0.3490658503988659 effort=50000 velocity=50000
- added joint r_hand_middle_0_gjoint: type revolute, parent r_hand, child r_hand_middle_0, origin xyz=-0.057540451023329 0.00604320000004786 0.0237779752515841 rpy=1.57079632679979 -2.87979333376279 2.06501482580279e-13, axis 0.0 0.0 1.0, limit lower=0.0 upper=0.3490658503988659 effort=50000 velocity=50000
- added joint r_hand_ring_0_gjoint: type revolute, parent r_hand, child r_hand_ring_0, origin xyz=-0.0606910842022157 0.00544319999997171 0.00865822622681494 rpy=-1.54796540941373 -0.154343069643928 3.05377499029501, axis 0.0 0.0 1.0, limit lower=0.0 upper=0.3490658503988659 effort=50000 velocity=50000
- added joint r_hand_thumb_0_gjoint: type revolute, parent r_hand, child r_hand_thumb_0, origin xyz=-0.0318492127582281 -0.00405679999993591 0.0192026964178796 rpy=0.0880846384483103 -1.32396952212432 2.97584384270403, axis 0.0 0.0 1.0, limit lower=0.0 upper=1.5707963267948966 effort=50000 velocity=50000
- added joint r_shoulder_pitch_rjoint: type revolute, parent chest, child r_shoulder_1, origin xyz=-0.120015999809 0.0928 0.0079693 rpy=0 -0.523598883792 3.14159265359, axis -0.9659257753743923 0.0 0.25881923511860305, limit lower=-1.66678943565 upper=0.174532925199 effort=50000 velocity=50000
- added joint r_shoulder_roll_rjoint: type revolute, parent r_shoulder_1, child r_shoulder_2, origin xyz=-0.00758046573227 0 0.0142102463639 rpy=-0.270597611583 -0.252680154648 -1.50155680035, axis -0.2588189595935754 0 -0.9659258492011169, limit lower=0.0 upper=2.80648943721 effort=50000 velocity=50000
- added joint r_shoulder_yaw_rjoint: type revolute, parent r_shoulder_2, child r_shoulder_3, origin xyz=-0.0253460713232 2.32750427306e-07 -0.00538764806457 rpy=-0.252689546175 0.0085186183214 0.067039889142, axis 0.9659258492011169 0 -0.2588189595935754, limit lower=-0.645771823238 upper=1.3962634016 effort=50000 velocity=50000
- added joint r_wrist_pitch_rjoint: type revolute, parent r_forearm, child r_wrist_1, origin xyz=-0.103505208873 7.00000000002e-06 0.0251977029936 rpy=0 0 0, axis 0.25881895959357540 0 0.9659258492011169, limit lower=-1.3962634016 upper=0.436332312999 effort=50000 velocity=50000
- added joint r_wrist_prosup_rjoint: type revolute, parent r_elbow_1, child r_forearm, origin xyz=-0.0384624299027 0.0224999 -0.00522316819403 rpy=0 0 0, axis 0.9659258492011169 0 -0.2588189595935754, limit lower=-1.0471975512 upper=1.0471975512 effort=50000 velocity=50000
- added joint r_wrist_yaw_rjoint: type revolute, parent r_wrist_1, child r_hand, origin xyz=0.000634106499644 -0.0194999 0.00236651831751 rpy=0 0 0, axis 2.22044604925e-16 -1.0 0.0, limit lower=-0.349065850399 upper=0.436332312999 effort=50000 velocity=50000
- joint eyes_tilt: type revolute -> fixed
- joint l_ankle_pitch: type revolute -> fixed
- joint l_ankle_roll: type revolute -> fixed
- joint l_elbow: type revolute -> fixed
- joint l_eye_pan_joint: type revolute -> fixed
- joint l_hand_index_0_joint: type revolute -> fixed
- joint l_hand_index_1_joint: type revolute -> fixed
- joint l_hand_index_2_joint: type revolute -> fixed
- joint l_hand_index_3_joint: type revolute -> fixed
- joint l_hand_little_0_joint: type revolute -> fixed
- joint l_hand_little_1_joint: type revolute -> fixed
- joint l_hand_little_2_joint: type revolute -> fixed
- joint l_hand_little_3_joint: type revolute -> fixed
- joint l_hand_middle_0_joint: type revolute -> fixed
- joint l_hand_middle_1_joint: type revolute -> fixed
- joint l_hand_middle_2_joint: type revolute -> fixed
- joint l_hand_middle_3_joint: type revolute -> fixed
- joint l_hand_ring_0_joint: type revolute -> fixed
- joint l_hand_ring_1_joint: type revolute -> fixed
- joint l_hand_ring_2_joint: type revolute -> fixed
- joint l_hand_ring_3_joint: type revolute -> fixed
- joint l_hand_thumb_0_joint: type revolute -> fixed
- joint l_hand_thumb_1_joint: type revolute -> fixed
- joint l_hand_thumb_2_joint: type revolute -> fixed
- joint l_hand_thumb_3_joint: type revolute -> fixed
- joint l_hip_pitch: type revolute -> fixed
- joint l_hip_roll: type revolute -> fixed
- joint l_hip_yaw: type revolute -> fixed
- joint l_knee: type revolute -> fixed
- joint l_shoulder_pitch: type revolute -> fixed
- joint l_shoulder_roll: type revolute -> fixed
- joint l_shoulder_yaw: type revolute -> fixed
- joint l_wrist_pitch: type revolute -> fixed
- joint l_wrist_prosup: type revolute -> fixed
- joint l_wrist_yaw: type revolute -> fixed
- joint neck_pitch: type revolute -> fixed
- joint neck_roll: type revolute -> fixed
- joint neck_yaw: type revolute -> fixed
- joint r_ankle_pitch: type revolute -> fixed
- joint r_ankle_roll: type revolute -> fixed
- joint r_eye_pan_joint: type revolute -> fixed
- joint r_hand_dh_frame_fixed_joint: child r_hand_dh_frame -> gripper
- joint r_hand_index_1_joint: type revolute -> fixed
- joint r_hand_index_2_joint: type revolute -> fixed
- joint r_hand_index_3_joint: type revolute -> fixed
- joint r_hand_little_1_joint: type revolute -> fixed
- joint r_hand_little_2_joint: type revolute -> fixed
- joint r_hand_little_3_joint: type revolute -> fixed
- joint r_hand_middle_1_joint: type revolute -> fixed
- joint r_hand_middle_2_joint: type revolute -> fixed
- joint r_hand_middle_3_joint: type revolute -> fixed
- joint r_hand_ring_1_joint: type revolute -> fixed
- joint r_hand_ring_2_joint: type revolute -> fixed
- joint r_hand_ring_3_joint: type revolute -> fixed
- joint r_hand_thumb_1_joint: type revolute -> fixed
- joint r_hand_thumb_2_joint: type revolute -> fixed
- joint r_hand_thumb_3_joint: type revolute -> fixed
- joint r_hip_pitch: type revolute -> fixed
- joint r_hip_roll: type revolute -> fixed
- joint r_hip_yaw: type revolute -> fixed
- joint r_knee: type revolute -> fixed
- joint torso_pitch: type revolute -> fixed
- joint torso_roll: type revolute -> fixed
- joint torso_yaw: type revolute -> fixed

File: myGym/envs/robots/ubtech/tiangong2pro_urdf/urdf/tiangong2.0_pro_with_hands.urdf (robot description, URDF)
Before this commit: robot tiangong2pro_urdf_with_hands, 68 links, 67 joints
Joints:
- joint ankle_pitch_l_joint: type revolute -> fixed
- joint ankle_pitch_r_joint: type revolute -> fixed
- joint ankle_roll_l_joint: type revolute -> fixed
- joint ankle_roll_r_joint: type revolute -> fixed
- joint elbow_pitch_l_joint: type revolute -> fixed
- joint elbow_yaw_l_joint: type revolute -> fixed
- joint head_pitch_joint: type revolute -> fixed
- joint head_roll_joint: type revolute -> fixed
- joint head_yaw_joint: type revolute -> fixed
- joint hip_pitch_l_joint: type revolute -> fixed
- joint hip_pitch_r_joint: type revolute -> fixed
- joint hip_roll_l_joint: type revolute -> fixed
- joint hip_roll_r_joint: type revolute -> fixed
- joint hip_yaw_l_joint: type revolute -> fixed
- joint hip_yaw_r_joint: type revolute -> fixed
- joint knee_pitch_l_joint: type revolute -> fixed
- joint knee_pitch_r_joint: type revolute -> fixed
- joint left_index_1_joint: type revolute -> fixed
- joint left_index_2_joint: type revolute -> fixed
- joint left_little_1_joint: type revolute -> fixed
- joint left_little_2_joint: type revolute -> fixed
- joint left_middle_1_joint: type revolute -> fixed
- joint left_middle_2_joint: type revolute -> fixed
- joint left_ring_1_joint: type revolute -> fixed
- joint left_ring_2_joint: type revolute -> fixed
- joint left_thumb_1_joint: type revolute -> fixed
- joint left_thumb_2_joint: type revolute -> fixed
- joint left_thumb_3_joint: type revolute -> fixed
- joint left_thumb_4_joint: type revolute -> fixed
- joint right_index_2_joint: type revolute -> fixed
- joint right_little_2_joint: type revolute -> fixed
- joint right_middle_2_joint: type revolute -> fixed
- joint right_ring_2_joint: type revolute -> fixed
- joint right_thumb_2_joint: type revolute -> fixed
- joint right_thumb_3_joint: type revolute -> fixed
- joint right_thumb_4_joint: type revolute -> fixed
- joint shoulder_pitch_l_joint: type revolute -> fixed
- joint shoulder_roll_l_joint: type revolute -> fixed
- joint shoulder_yaw_l_joint: type revolute -> fixed
- joint wrist_pitch_l_joint: type revolute -> fixed
- joint wrist_roll_l_joint: type revolute -> fixed

Commit message: icub update

File: myGym/envs/robots/iCub/icub.urdf (robot description, URDF)
Before this commit: robot iCub, 59 links, 58 joints
Links:
- link gripper: geometry visual mesh filename=package://iCub/meshes/visual/sim_sea_2-5_r_hand_prt-binary.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 scale=0.001 0.001 0.001
