Commit message: walker urdf

File: myGym/envs/robots/S2_/S2.urdf (robot description, URDF)
Before this commit: robot S2, 63 links, 62 joints
Links:
- added link ee_x_axis; visual cylinder length=0.06 radius=0.002
- added link ee_y_axis; visual cylinder length=0.06 radius=0.002
- added link ee_z_axis; visual cylinder length=0.06 radius=0.002
- added link endeffector; visual sphere radius=0.005
- added link gripper, mass 0.15210234; collision mesh filename=package://walkerS2/meshes/R_base_link.STL; visual mesh filename=package://walkerS2/meshes/R_base_link.STL
Joints:
- added joint R_base_gripper_fix: type fixed, parent R_base_link, child gripper, origin xyz=0 0 0 rpy=0 0 0
- added joint ee_x_axis_joint: type fixed, parent gripper, child ee_x_axis, origin xyz=0.05 0.0 0.1 rpy=-1.57 -1.57 0
- added joint ee_y_axis_joint: type fixed, parent gripper, child ee_y_axis, origin xyz=0.05 0.0 0.1 rpy=-1.57 -1.57 0
- added joint ee_z_axis_joint: type fixed, parent gripper, child ee_z_axis, origin xyz=0.05 0.0 0.1 rpy=-1.57 -1.57 0
- added joint endeffector_joint: type fixed, parent gripper, child endeffector, origin xyz=0.05 0.0 0.1 rpy=1.57 0 0

Commit message: walker working

File: myGym/envs/robots/S2_/S2.urdf (robot description, URDF)
Before this commit: robot S2, 68 links, 67 joints
Links:
- link gripper: geometry collision mesh filename=package://S2_/meshes/R_base_link.STL; visual mesh filename=package://S2_/meshes/R_base_link.STL
