Commit message: S2 update

File: myGym/envs/robots/ubtech/S2.urdf (robot description, URDF)
Before this commit: robot S2, 68 links, 67 joints
Joints:
- joint ankle_pitch_l_joint: type revolute -> fixed
- joint ankle_pitch_r_joint: type revolute -> fixed
- joint ankle_roll_l_joint: type revolute -> fixed
- joint ankle_roll_r_joint: type revolute -> fixed
- joint elbow_pitch_l_joint: type revolute -> fixed
- joint elbow_yaw_l_joint: type revolute -> fixed
- joint head_pitch_joint: type revolute -> fixed
- joint head_roll_joint: type revolute -> fixed
- joint head_yaw_joint: type revolute -> fixed
- joint hip_pitch_l_joint: type revolute -> fixed
- joint hip_pitch_r_joint: type revolute -> fixed
- joint hip_roll_l_joint: type revolute -> fixed
- joint hip_roll_r_joint: type revolute -> fixed
- joint hip_yaw_l_joint: type revolute -> fixed
- joint hip_yaw_r_joint: type revolute -> fixed
- joint knee_pitch_l_joint: type revolute -> fixed
- joint knee_pitch_r_joint: type revolute -> fixed
- joint left_index_1_joint: type revolute -> fixed
- joint left_index_2_joint: type revolute -> fixed
- joint left_little_1_joint: type revolute -> fixed
- joint left_little_2_joint: type revolute -> fixed
- joint left_middle_1_joint: type revolute -> fixed
- joint left_middle_2_joint: type revolute -> fixed
- joint left_ring_1_joint: type revolute -> fixed
- joint left_ring_2_joint: type revolute -> fixed
- joint left_thumb_1_joint: type revolute -> fixed
- joint left_thumb_2_joint: type revolute -> fixed
- joint left_thumb_3_joint: type revolute -> fixed
- joint left_thumb_4_joint: type revolute -> fixed
- joint right_index_2_joint: type revolute -> fixed
- joint right_little_2_joint: type revolute -> fixed
- joint right_middle_2_joint: type revolute -> fixed
- joint right_ring_2_joint: type revolute -> fixed
- joint right_thumb_2_joint: type revolute -> fixed
- joint right_thumb_3_joint: type revolute -> fixed
- joint right_thumb_4_joint: type revolute -> fixed
- joint shoulder_pitch_l_joint: type revolute -> fixed
- joint shoulder_roll_l_joint: type revolute -> fixed
- joint shoulder_yaw_l_joint: type revolute -> fixed
- joint wrist_pitch_l_joint: type revolute -> fixed
- joint wrist_roll_l_joint: type revolute -> fixed
