Commit message: disabled finger collisions for S2, endeffector pos fixed

File: myGym/envs/robots/ubtech/S2.urdf (robot description, URDF)
Before this commit: robot S2, 68 links, 67 joints
Links:
- link left_index_1: geometry visual mesh filename=package://ubtech/meshes/left_index_1.STL
- link left_index_2: geometry visual mesh filename=package://ubtech/meshes/left_index_2.STL
- link left_little_1: geometry visual mesh filename=package://ubtech/meshes/left_little_1.STL
- link left_little_2: geometry visual mesh filename=package://ubtech/meshes/left_little_2.STL
- link left_middle_1: geometry visual mesh filename=package://ubtech/meshes/left_middle_1.STL
- link left_middle_2: geometry visual mesh filename=package://ubtech/meshes/left_middle_2.STL
- link left_ring_1: geometry visual mesh filename=package://ubtech/meshes/left_ring_1.STL
- link left_ring_2: geometry visual mesh filename=package://ubtech/meshes/left_ring_2.STL
- link left_thumb_1: geometry visual mesh filename=package://ubtech/meshes/left_thumb_1.STL
- link left_thumb_2: geometry visual mesh filename=package://ubtech/meshes/left_thumb_2.STL
- link left_thumb_3: geometry visual mesh filename=package://ubtech/meshes/left_thumb_3.STL
- link left_thumb_4: geometry visual mesh filename=package://ubtech/meshes/left_thumb_4.STL
- link right_index_1: geometry visual mesh filename=package://ubtech/meshes/right_index_1.STL
- link right_index_2: geometry visual mesh filename=package://ubtech/meshes/right_index_2.STL
- link right_little_1: geometry visual mesh filename=package://ubtech/meshes/right_little_1.STL
- link right_little_2: geometry visual mesh filename=package://ubtech/meshes/right_little_2.STL
- link right_middle_1: geometry visual mesh filename=package://ubtech/meshes/right_middle_1.STL
- link right_middle_2: geometry visual mesh filename=package://ubtech/meshes/right_middle_2.STL
- link right_ring_1: geometry visual mesh filename=package://ubtech/meshes/right_ring_1.STL
- link right_ring_2: geometry visual mesh filename=package://ubtech/meshes/right_ring_2.STL
- link right_thumb_1: geometry visual mesh filename=package://ubtech/meshes/right_thumb_1.STL
- link right_thumb_2: geometry visual mesh filename=package://ubtech/meshes/right_thumb_2.STL
- link right_thumb_3: geometry visual mesh filename=package://ubtech/meshes/right_thumb_3.STL
- link right_thumb_4: geometry visual mesh filename=package://ubtech/meshes/right_thumb_4.STL
Joints:
- joint ee_x_axis_joint: origin xyz=0.05 0.0 0.1 rpy=0 0 1.57 -> xyz=0.1 0.0 0.1 rpy=0 0 1.57
- joint ee_y_axis_joint: origin xyz=0.05 0.0 0.1 rpy=1.57 0 0 -> xyz=0.1 0.0 0.1 rpy=1.57 0 0
- joint ee_z_axis_joint: origin xyz=0.05 0.0 0.1 rpy=0 1.57 0 -> xyz=0.1 0.0 0.1 rpy=0 1.57 0
- joint endeffector_joint: origin xyz=0.05 0.0 0.1 rpy=1.57 -1.57 -1.57 -> xyz=0.1 0.0 0.1 rpy=1.57 -1.57 -1.57
