Commit message: S2 working

File: myGym/envs/robots/S2/S2.urdf (robot description, URDF)
Before this commit: robot S2, 68 links, 67 joints
Links:
- removed link body_yaw_link
- added link waist_yaw_link, mass 22.0; collision mesh filename=package://S2/meshes/waist_yaw_link.STL; visual mesh filename=package://S2/meshes/waist_yaw_link.STL
- link L_base_link: geometry collision mesh filename=package://S2/meshes/L_base_link.STL; visual mesh filename=package://S2/meshes/L_base_link.STL
- link R_base_link: geometry collision mesh filename=package://S2/meshes/R_base_link.STL; visual mesh filename=package://S2/meshes/R_base_link.STL
- link ankle_pitch_l_link: geometry collision mesh filename=package://S2/meshes/ankle_pitch_l_link.STL; visual mesh filename=package://S2/meshes/ankle_pitch_l_link.STL
- link ankle_pitch_r_link: geometry collision mesh filename=package://S2/meshes/ankle_pitch_r_link.STL; visual mesh filename=package://S2/meshes/ankle_pitch_r_link.STL
- link ankle_roll_l_link: geometry collision mesh filename=package://S2/meshes/ankle_roll_l_link.STL; visual mesh filename=package://S2/meshes/ankle_roll_l_link.STL
- link ankle_roll_r_link: geometry collision mesh filename=package://S2/meshes/ankle_roll_r_link.STL; visual mesh filename=package://S2/meshes/ankle_roll_r_link.STL
- link camera_body_back_link: geometry collision mesh filename=package://S2/meshes/camera_body_back_link.STL; visual mesh filename=package://S2/meshes/camera_body_back_link.STL
- link camera_body_front_link: geometry collision mesh filename=package://S2/meshes/camera_body_front_link.STL; visual mesh filename=package://S2/meshes/camera_body_front_link.STL
- link camera_head_link: geometry collision mesh filename=package://S2/meshes/camera_head_link.STL; visual mesh filename=package://S2/meshes/camera_head_link.STL
- link ee_x_axis: mass None -> 0.0001
- link ee_y_axis: mass None -> 0.0001
- link ee_z_axis: mass None -> 0.0001
- link elbow_pitch_l_link: geometry collision mesh filename=package://S2/meshes/elbow_pitch_l_link.STL; visual mesh filename=package://S2/meshes/elbow_pitch_l_link.STL
- link elbow_pitch_r_link: geometry collision mesh filename=package://S2/meshes/elbow_pitch_r_link.STL; visual mesh filename=package://S2/meshes/elbow_pitch_r_link.STL
- link elbow_yaw_l_link: geometry collision mesh filename=package://S2/meshes/elbow_yaw_l_link.STL; visual mesh filename=package://S2/meshes/elbow_yaw_l_link.STL
- link elbow_yaw_r_link: geometry collision mesh filename=package://S2/meshes/elbow_yaw_r_link.STL; visual mesh filename=package://S2/meshes/elbow_yaw_r_link.STL
- link endeffector: mass None -> 0.0001
- link gripper: mass 0.15210234 -> 0.0001; geometry visual sphere radius=0.005
- link head_pitch_link: geometry collision mesh filename=package://S2/meshes/head_pitch_link.STL; visual mesh filename=package://S2/meshes/head_pitch_link.STL
- link head_roll_link: geometry collision mesh filename=package://S2/meshes/head_roll_link.STL; visual mesh filename=package://S2/meshes/head_roll_link.STL
- link head_yaw_link: geometry collision mesh filename=package://S2/meshes/head_yaw_link.STL; visual mesh filename=package://S2/meshes/head_yaw_link.STL
- link hip_pitch_l_link: geometry collision mesh filename=package://S2/meshes/hip_pitch_l_link.STL; visual mesh filename=package://S2/meshes/hip_pitch_l_link.STL
- link hip_pitch_r_link: geometry collision mesh filename=package://S2/meshes/hip_pitch_r_link.STL; visual mesh filename=package://S2/meshes/hip_pitch_r_link.STL
- link hip_roll_l_link: geometry collision mesh filename=package://S2/meshes/hip_roll_l_link.STL; visual mesh filename=package://S2/meshes/hip_roll_l_link.STL
- link hip_roll_r_link: geometry collision mesh filename=package://S2/meshes/hip_roll_r_link.STL; visual mesh filename=package://S2/meshes/hip_roll_r_link.STL
- link hip_yaw_l_link: geometry collision mesh filename=package://S2/meshes/hip_yaw_l_link.STL; visual mesh filename=package://S2/meshes/hip_yaw_l_link.STL
- link hip_yaw_r_link: geometry collision mesh filename=package://S2/meshes/hip_yaw_r_link.STL; visual mesh filename=package://S2/meshes/hip_yaw_r_link.STL
- link imu_link: geometry collision mesh filename=package://S2/meshes/imu_link.STL; visual mesh filename=package://S2/meshes/imu_link.STL
- link knee_pitch_l_link: geometry collision mesh filename=package://S2/meshes/knee_pitch_l_link.STL; visual mesh filename=package://S2/meshes/knee_pitch_l_link.STL
- link knee_pitch_r_link: geometry collision mesh filename=package://S2/meshes/knee_pitch_r_link.STL; visual mesh filename=package://S2/meshes/knee_pitch_r_link.STL
- link left_index_1: geometry collision mesh filename=package://S2/meshes/left_index_1.STL; visual mesh filename=package://S2/meshes/left_index_1.STL
- link left_index_2: geometry collision mesh filename=package://S2/meshes/left_index_2.STL; visual mesh filename=package://S2/meshes/left_index_2.STL
- link left_little_1: geometry collision mesh filename=package://S2/meshes/left_little_1.STL; visual mesh filename=package://S2/meshes/left_little_1.STL
- link left_little_2: geometry collision mesh filename=package://S2/meshes/left_little_2.STL; visual mesh filename=package://S2/meshes/left_little_2.STL
- link left_middle_1: geometry collision mesh filename=package://S2/meshes/left_middle_1.STL; visual mesh filename=package://S2/meshes/left_middle_1.STL
- link left_middle_2: geometry collision mesh filename=package://S2/meshes/left_middle_2.STL; visual mesh filename=package://S2/meshes/left_middle_2.STL
- link left_ring_1: geometry collision mesh filename=package://S2/meshes/left_ring_1.STL; visual mesh filename=package://S2/meshes/left_ring_1.STL
- link left_ring_2: geometry collision mesh filename=package://S2/meshes/left_ring_2.STL; visual mesh filename=package://S2/meshes/left_ring_2.STL
- link left_tcp_link: geometry collision mesh filename=package://S2/meshes/left_tcp_link.STL; visual mesh filename=package://S2/meshes/left_tcp_link.STL
- link left_thumb_1: geometry collision mesh filename=package://S2/meshes/left_thumb_1.STL; visual mesh filename=package://S2/meshes/left_thumb_1.STL
- link left_thumb_2: geometry collision mesh filename=package://S2/meshes/left_thumb_2.STL; visual mesh filename=package://S2/meshes/left_thumb_2.STL
- link left_thumb_3: geometry collision mesh filename=package://S2/meshes/left_thumb_3.STL; visual mesh filename=package://S2/meshes/left_thumb_3.STL
- link left_thumb_4: geometry collision mesh filename=package://S2/meshes/left_thumb_4.STL; visual mesh filename=package://S2/meshes/left_thumb_4.STL
- link pelvis: geometry collision mesh filename=package://S2/meshes/pelvis.STL; visual mesh filename=package://S2/meshes/pelvis.STL
- link right_index_1: geometry collision mesh filename=package://S2/meshes/right_index_1.STL; visual mesh filename=package://S2/meshes/right_index_1.STL
- link right_index_2: geometry collision mesh filename=package://S2/meshes/right_index_2.STL; visual mesh filename=package://S2/meshes/right_index_2.STL
- link right_little_1: geometry collision mesh filename=package://S2/meshes/right_little_1.STL; visual mesh filename=package://S2/meshes/right_little_1.STL
- link right_little_2: geometry collision mesh filename=package://S2/meshes/right_little_2.STL; visual mesh filename=package://S2/meshes/right_little_2.STL
- link right_middle_1: geometry collision mesh filename=package://S2/meshes/right_middle_1.STL; visual mesh filename=package://S2/meshes/right_middle_1.STL
- link right_middle_2: geometry collision mesh filename=package://S2/meshes/right_middle_2.STL; visual mesh filename=package://S2/meshes/right_middle_2.STL
- link right_ring_1: geometry collision mesh filename=package://S2/meshes/right_ring_1.STL; visual mesh filename=package://S2/meshes/right_ring_1.STL
- link right_ring_2: geometry collision mesh filename=package://S2/meshes/right_ring_2.STL; visual mesh filename=package://S2/meshes/right_ring_2.STL
- link right_tcp_link: geometry collision mesh filename=package://S2/meshes/right_tcp_link.STL; visual mesh filename=package://S2/meshes/right_tcp_link.STL
- link right_thumb_1: geometry collision mesh filename=package://S2/meshes/right_thumb_1.STL; visual mesh filename=package://S2/meshes/right_thumb_1.STL
- link right_thumb_2: geometry collision mesh filename=package://S2/meshes/right_thumb_2.STL; visual mesh filename=package://S2/meshes/right_thumb_2.STL
- link right_thumb_3: geometry collision mesh filename=package://S2/meshes/right_thumb_3.STL; visual mesh filename=package://S2/meshes/right_thumb_3.STL
- link right_thumb_4: geometry collision mesh filename=package://S2/meshes/right_thumb_4.STL; visual mesh filename=package://S2/meshes/right_thumb_4.STL
- link shoulder_pitch_l_link: geometry collision mesh filename=package://S2/meshes/shoulder_pitch_l_link.STL; visual mesh filename=package://S2/meshes/shoulder_pitch_l_link.STL
- link shoulder_pitch_r_link: geometry collision mesh filename=package://S2/meshes/shoulder_pitch_r_link.STL; visual mesh filename=package://S2/meshes/shoulder_pitch_r_link.STL
- link shoulder_roll_l_link: geometry collision mesh filename=package://S2/meshes/shoulder_roll_l_link.STL; visual mesh filename=package://S2/meshes/shoulder_roll_l_link.STL
- link shoulder_roll_r_link: geometry collision mesh filename=package://S2/meshes/shoulder_roll_r_link.STL; visual mesh filename=package://S2/meshes/shoulder_roll_r_link.STL
- link shoulder_yaw_l_link: geometry collision mesh filename=package://S2/meshes/shoulder_yaw_l_link.STL; visual mesh filename=package://S2/meshes/shoulder_yaw_l_link.STL
- link shoulder_yaw_r_link: geometry collision mesh filename=package://S2/meshes/shoulder_yaw_r_link.STL; visual mesh filename=package://S2/meshes/shoulder_yaw_r_link.STL
- link wrist_pitch_l_link: geometry collision mesh filename=package://S2/meshes/wrist_pitch_l_link.STL; visual mesh filename=package://S2/meshes/wrist_pitch_l_link.STL
- link wrist_pitch_r_link: geometry collision mesh filename=package://S2/meshes/wrist_pitch_r_link.STL; visual mesh filename=package://S2/meshes/wrist_pitch_r_link.STL
- link wrist_roll_l_link: geometry collision mesh filename=package://S2/meshes/wrist_roll_l_link.STL; visual mesh filename=package://S2/meshes/wrist_roll_l_link.STL
- link wrist_roll_r_link: geometry collision mesh filename=package://S2/meshes/wrist_roll_r_link.STL; visual mesh filename=package://S2/meshes/wrist_roll_r_link.STL
Joints:
- removed joint R_base_gripper_fix
- removed joint body_yaw_joint
- removed joint elbow_pitch_r_joint
- removed joint elbow_yaw_r_joint
- removed joint right_index_1_joint
- removed joint right_little_1_joint
- removed joint right_middle_1_joint
- removed joint right_ring_1_joint
- removed joint right_thumb_1_joint
- removed joint shoulder_pitch_r_joint
- removed joint shoulder_roll_r_joint
- removed joint shoulder_yaw_r_joint
- removed joint wrist_pitch_r_joint
- removed joint wrist_roll_r_joint
- added joint body_yaw_rjoint: type revolute, parent pelvis, child waist_yaw_link, origin xyz=0 0 0 rpy=0 0 0, axis 0 0 1, limit lower=-2.9670597283903604 upper=3.141592653589793 effort=91.0 velocity=9.215338450530059
- added joint elbow_pitch_r_rjoint: type revolute, parent shoulder_yaw_r_link, child elbow_pitch_r_link, origin xyz=0.02 0 -0.1975 rpy=0 0 0, axis 0 1 0, limit lower=-2.6179938779914944 upper=0.2617993877991494 effort=35.0 velocity=5.235987755982989
- added joint elbow_yaw_r_rjoint: type revolute, parent elbow_pitch_r_link, child elbow_yaw_r_link, origin xyz=-0.02 0 -0.0543 rpy=0 0 0, axis 0 0 1, limit lower=-2.9670597283903604 upper=2.9670597283903604 effort=24.0 velocity=10.471975511965978
- added joint gripper_joint: type fixed, parent R_base_link, child gripper, origin xyz=-0.00 -0.00 0.0 rpy=0 0 0
- added joint right_index_1_gjoint: type revolute, parent R_base_link, child right_index_1, origin xyz=-0.000285 0.020275 0.136946 rpy=1.5359 0 0, axis 0 -0.069756  -0.997564, limit lower=0 upper=1.333 effort=50 velocity=1
- added joint right_little_1_gjoint: type revolute, parent R_base_link, child right_little_1, origin xyz=-0.000285 -0.037422 0.13446 rpy=1.6755 0 0, axis 0 0 -1, limit lower=0 upper=1.333 effort=50 velocity=1
- added joint right_middle_1_gjoint: type revolute, parent R_base_link, child right_middle_1, origin xyz=-0.000285 0.00295 0.1371 rpy=1.5708 0 0, axis 0 0 -1, limit lower=0 upper=1.333 effort=50 velocity=1
- added joint right_ring_1_gjoint: type revolute, parent R_base_link, child right_ring_1, origin xyz=-0.000285 -0.018271 0.136282 rpy=1.6232 0 0, axis 0 0 -1, limit lower=0 upper=1.333 effort=50 velocity=1
- added joint right_thumb_1_gjoint: type revolute, parent R_base_link, child right_thumb_1, origin xyz=0.01696 0.02045 0.06635 rpy=0 0 0, axis 0 0 -1, limit lower=0 upper=1.246165 effort=50 velocity=1
- added joint shoulder_pitch_r_rjoint: type revolute, parent waist_yaw_link, child shoulder_pitch_r_link, origin xyz=0 -0.1444 0.37712 rpy=-0.087266 0 0, axis 0 1 0, limit lower=-2.9670597283903604 upper=2.9670597283903604 effort=91.0 velocity=9.215338450530059
- added joint shoulder_roll_r_rjoint: type revolute, parent shoulder_pitch_r_link, child shoulder_roll_r_link, origin xyz=0 -0.068 0 rpy=0 0 0, axis 1 0 0, limit lower=-2.6179938779914944 upper=0.2617993877991494 effort=95.0 velocity=3.979350694547071
- added joint shoulder_yaw_r_rjoint: type revolute, parent shoulder_roll_r_link, child shoulder_yaw_r_link, origin xyz=0 0 -0.1025 rpy=0 0 0, axis 0 0 1, limit lower=-2.9670597283903604 upper=2.9670597283903604 effort=35.0 velocity=5.235987755982989
- added joint wrist_pitch_r_rjoint: type revolute, parent elbow_yaw_r_link, child wrist_pitch_r_link, origin xyz=0 0 -0.1887 rpy=0 0 0, axis 0 1 0, limit lower=-0.7853981633974483 upper=1.0471975511965976 effort=6.3 velocity=7.5398223686155035
- added joint wrist_roll_r_rjoint: type revolute, parent wrist_pitch_r_link, child wrist_roll_r_link, origin xyz=0 0 -0.02 rpy=0 0 0, axis 1 0 0, limit lower=-1.3089969389957472 upper=1.6580627893946132 effort=6.3 velocity=7.5398223686155035
- joint ankle_pitch_l_joint: type revolute -> fixed
- joint ankle_pitch_r_joint: type revolute -> fixed
- joint ankle_roll_l_joint: type revolute -> fixed
- joint ankle_roll_r_joint: type revolute -> fixed
- joint camera_body_back_joint: parent body_yaw_link -> waist_yaw_link
- joint camera_body_front_joint: parent body_yaw_link -> waist_yaw_link
- joint ee_x_axis_joint: origin xyz=0.05 0.0 0.1 rpy=-1.57 -1.57 0 -> xyz=0.03 0.0 0.10 rpy=0 0 1.57
- joint ee_y_axis_joint: origin xyz=0.05 0.0 0.1 rpy=-1.57 -1.57 0 -> xyz=0.03 0.0 0.10 rpy=1.57 0 0
- joint ee_z_axis_joint: origin xyz=0.05 0.0 0.1 rpy=-1.57 -1.57 0 -> xyz=0.03 0.0 0.10 rpy=0 1.57 0
- joint elbow_pitch_l_joint: type revolute -> fixed
- joint elbow_yaw_l_joint: type revolute -> fixed
- joint endeffector_joint: origin xyz=0.05 0.0 0.1 rpy=1.57 0 0 -> xyz=0.03 0.0 0.10 rpy=0 -1.57 0
- joint head_pitch_joint: type revolute -> fixed
- joint head_roll_joint: type revolute -> fixed
- joint head_yaw_joint: parent body_yaw_link -> waist_yaw_link; type revolute -> fixed
- joint hip_pitch_l_joint: type revolute -> fixed
- joint hip_pitch_r_joint: type revolute -> fixed
- joint hip_roll_l_joint: type revolute -> fixed
- joint hip_roll_r_joint: type revolute -> fixed
- joint hip_yaw_l_joint: type revolute -> fixed
- joint hip_yaw_r_joint: type revolute -> fixed
- joint knee_pitch_l_joint: type revolute -> fixed
- joint knee_pitch_r_joint: type revolute -> fixed
- joint left_index_1_joint: type revolute -> fixed
- joint left_index_2_joint: type revolute -> fixed
- joint left_little_1_joint: type revolute -> fixed
- joint left_little_2_joint: type revolute -> fixed
- joint left_middle_1_joint: type revolute -> fixed
- joint left_middle_2_joint: type revolute -> fixed
- joint left_ring_1_joint: type revolute -> fixed
- joint left_ring_2_joint: type revolute -> fixed
- joint left_thumb_1_joint: type revolute -> fixed
- joint left_thumb_2_joint: type revolute -> fixed
- joint left_thumb_3_joint: type revolute -> fixed
- joint left_thumb_4_joint: type revolute -> fixed
- joint right_index_2_joint: type revolute -> fixed
- joint right_little_2_joint: type revolute -> fixed
- joint right_middle_2_joint: type revolute -> fixed
- joint right_ring_2_joint: type revolute -> fixed
- joint right_thumb_2_joint: type revolute -> fixed
- joint right_thumb_3_joint: type revolute -> fixed
- joint right_thumb_4_joint: type revolute -> fixed
- joint shoulder_pitch_l_joint: parent body_yaw_link -> waist_yaw_link; type revolute -> fixed
- joint shoulder_roll_l_joint: limit lower=-1.0471975511965976 upper=1.8325957145940461 effort=95.0 velocity=3.979350694547071 -> lower=-0.2617993877991494 upper=2.6179938779914944 effort=95.0 velocity=3.979350694547071; type revolute -> fixed
- joint shoulder_yaw_l_joint: type revolute -> fixed
- joint wrist_pitch_l_joint: limit lower=-1.3089969389957472 upper=1.6580627893946132 effort=6.3 velocity=7.5398223686155035 -> lower=-0.7853981633974483 upper=1.0471975511965976 effort=6.3 velocity=7.5398223686155035; type revolute -> fixed
- joint wrist_roll_l_joint: limit lower=-1.0471975511965976 upper=0.7853981633974483 effort=6.3 velocity=7.5398223686155035 -> lower=-1.6580627893946132 upper=1.3089969389957472 effort=6.3 velocity=7.5398223686155035; type revolute -> fixed
